File: Drivers.sch (KiCad schematic (older format))
At the start: 23 parts

Commit message: 1
Other:
- note added: "change torqer driver to BD6210F-E2\n"
- note added: "these wont drive the bldc motors"
Changed lines of the file:
@@
 $Descr B 17000 11000
 encoding utf-8
-Sheet 3 5
+Sheet 4 5
 Title ""
 Date ""
@@
 Text Notes 9400 8350 0    100  ~ 20
 figure connectors out for torqe rods
+Text Notes 4150 5500 0    50   ~ 0
+change torqer driver to BD6210F-E2\n
+Text Notes 4150 5600 0    50   ~ 0
+these wont drive the bldc motors
 $EndSCHEMATC
