File: Full_Bridge.kicad_sch (KiCad schematic)
At the start: 8 parts, among them U1 DRV8838DSGT

Commit message: design updates
Parts:
- renumbered C1 to C49, C2 to C50, C3 to C51, D1 to D6, R1 to R59, R2 to R60, R3 to R61, U1 to U16
Changed lines of the file:
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@@
     (effects (font (size 1.27 1.27)) (justify left))
   )
-  (symbol (lib_id "power:GND") (at 80.01 88.9 0)
+  (symbol (lib_id "power:GND") (at 80.01 88.9 0) (unit 1)
     (in_bom yes) (on_board yes) (fields_autoplaced)
-    (property "Reference" "#PWR07" (id 0) (at 80.01 95.25 0)
+    (property "Reference" "#PWR044" (id 0) (at 80.01 95.25 0)
       (effects (font (size 1.27 1.27)) hide)
     )
@@
     (pin "1")
   )
-  (symbol (lib_id "Device:D_TVS") (at 161.29 92.71 90)
+  (symbol (lib_id "Device:D_TVS") (at 161.29 92.71 90) (unit 1)
     (in_bom yes) (on_board yes) (fields_autoplaced)
-    (property "Reference" "D1" (id 0) (at 163.83 91.4399 90)
+    (property "Reference" "D6" (id 0) (at 163.83 91.4399 90)
       (effects (font (size 1.27 1.27)) (justify right))
     )
@@
       (effects (font (size 1.27 1.27)) hide)
     )
-    (property "Datasheet" "~" (id 3) (at 161.29 92.71 0)
+    (property "Datasheet" "TPSMF4L6.0A" (id 3) (at 161.29 92.71 0)
       (effects (font (size 1.27 1.27)) hide)
     )
@@
     (pin "2")
   )
-  (symbol (lib_id "Device:C") (at 80.01 85.09 0)
+  (symbol (lib_id "Device:C") (at 80.01 85.09 0) (unit 1)
     (in_bom yes) (on_board yes) (fields_autoplaced)
-    (property "Reference" "C1" (id 0) (at 82.931 84.1815 0)
+    (property "Reference" "C49" (id 0) (at 82.931 84.1815 0)
       (effects (font (size 1.27 1.27)) (justify left))
     )
@@
     (pin "2")
   )
-  (symbol (lib_id "Device:R_US") (at 118.11 91.44 90)
+  (symbol (lib_id "Device:R_US") (at 118.11 91.44 90) (unit 1)
     (in_bom yes) (on_board yes)
-    (property "Reference" "R2" (id 0) (at 114.3 90.17 90))
+    (property "Reference" "R60" (id 0) (at 114.3 90.17 90))
     (property "Value" "100" (id 1) (at 121.92 90.17 90))
     (property "Footprint" "Resistor_SMD:R_0603_1608Metric" (id 2) (at 118.364 90.424 90)
@@
     (pin "2")
   )
-  (symbol (lib_id "power:GND") (at 193.04 88.9 0)
+  (symbol (lib_id "power:GND") (at 193.04 88.9 0) (unit 1)
     (in_bom yes) (on_board yes) (fields_autoplaced)
-    (property "Reference" "#PWR010" (id 0) (at 193.04 95.25 0)
+    (property "Reference" "#PWR047" (id 0) (at 193.04 95.25 0)
       (effects (font (size 1.27 1.27)) hide)
     )
@@
     (pin "1")
   )
-  (symbol (lib_id "power:GND") (at 147.32 96.52 0)
+  (symbol (lib_id "power:GND") (at 147.32 96.52 0) (unit 1)
     (in_bom yes) (on_board yes) (fields_autoplaced)
-    (property "Reference" "#PWR08" (id 0) (at 147.32 102.87 0)
+    (property "Reference" "#PWR045" (id 0) (at 147.32 102.87 0)
       (effects (font (size 1.27 1.27)) hide)
     )
@@
     (pin "1")
   )
-  (symbol (lib_id "power:GND") (at 180.34 88.9 0)
+  (symbol (lib_id "power:GND") (at 180.34 88.9 0) (unit 1)
     (in_bom yes) (on_board yes) (fields_autoplaced)
-    (property "Reference" "#PWR09" (id 0) (at 180.34 95.25 0)
+    (property "Reference" "#PWR046" (id 0) (at 180.34 95.25 0)
       (effects (font (size 1.27 1.27)) hide)
     )
@@
     (pin "1")
   )
-  (symbol (lib_id "Device:R_US") (at 118.11 93.98 90)
+  (symbol (lib_id "Device:R_US") (at 118.11 93.98 90) (unit 1)
     (in_bom yes) (on_board yes)
-    (property "Reference" "R3" (id 0) (at 114.3 92.71 90))
+    (property "Reference" "R61" (id 0) (at 114.3 92.71 90))
     (property "Value" "100" (id 1) (at 121.92 92.71 90))
     (property "Footprint" "Resistor_SMD:R_0603_1608Metric" (id 2) (at 118.364 92.964 90)
@@
     (pin "2")
   )
-  (symbol (lib_id "magnetotorquer-test-board:DRV8838DSGT") (at 134.62 87.63 0)
+  (symbol (lib_id "magnetotorquer-test-board:DRV8838DSGT") (at 134.62 87.63 0) (unit 1)
     (in_bom yes) (on_board yes) (fields_autoplaced)
-    (property "Reference" "U1" (id 0) (at 134.62 73.5035 0))
+    (property "Reference" "U16" (id 0) (at 134.62 73.5035 0))
     (property "Value" "DRV8838DSGT" (id 1) (at 134.62 76.2786 0))
     (property "Footprint" "Package_SON:WSON-8-1EP_2x2mm_P0.5mm_EP0.9x1.6mm" (id 2) (at 134.62 109.22 0)
@@
     (pin "9")
   )
-  (symbol (lib_id "Device:R_US") (at 118.11 88.9 90)
+  (symbol (lib_id "Device:R_US") (at 118.11 88.9 90) (unit 1)
     (in_bom yes) (on_board yes)
-    (property "Reference" "R1" (id 0) (at 114.3 87.63 90))
+    (property "Reference" "R59" (id 0) (at 114.3 87.63 90))
     (property "Value" "100" (id 1) (at 121.92 87.63 90))
     (property "Footprint" "Resistor_SMD:R_0603_1608Metric" (id 2) (at 118.364 87.884 90)
@@
     (pin "2")
   )
-  (symbol (lib_id "power:+3.3V") (at 80.01 81.28 0)
+  (symbol (lib_id "power:+3.3V") (at 80.01 81.28 0) (unit 1)
     (in_bom yes) (on_board yes) (fields_autoplaced)
-    (property "Reference" "#PWR06" (id 0) (at 80.01 85.09 0)
+    (property "Reference" "#PWR043" (id 0) (at 80.01 85.09 0)
       (effects (font (size 1.27 1.27)) hide)
     )
@@
     (pin "1")
   )
-  (symbol (lib_id "Device:C") (at 180.34 85.09 0)
+  (symbol (lib_id "Device:C") (at 180.34 85.09 0) (unit 1)
     (in_bom yes) (on_board yes) (fields_autoplaced)
-    (property "Reference" "C2" (id 0) (at 183.261 84.1815 0)
+    (property "Reference" "C50" (id 0) (at 183.261 84.1815 0)
       (effects (font (size 1.27 1.27)) (justify left))
     )
@@
     (pin "2")
   )
-  (symbol (lib_id "Device:C") (at 193.04 85.09 0)
+  (symbol (lib_id "Device:C") (at 193.04 85.09 0) (unit 1)
     (in_bom yes) (on_board yes) (fields_autoplaced)
-    (property "Reference" "C3" (id 0) (at 195.961 84.1815 0)
+    (property "Reference" "C51" (id 0) (at 195.961 84.1815 0)
       (effects (font (size 1.27 1.27)) (justify left))
     )

Commit message: misc
Parts:
- added R?: 100k, Resistor_SMD:R_0603_1608Metric, symbol Device:R_US
Connections:
- net GND: now also R?.2
- net ~{SLEEP}: now also R?.1
Changed lines of the file:
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@@
   (junction (at 161.29 97.79) (diameter 0) (color 0 0 0 0)
   )
+  (junction (at 99.06 88.9) (diameter 0) (color 0 0 0 0)
+  )
   (polyline (pts (xy 167.64 100.33) (xy 167.64 105.41))
     (stroke (width 0) (type default) (color 0 0 0 0))
@@
     (stroke (width 0) (type default) (color 0 0 0 0))
   )
+  (wire (pts (xy 161.29 97.79) (xy 166.37 97.79))
+    (stroke (width 0) (type default) (color 0 0 0 0))
+  )
   (wire (pts (xy 80.01 81.28) (xy 124.46 81.28))
     (stroke (width 0) (type default) (color 0 0 0 0))
   )
-  (wire (pts (xy 161.29 97.79) (xy 166.37 97.79))
-    (stroke (width 0) (type default) (color 0 0 0 0))
-  )
   (wire (pts (xy 161.29 96.52) (xy 161.29 97.79))
     (stroke (width 0) (type default) (color 0 0 0 0))
@@
     (stroke (width 0) (type default) (color 0 0 0 0))
   )
+  (wire (pts (xy 97.79 88.9) (xy 99.06 88.9))
+    (stroke (width 0) (type default) (color 0 0 0 0))
+  )
   (polyline (pts (xy 134.62 58.42) (xy 134.62 110.49))
     (stroke (width 0) (type default) (color 0 0 0 0))
@@
     (stroke (width 0) (type default) (color 0 0 0 0))
   )
-  (wire (pts (xy 111.76 88.9) (xy 114.3 88.9))
+  (wire (pts (xy 99.06 88.9) (xy 114.3 88.9))
     (stroke (width 0) (type default) (color 0 0 0 0))
   )
@@
     (effects (font (size 1.27 1.27)) (justify left bottom))
   )
-  (hierarchical_label "~{SLEEP}" (shape input) (at 111.76 88.9 180)
+  (hierarchical_label "~{SLEEP}" (shape input) (at 97.79 88.9 180)
     (effects (font (size 1.27 1.27)) (justify right))
   )
@@
     (pin "9")
   )
+  (symbol (lib_id "Device:R_US") (at 99.06 92.71 0) (unit 1)
+    (in_bom yes) (on_board yes) (fields_autoplaced)
+    (property "Reference" "R?" (id 0) (at 101.6 91.4399 0)
+      (effects (font (size 1.27 1.27)) (justify left))
+    )
+    (property "Value" "100k" (id 1) (at 101.6 93.9799 0)
+      (effects (font (size 1.27 1.27)) (justify left))
+    )
+    (property "Footprint" "Resistor_SMD:R_0603_1608Metric" (id 2) (at 100.076 92.964 90)
+      (effects (font (size 1.27 1.27)) hide)
+    )
+    (property "Datasheet" "~" (id 3) (at 99.06 92.71 0)
+      (effects (font (size 1.27 1.27)) hide)
+    )
+    (pin "1")
+    (pin "2")
+  )
   (symbol (lib_id "Device:R_US") (at 118.11 88.9 90) (unit 1)
     (in_bom yes) (on_board yes)
@@
     (pin "2")
   )
+  (symbol (lib_id "power:GND") (at 99.06 96.52 0) (unit 1)
+    (in_bom yes) (on_board yes) (fields_autoplaced)
+    (property "Reference" "#PWR?" (id 0) (at 99.06 102.87 0)
+      (effects (font (size 1.27 1.27)) hide)
+    )
+    (property "Value" "GND" (id 1) (at 99.06 101.0825 0))
+    (property "Footprint" "" (id 2) (at 99.06 96.52 0)
+      (effects (font (size 1.27 1.27)) hide)
+    )
+    (property "Datasheet" "" (id 3) (at 99.06 96.52 0)
+      (effects (font (size 1.27 1.27)) hide)
+    )
+    (pin "1")
+  )
   (symbol (lib_id "Device:C") (at 193.04 85.09 0) (unit 1)
