File: Full_Bridge.kicad_sch (KiCad schematic)
At the start: 9 parts, among them U16 DRV8838DSGT

Commit message: updates
Parts:
- gave numbers to parts that had none: 1
Changed lines of the file:
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@@
   (symbol (lib_id "Device:R_US") (at 99.06 92.71 0) (unit 1)
     (in_bom yes) (on_board yes) (fields_autoplaced)
-    (property "Reference" "R?" (id 0) (at 101.6 91.4399 0)
+    (property "Reference" "R111" (id 0) (at 101.6 91.4399 0)
       (effects (font (size 1.27 1.27)) (justify left))
     )
@@
   (symbol (lib_id "power:GND") (at 99.06 96.52 0) (unit 1)
     (in_bom yes) (on_board yes) (fields_autoplaced)
-    (property "Reference" "#PWR?" (id 0) (at 99.06 102.87 0)
+    (property "Reference" "#PWR0135" (id 0) (at 99.06 102.87 0)
       (effects (font (size 1.27 1.27)) hide)
     )
