File: FP Interface Card.kicad_sch (KiCad schematic)
At the start: 18 parts, among them J1 T2M-105-01-X-D-TH-DS, P1 Card Edge for HSEC8-160-01-S-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, Q1 Q_NMOS_GSD, Q2 Q_NMOS_GSD, Q3 Q_NMOS_GSD, Q4 Q_NMOS_GSD

Commit message: 1
Parts:
- added TP1, TP2, TP3, TP4, TP5, TP6, TP7, TP8: TestPoint, TestPoint:TestPoint_Pad_2.5x2.5mm, symbol Connector:TestPoint
Connections:
- net H1-19: now also TP5.1
- net H1-20: now also TP6.1
- net H1-6: now also TP1.1
- net H2-6: now also TP2.1
- net RESET: now also TP3.1
- net RXD: now also TP8.1
- net SERVO_PWR_CTRL: now also TP4.1
- net TXD: now also TP7.1

Commit message: generated fab files
Connections:
- net +5V: now also J1.10 (Pin_10), J1.8 (Pin_8), J1.9 (Pin_9)
Changed lines of the file:
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@@
     (pin "3")
+  )
+  (symbol (lib_id "power:+5V") (at 328.93 52.07 0) (unit 1)
+    (in_bom yes) (on_board yes) (fields_autoplaced)
+    (property "Reference" "#PWR?" (id 0) (at 328.93 55.88 0)
+      (effects (font (size 1.27 1.27)) hide)
+    )
+    (property "Value" "+5V" (id 1) (at 328.93 48.4655 0))
+    (property "Footprint" "" (id 2) (at 328.93 52.07 0)
+      (effects (font (size 1.27 1.27)) hide)
+    )
+    (property "Datasheet" "" (id 3) (at 328.93 52.07 0)
+      (effects (font (size 1.27 1.27)) hide)
+    )
+    (pin "1")
   )
   (symbol (lib_id "Device:R") (at 322.58 158.115 270) (unit 1)
@@
       (reference "#PWR012") (unit 1) (value "+3.3V") (footprint "")
     )
+    (path "/800e4b03-3f41-427c-8741-99a61b567cb8"
+      (reference "#PWR?") (unit 1) (value "+5V") (footprint "")
+    )
     (path "/00000000-0000-0000-0000-000061d3502c/00000000-0000-0000-0000-000061df4655"

Commit message: 1
Other:
- added sheet I2C-Protection (I2C-Protection.kicad_sch)
- added sheet IMU (IMU.kicad_sch)
- added sheet Magnetotorquer Drivers (magnetotorquer-driver.kicad_sch)
- moved on the sheet: J1

Commit message: majority of routing completed
Parts:
- removed Q1, Q2, Q3, Q4: Q_NMOS_GSD, Package_TO_SOT_SMD:SOT-23, symbol Device:Q_NMOS_GSD
- removed R1, R10, R2, R3, R4, R7, R8, R9: 10k, Resistor_SMD:R_0603_1608Metric_Pad0.98x0.95mm_HandSolder, symbol Device:R
- removed R11, R12, R5, R6: 0, Resistor_SMD:R_0603_1608Metric_Pad0.98x0.95mm_HandSolder, symbol Device:R
- removed TP1, TP2, TP3, TP4, TP5, TP6, TP7, TP8: TestPoint, TestPoint:TestPoint_Pad_2.5x2.5mm, symbol Connector:TestPoint
- added J2: T2M-105-01-X-D-TH-DS, payload-interface-board:SAMTEC_T2M-105-01-X-D-TH-DS, symbol Connector_Generic:Conn_01x10
Connections:
- new net X+: J2.1 (Pin_1)
- new net X-: J2.2 (Pin_2)
- new net Y+: J2.5 (Pin_5)
- new net Y-: J2.6 (Pin_6)
- new net Z+: J2.9 (Pin_9)
- new net Z-: J2.10 (Pin_10)
- no-connect marks 0 -> 4
Other:
- sheet I2C-Protection renamed I2C-Protection-2
- added sheet I2C-Protection-1 (I2C-Protection.kicad_sch)
- added sheet Level Shifter 1 (Level_Shifter.kicad_sch)
- added sheet Level Shifter 2 (Level_Shifter.kicad_sch)
- added sheet Level Shifter 3 (Level_Shifter.kicad_sch)
- added sheet Level Shifter 4 (Level_Shifter.kicad_sch)
- added sheet RockBLOCKmk2 (rockBLOCKmk2.kicad_sch)
- sheet Magnetotorquer Drivers ports: added SCL, SDA, X+, X-, Y+, Y-, Z+, Z-; removed none
- note added: "I2C PROTECTION"
- note added: "IMU"
- note added: "MAGNETORQUER DRIVERS"
- note added: "PAYLOAD LEVEL SHIFTERS"
- note added: "TO MAGNETOTORQUERS"
- note removed: "LEVEL SHIFTERS"
- moved on the sheet: J1

Commit message: 1
Parts:
- added J?: T2M-105-01-X-D-TH-DS, payload-interface-board:SAMTEC_T2M-105-01-X-D-TH-DS, symbol Connector_Generic:Conn_01x10
Other:
- removed sheet RockBLOCKmk2
- added sheet Level Shifter 5 (Level_Shifter.kicad_sch)
- added sheet Level Shifter 6 (Level_Shifter.kicad_sch)
- added sheet Level Shifter 7 (Level_Shifter.kicad_sch)
- added sheet Level Shifter 8 (Level_Shifter.kicad_sch)
- added sheet Level Shifter 9 (Level_Shifter.kicad_sch)
- note added: "ROCKBLOCK LEVEL SHIFTERS"
- note added: "TO ROCKBLOCK 9602"
- moved on the sheet: J2

Commit message: working on sch changes
Connections:
- net H1-33 is gone; now on net 5V_RF: P1.73 (Pin_73)
- net GND: now also J?.10 (Pin_10), J?.9 (Pin_9)
- net RB_rx: now also J?.7 (Pin_7)
- net RB_tx: now also J?.6 (Pin_6)
- net 5V_RF: now reaches J?.1 (Pin_1)
- net 5V_RF: now also J?.2 (Pin_2)
- net RB_OnOff: now reaches J?.8 (Pin_8)
Other:
- added sheet Ball Deployer (ball_deployer.kicad_sch)
- sheet Magnetotorquer Drivers ports: added Ball_Deploy; removed none
- note added: "PAYLOAD BALL DEPLOYER"
- note added: "make more concise"
- moved on the sheet: J?

Commit message: working on EM
Parts:
- added J?: T2M-105-01-X-D-TH-DS, payload-interface-board:SAMTEC_T2M-105-01-X-D-TH-DS, symbol Connector_Generic:Conn_01x10
Connections:
- net X+: now also J?.1 (Pin_1)
- net X-: now also J?.2 (Pin_2)
- net Y+: now also J?.5 (Pin_5)
- net Y-: now also J?.6 (Pin_6)
- net Z+: now also J?.9 (Pin_9)
- net Z-: now also J?.10 (Pin_10)
- no-connect marks 4 -> 8
Other:
- removed sheet Ball Deployer
- note added: "TO STAR TRACKER"
- note removed: "PAYLOAD BALL DEPLOYER"

Commit message: 1
Parts:
- removed J?: T2M-105-01-X-D-TH-DS, payload-interface-board:SAMTEC_T2M-105-01-X-D-TH-DS, symbol Connector_Generic:Conn_01x10
- added J? (x2): T1M-05-GF-DV, symbol Connector_Generic:Conn_02x05_Odd_Even
- added J?: T1M-03-GF-DV, symbol Connector_Generic:Conn_02x03_Odd_Even
- J1: value T2M-105-01-X-D-TH-DS -> T1M-05-GF-DV; footprint payload-interface-board:SAMTEC_T2M-105-01-X-D-TH-DS -> (none)
Connections:
- no-connect marks 8 -> 4
Other:
- note added: "make rockblock sch symbol and FP"
