File: FP Interface Card.kicad_sch (KiCad schematic)
At the start: 23 parts, among them J1 T1M-10-F-SV-L, J4 T1M-6-F-SV-L, J5 T1M-10-F-SV-L, P1 Card Edge for HSEC8-160-01-S-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, Q17 MMBT4401-7-F, Q18 MMBT4401-7-F, Q19 IRF7404TRPBF, Q22 MMBT4401-7-F, Q23 IRF7404TRPBF, U24 RockBlock_9603

Commit message: misc
Other:
- note added: "MAKE A UART PROTECTION CIRCUIT"
Changed lines of the file:
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@@
     (effects (font (size 1.27 1.27)) (justify left bottom))
+  )
+  (text "MAKE A UART PROTECTION CIRCUIT" (at 123.19 226.06 0)
+    (effects (font (size 3 3) (thickness 0.6) bold) (justify left bottom))
   )
   (text "I2C PROTECTION" (at 144.78 97.79 0)
@@
       (reference "#PWR0130") (unit 1) (value "+5V") (footprint "")
     )
+    (path "/66fbc293-b490-4097-aa2e-a081509eef04/cef6bc38-b409-4d11-9d9d-66f5cdf820a8"
+      (reference "#PWR?") (unit 1) (value "GND") (footprint "")
+    )
+    (path "/66fbc293-b490-4097-aa2e-a081509eef04/da64b43d-1777-42fd-aa6c-83f1693f3a75"
+      (reference "#PWR?") (unit 1) (value "+3.3V") (footprint "")
+    )
+    (path "/66fbc293-b490-4097-aa2e-a081509eef04/09e89dab-acb9-41af-be20-2de645189f17/eefbac55-befa-41d4-8e97-8e8daa199c09"
+      (reference "#PWR?") (unit 1) (value "GND") (footprint "")
+    )
+    (path "/66fbc293-b490-4097-aa2e-a081509eef04/5b8330c6-72aa-4625-a65f-d4d55ae3e3e8/eefbac55-befa-41d4-8e97-8e8daa199c09"
+      (reference "#PWR?") (unit 1) (value "GND") (footprint "")
+    )
+    (path "/66fbc293-b490-4097-aa2e-a081509eef04/e1ca2fa4-878d-4b56-b8ce-583c4e6d5869/eefbac55-befa-41d4-8e97-8e8daa199c09"
+      (reference "#PWR?") (unit 1) (value "GND") (footprint "")
+    )
+    (path "/66fbc293-b490-4097-aa2e-a081509eef04/f843106b-fd17-4228-bad0-d75a9c91031e"
+      (reference "#PWR?") (unit 1) (value "GND") (footprint "")
+    )
     (path "/598f4529-df2c-4919-a701-d82b23d8a129/9add4c13-659d-4245-a94b-1f7557a8d341"
       (reference "#SUPPLY01") (unit 1) (value "3.3V") (footprint "")
@@
       (reference "R116") (unit 1) (value "10k") (footprint "Resistor_SMD:R_0603_1608Metric")
     )
+    (path "/66fbc293-b490-4097-aa2e-a081509eef04/81e38486-2d79-4f20-8e68-ccba86566838"
+      (reference "R?") (unit 1) (value "100k") (footprint "Resistor_SMD:R_0603_1608Metric")
+    )
+    (path "/66fbc293-b490-4097-aa2e-a081509eef04/5b8330c6-72aa-4625-a65f-d4d55ae3e3e8/8613a8e6-b3a5-4cc5-9e3a-95a048d4aa21"
+      (reference "R?") (unit 1) (value "100k") (footprint "Resistor_SMD:R_0603_1608Metric")
+    )
+    (path "/66fbc293-b490-4097-aa2e-a081509eef04/e1ca2fa4-878d-4b56-b8ce-583c4e6d5869/8613a8e6-b3a5-4cc5-9e3a-95a048d4aa21"
+      (reference "R?") (unit 1) (value "100k") (footprint "Resistor_SMD:R_0603_1608Metric")
+    )
+    (path "/66fbc293-b490-4097-aa2e-a081509eef04/09e89dab-acb9-41af-be20-2de645189f17/8613a8e6-b3a5-4cc5-9e3a-95a048d4aa21"
+      (reference "R?") (unit 1) (value "100k") (footprint "Resistor_SMD:R_0603_1608Metric")
+    )
     (path "/66fbc293-b490-4097-aa2e-a081509eef04/0d41b933-8bc8-4fa4-b49a-44e034cc3fe8/d864aed9-fd97-43df-a424-d72767de2e57"

Commit message: updates
Parts:
- added C73: 0.01uF, Capacitor_SMD:C_0603_1608Metric, symbol Device:C
- added R113, R117: 4.7k, Resistor_SMD:R_0603_1608Metric, symbol Device:R_US
- added U26: LTC4307, Package_SO:MSOP-8_3x3mm_P0.65mm, symbol mainboard_SLI:LTC4307
Connections:
- net +3V3: now also C73.1, R113.1, R117.1, U26.1 (EN), U26.8 (VCC)
- net GND: now also C73.2, U26.4 (GND)
- net SCL_SYS: now also U26.3 (SCLIN)
- net SDA_SYS: now also U26.6 (SDAIN)
- new net I2C-Protection-1/SCL_IN: R113.2, U26.2 (SCLOUT)
- new net I2C-Protection-1/SDA_IN: R117.2, U26.7 (SDAOUT)
Other:
- note added: "main i2c bus, pycubed processor is master."
