File: 5V_amp.kicad_sch (KiCad schematic)
At the start: 6 parts, among them U23 OPA340MDBVTEP

Commit message: design updates
Parts:
- TP28: renamed from TP29; footprint TestPoint:TestPoint_Pad_2.5x2.5mm -> TestPoint:TestPoint_Pad_D1.0mm
- renumbered C67 to C64, C68 to C65, C69 to C66, RN3 to RN2, U23 to U22
Changed lines of the file:
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@@
     (effects (font (size 1.27 1.27)) (justify left))
   )
-  (symbol (lib_id "Amplifier_Operational:OPA340NA") (at 128.27 90.17 0)
+  (symbol (lib_id "Amplifier_Operational:OPA340NA") (at 128.27 90.17 0) (unit 1)
     (in_bom yes) (on_board yes) (fields_autoplaced)
-    (property "Reference" "U23" (id 0) (at 139.7 85.471 0))
+    (property "Reference" "U22" (id 0) (at 139.7 85.471 0))
     (property "Value" "OPA340MDBVTEP" (id 1) (at 139.7 88.011 0))
     (property "Footprint" "Package_TO_SOT_SMD:SOT-23-5" (id 2) (at 125.73 95.25 0)
@@
     (pin "4")
   )
-  (symbol (lib_id "power:GND") (at 166.37 97.79 0)
+  (symbol (lib_id "power:GND") (at 166.37 97.79 0) (unit 1)
     (in_bom yes) (on_board yes) (fields_autoplaced)
-    (property "Reference" "#PWR073" (id 0) (at 166.37 104.14 0)
+    (property "Reference" "#PWR068" (id 0) (at 166.37 104.14 0)
       (effects (font (size 1.27 1.27)) hide)
     )
@@
     (pin "1")
   )
-  (symbol (lib_id "Connector:TestPoint") (at 166.37 90.17 0)
+  (symbol (lib_id "Connector:TestPoint") (at 166.37 90.17 0) (unit 1)
     (in_bom yes) (on_board yes)
-    (property "Reference" "TP29" (id 0) (at 165.1 83.82 0)
+    (property "Reference" "TP28" (id 0) (at 165.1 83.82 0)
       (effects (font (size 1.27 1.27)) (justify left))
     )
@@
       (effects (font (size 1.27 1.27)) (justify left) hide)
     )
-    (property "Footprint" "TestPoint:TestPoint_Pad_2.5x2.5mm" (id 2) (at 171.45 90.17 0)
+    (property "Footprint" "TestPoint:TestPoint_Pad_D1.0mm" (id 2) (at 171.45 90.17 0)
       (effects (font (size 1.27 1.27)) hide)
     )
@@
     (pin "1")
   )
-  (symbol (lib_id "power:GND") (at 134.62 80.01 0)
+  (symbol (lib_id "power:GND") (at 134.62 80.01 0) (unit 1)
     (in_bom yes) (on_board yes) (fields_autoplaced)
-    (property "Reference" "#PWR071" (id 0) (at 134.62 86.36 0)
+    (property "Reference" "#PWR066" (id 0) (at 134.62 86.36 0)
       (effects (font (size 1.27 1.27)) hide)
     )
@@
     (pin "1")
   )
-  (symbol (lib_id "Device:C") (at 166.37 93.98 0)
+  (symbol (lib_id "Device:C") (at 166.37 93.98 0) (unit 1)
     (in_bom yes) (on_board yes) (fields_autoplaced)
-    (property "Reference" "C69" (id 0) (at 169.545 92.7099 0)
+    (property "Reference" "C66" (id 0) (at 169.545 92.7099 0)
       (effects (font (size 1.27 1.27)) (justify left))
     )
@@
     (pin "2")
   )
-  (symbol (lib_id "power:+5V") (at 125.73 72.39 0)
+  (symbol (lib_id "power:+5V") (at 125.73 72.39 0) (unit 1)
     (in_bom yes) (on_board yes) (fields_autoplaced)
-    (property "Reference" "#PWR069" (id 0) (at 125.73 76.2 0)
+    (property "Reference" "#PWR064" (id 0) (at 125.73 76.2 0)
       (effects (font (size 1.27 1.27)) hide)
     )
@@
     (pin "1")
   )
-  (symbol (lib_id "Device:C") (at 134.62 76.2 0)
+  (symbol (lib_id "Device:C") (at 134.62 76.2 0) (unit 1)
     (in_bom yes) (on_board yes) (fields_autoplaced)
-    (property "Reference" "C67" (id 0) (at 137.795 74.9299 0)
+    (property "Reference" "C64" (id 0) (at 137.795 74.9299 0)
       (effects (font (size 1.27 1.27)) (justify left))
     )
@@
     (pin "2")
   )
-  (symbol (lib_id "power:GND") (at 151.13 118.11 0)
+  (symbol (lib_id "power:GND") (at 151.13 118.11 0) (unit 1)
     (in_bom yes) (on_board yes) (fields_autoplaced)
-    (property "Reference" "#PWR072" (id 0) (at 151.13 124.46 0)
+    (property "Reference" "#PWR067" (id 0) (at 151.13 124.46 0)
       (effects (font (size 1.27 1.27)) hide)
     )
@@
     (pin "1")
   )
-  (symbol (lib_id "FP-Interface-Card:MAX5490GC01000+T") (at 151.13 101.6 0) (mirror y)
+  (symbol (lib_id "FP-Interface-Card:MAX5490GC01000+T") (at 151.13 101.6 0) (mirror y) (unit 1)
     (in_bom yes) (on_board yes) (fields_autoplaced)
-    (property "Reference" "RN3" (id 0) (at 156.21 107.9499 0)
+    (property "Reference" "RN2" (id 0) (at 156.21 107.9499 0)
       (effects (font (size 1.27 1.27)) (justify right))
     )
@@
     (pin "3")
   )
-  (symbol (lib_id "Device:C") (at 139.7 100.33 0)
+  (symbol (lib_id "Device:C") (at 139.7 100.33 0) (unit 1)
     (in_bom yes) (on_board yes)
-    (property "Reference" "C68" (id 0) (at 143.51 99.0599 0)
+    (property "Reference" "C65" (id 0) (at 143.51 99.0599 0)
       (effects (font (size 1.27 1.27)) (justify left))
     )
@@
     (pin "2")
   )
-  (symbol (lib_id "power:GND") (at 125.73 97.79 0)
+  (symbol (lib_id "power:GND") (at 125.73 97.79 0) (unit 1)
     (in_bom yes) (on_board yes) (fields_autoplaced)
-    (property "Reference" "#PWR070" (id 0) (at 125.73 104.14 0)
+    (property "Reference" "#PWR065" (id 0) (at 125.73 104.14 0)
       (effects (font (size 1.27 1.27)) hide)
     )
