File: Blank-Card-Default.kicad_sch (KiCad schematic)
At the start: 39 parts, among them J100 ZX62-AB-5PA(31), Q100 BC847BM3T5G, Q101 BC847BM3T5G, Q102 BC847BM3T5G, Q103 BC847BM3T5G, SW100 SW_Push_SPST, U100 AP2161W

Commit message: 1
Parts:
- renumbered C102 to C1, C109 to C10, C103 to C2, C100 to C3, C101 to C4, C104 to C5, C105 to C6, C106 to C7, C107 to C8, C108 to C9, D100 to D1, D101 to D2, D102 to D3, D103 to D4, H100 to H1, H101 to H2, H102 to H3, H103 to H4, J100 to J2, Q100 to Q5, Q101 to Q6, Q102 to Q7, Q103 to Q8, R100 to R13, R111 to R14, R101 to R15, R102 to R16, R103 to R17, R104 to R18, R105 to R19, R106 to R20, R107 to R21, R108 to R22, R109 to R23, R110 to R24, SW100 to SW1, U100 to U1, Z100 to Z1, Z101 to Z2

Commit message: majority of routing completed
Parts:
- renumbered C3 to C10, C4 to C11, C1 to C12, C2 to C13, C7 to C4, C8 to C5, C9 to C6, C10 to C7, C5 to C8, C6 to C9, D1 to D2, D2 to D3, D3 to D4, D4 to D5, J2 to J3, Q5 to Q1, Q6 to Q2, Q7 to Q3, Q8 to Q4, R14 to R10, R22 to R11, R18 to R12, R23 to R14, R19 to R15, R20 to R4, R15 to R5, R24 to R6, R16 to R7, R21 to R8, R17 to R9, U1 to U2
Changed lines of the file:
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@@
   (symbol (lib_id "Device:R_US") (at 176.53 63.5 0) (unit 1)
     (in_bom yes) (on_board yes)
-    (property "Reference" "R14" (id 0) (at 178.2572 62.3316 0)
+    (property "Reference" "R10" (id 0) (at 178.2572 62.3316 0)
       (effects (font (size 1.27 1.27)) (justify left))
     )
@@
   (symbol (lib_id "Connector:USB_B_Micro") (at 100.33 52.07 0) (unit 1)
     (in_bom yes) (on_board yes)
-    (property "Reference" "J2" (id 0) (at 101.7778 40.2082 0))
+    (property "Reference" "J3" (id 0) (at 101.7778 40.2082 0))
     (property "Value" "ZX62-AB-5PA(31)" (id 1) (at 101.7778 42.5196 0))
     (property "Footprint" "SLI-Backplane-Blank-Card-KiCad:ZX62-AB-5PA(31)" (id 2) (at 104.14 53.34 0)
@@
   (symbol (lib_id "Device:R_US") (at 90.17 68.58 0) (unit 1)
     (in_bom yes) (on_board yes)
-    (property "Reference" "R15" (id 0) (at 91.8972 67.4116 0)
+    (property "Reference" "R5" (id 0) (at 91.8972 67.4116 0)
       (effects (font (size 1.27 1.27)) (justify left))
     )
@@
   (symbol (lib_id "Device:C") (at 80.01 68.58 0) (unit 1)
     (in_bom yes) (on_board yes)
-    (property "Reference" "C6" (id 0) (at 82.931 67.4116 0)
+    (property "Reference" "C9" (id 0) (at 82.931 67.4116 0)
       (effects (font (size 1.27 1.27)) (justify left))
     )
@@
   (symbol (lib_id "Device:C") (at 68.58 68.58 0) (unit 1)
     (in_bom yes) (on_board yes)
-    (property "Reference" "C5" (id 0) (at 71.501 67.4116 0)
+    (property "Reference" "C8" (id 0) (at 71.501 67.4116 0)
       (effects (font (size 1.27 1.27)) (justify left))
     )
@@
   (symbol (lib_id "Power_Management:AP2161W") (at 185.42 49.53 0) (unit 1)
     (in_bom yes) (on_board yes)
-    (property "Reference" "U1" (id 0) (at 185.42 40.2082 0))
+    (property "Reference" "U2" (id 0) (at 185.42 40.2082 0))
     (property "Value" "AP2161W" (id 1) (at 185.42 42.5196 0))
     (property "Footprint" "Package_TO_SOT_SMD:SOT-23-5" (id 2) (at 185.42 59.69 0)
@@
   (symbol (lib_id "Device:C") (at 240.03 60.96 0) (unit 1)
     (in_bom yes) (on_board yes)
-    (property "Reference" "C1" (id 0) (at 242.951 59.7916 0)
+    (property "Reference" "C12" (id 0) (at 242.951 59.7916 0)
       (effects (font (size 1.27 1.27)) (justify left))
     )
@@
   (symbol (lib_id "Device:R_US") (at 102.87 99.06 0) (unit 1)
     (in_bom yes) (on_board yes)
-    (property "Reference" "R16" (id 0) (at 104.5972 97.8916 0)
+    (property "Reference" "R7" (id 0) (at 104.5972 97.8916 0)
       (effects (font (size 1.27 1.27)) (justify left))
     )
@@
   (symbol (lib_id "Device:D") (at 102.87 109.22 90) (unit 1)
     (in_bom yes) (on_board yes)
-    (property "Reference" "D1" (id 0) (at 104.902 108.0516 90)
+    (property "Reference" "D2" (id 0) (at 104.902 108.0516 90)
       (effects (font (size 1.27 1.27)) (justify right))
     )
@@
   (symbol (lib_id "Device:Q_NPN_BEC") (at 100.33 120.65 0) (unit 1)
     (in_bom yes) (on_board yes)
-    (property "Reference" "Q5" (id 0) (at 105.1814 119.4816 0)
+    (property "Reference" "Q1" (id 0) (at 105.1814 119.4816 0)
       (effects (font (size 1.27 1.27)) (justify left))
     )
@@
   (symbol (lib_id "Device:R_US") (at 88.9 120.65 270) (unit 1)
     (in_bom yes) (on_board yes)
-    (property "Reference" "R20" (id 0) (at 88.9 115.443 90))
+    (property "Reference" "R4" (id 0) (at 88.9 115.443 90))
     (property "Value" "1.5k" (id 1) (at 88.9 117.7544 90))
     (property "Footprint" "Resistor_SMD:R_0402_1005Metric" (id 2) (at 88.646 121.666 90)
@@
   (symbol (lib_id "Device:R_US") (at 151.13 99.06 0) (unit 1)
     (in_bom yes) (on_board yes)
-    (property "Reference" "R17" (id 0) (at 152.8572 97.8916 0)
+    (property "Reference" "R9" (id 0) (at 152.8572 97.8916 0)
       (effects (font (size 1.27 1.27)) (justify left))
     )
@@
   (symbol (lib_id "Device:D") (at 151.13 109.22 90) (unit 1)
     (in_bom yes) (on_board yes)
-    (property "Reference" "D2" (id 0) (at 153.162 108.0516 90)
+    (property "Reference" "D3" (id 0) (at 153.162 108.0516 90)
       (effects (font (size 1.27 1.27)) (justify right))
     )
@@
   (symbol (lib_id "Device:R_US") (at 137.16 120.65 270) (unit 1)
     (in_bom yes) (on_board yes)
-    (property "Reference" "R21" (id 0) (at 137.16 115.443 90))
+    (property "Reference" "R8" (id 0) (at 137.16 115.443 90))
     (property "Value" "1.5k" (id 1) (at 137.16 117.7544 90))
     (property "Footprint" "Resistor_SMD:R_0402_1005Metric" (id 2) (at 136.906 121.666 90)
@@
   (symbol (lib_id "Device:R_US") (at 199.39 99.06 0) (unit 1)
     (in_bom yes) (on_board yes)
-    (property "Reference" "R18" (id 0) (at 201.1172 97.8916 0)
+    (property "Reference" "R12" (id 0) (at 201.1172 97.8916 0)
       (effects (font (size 1.27 1.27)) (justify left))
     )
@@
   (symbol (lib_id "Device:D") (at 199.39 109.22 90) (unit 1)
     (in_bom yes) (on_board yes)
-    (property "Reference" "D3" (id 0) (at 201.422 108.0516 90)
+    (property "Reference" "D4" (id 0) (at 201.422 108.0516 90)
       (effects (font (size 1.27 1.27)) (justify right))
     )
@@
   (symbol (lib_id "Device:R_US") (at 185.42 120.65 270) (unit 1)
     (in_bom yes) (on_board yes)
-    (property "Reference" "R22" (id 0) (at 185.42 115.443 90))
+    (property "Reference" "R11" (id 0) (at 185.42 115.443 90))
     (property "Value" "1.5k" (id 1) (at 185.42 117.7544 90))
     (property "Footprint" "Resistor_SMD:R_0402_1005Metric" (id 2) (at 185.166 121.666 90)
@@
   (symbol (lib_id "Device:R_US") (at 248.92 99.06 0) (unit 1)
     (in_bom yes) (on_board yes)
-    (property "Reference" "R19" (id 0) (at 250.6472 97.8916 0)
+    (property "Reference" "R15" (id 0) (at 250.6472 97.8916 0)
       (effects (font (size 1.27 1.27)) (justify left))
     )
@@
   (symbol (lib_id "Device:D") (at 248.92 109.22 90) (unit 1)
     (in_bom yes) (on_board yes)
-    (property "Reference" "D4" (id 0) (at 250.952 108.0516 90)
+    (property "Reference" "D5" (id 0) (at 250.952 108.0516 90)
       (effects (font (size 1.27 1.27)) (justify right))
     )
@@
   (symbol (lib_id "Device:R_US") (at 234.95 120.65 270) (unit 1)
     (in_bom yes) (on_board yes)
-    (property "Reference" "R23" (id 0) (at 234.95 115.443 90))
+    (property "Reference" "R14" (id 0) (at 234.95 115.443 90))
     (property "Value" "1.5k" (id 1) (at 234.95 117.7544 90))
     (property "Footprint" "Resistor_SMD:R_0402_1005Metric" (id 2) (at 234.696 121.666 90)
@@
   (symbol (lib_id "Device:Q_NPN_BEC") (at 148.59 120.65 0) (unit 1)
     (in_bom yes) (on_board yes)
-    (property "Reference" "Q6" (id 0) (at 153.4414 119.4816 0)
+    (property "Reference" "Q2" (id 0) (at 153.4414 119.4816 0)
       (effects (font (size 1.27 1.27)) (justify left))
     )
@@
   (symbol (lib_id "Device:Q_NPN_BEC") (at 196.85 120.65 0) (unit 1)
     (in_bom yes) (on_board yes)
-    (property "Reference" "Q7" (id 0) (at 201.7014 119.4816 0)
+    (property "Reference" "Q3" (id 0) (at 201.7014 119.4816 0)
       (effects (font (size 1.27 1.27)) (justify left))
     )
@@
   (symbol (lib_id "Device:Q_NPN_BEC") (at 246.38 120.65 0) (unit 1)
     (in_bom yes) (on_board yes)
-    (property "Reference" "Q8" (id 0) (at 251.2314 119.4816 0)
+    (property "Reference" "Q4" (id 0) (at 251.2314 119.4816 0)
       (effects (font (size 1.27 1.27)) (justify left))
     )
@@
   (symbol (lib_id "Device:C") (at 252.73 60.96 0) (unit 1)
     (in_bom yes) (on_board yes)
-    (property "Reference" "C2" (id 0) (at 255.651 59.7916 0)
+    (property "Reference" "C13" (id 0) (at 255.651 59.7916 0)
       (effects (font (size 1.27 1.27)) (justify left))
     )
@@
   (symbol (lib_id "Device:R_US") (at 100.33 168.91 0) (unit 1)
     (in_bom yes) (on_board yes)
-    (property "Reference" "R24" (id 0) (at 102.0572 167.7416 0)
+    (property "Reference" "R6" (id 0) (at 102.0572 167.7416 0)
       (effects (font (size 1.27 1.27)) (justify left))
     )
@@
   (symbol (lib_id "Device:C") (at 41.91 101.6 270) (unit 1)
     (in_bom yes) (on_board yes)
-    (property "Reference" "C7" (id 0) (at 41.91 95.1992 90))
+    (property "Reference" "C4" (id 0) (at 41.91 95.1992 90))
     (property "Value" "0.1uF" (id 1) (at 41.91 97.5106 90))
     (property "Footprint" "Capacitor_SMD:C_0402_1005Metric" (id 2) (at 38.1 102.5652 0)
@@
   (symbol (lib_id "Device:C") (at 41.91 111.76 270) (unit 1)
     (in_bom yes) (on_board yes)
-    (property "Reference" "C8" (id 0) (at 41.91 105.3592 90))
+    (property "Reference" "C5" (id 0) (at 41.91 105.3592 90))
     (property "Value" "0.1uF" (id 1) (at 41.91 107.6706 90))
     (property "Footprint" "Capacitor_SMD:C_0402_1005Metric" (id 2) (at 38.1 112.7252 0)
@@
   (symbol (lib_id "Device:C") (at 41.91 121.92 270) (unit 1)
     (in_bom yes) (on_board yes)
-    (property "Reference" "C9" (id 0) (at 41.91 115.5192 90))
+    (property "Reference" "C6" (id 0) (at 41.91 115.5192 90))
     (property "Value" "0.1uF" (id 1) (at 41.91 117.8306 90))
     (property "Footprint" "Capacitor_SMD:C_0402_1005Metric" (id 2) (at 38.1 122.8852 0)
@@
   (symbol (lib_id "Device:C") (at 41.91 132.08 270) (unit 1)
     (in_bom yes) (on_board yes)
-    (property "Reference" "C10" (id 0) (at 41.91 125.6792 90))
+    (property "Reference" "C7" (id 0) (at 41.91 125.6792 90))
     (property "Value" "0.1uF" (id 1) (at 41.91 127.9906 90))
     (property "Footprint" "Capacitor_SMD:C_0402_1005Metric" (id 2) (at 38.1 133.0452 0)
@@
   (symbol (lib_id "Device:C") (at 154.94 63.5 0) (unit 1)
     (in_bom yes) (on_board yes)
-    (property "Reference" "C3" (id 0) (at 157.861 62.3316 0)
+    (property "Reference" "C10" (id 0) (at 157.861 62.3316 0)
       (effects (font (size 1.27 1.27)) (justify left))
     )
@@
   (symbol (lib_id "Device:C") (at 165.1 63.5 0) (unit 1)
     (in_bom yes) (on_board yes)
-    (property "Reference" "C4" (id 0) (at 168.021 62.3316 0)
-      (effects (font (size 1.27 1.27)) (justify left))
-    )
+    (property "Reference" "C11" (id 0) (at 168.021 62.3316 0)
+      (effects (font (size 1.27 1.27)) (justify left))
+    )

Commit message: design updates
Parts:
- H1: value MountingHole_Pad -> SLI-Backplane-Blank-Card-KiCad:125mil_hole
Changed lines of the file:
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@@
     (in_bom yes) (on_board yes)
     (property "Reference" "H1" (id 0) (at 29.1338 97.917 90))
-    (property "Value" "MountingHole_Pad" (id 1) (at 29.1338 97.8916 90)
+    (property "Value" "SLI-Backplane-Blank-Card-KiCad:125mil_hole" (id 1) (at 29.1338 97.8916 90)
       (effects (font (size 1.27 1.27)) hide)
     )
