File: Level_Shifter.kicad_sch (KiCad schematic)
At the start: 6 parts, among them Q9 Q_NMOS_GSD

Commit message: 1
Parts:
- renumbered Q9 to Q?, R67 to R?, R66 to R?, R65 to R?, TP20 to TP?, TP19 to TP?
Changed lines of the file:
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@@
   (symbol (lib_id "Device:R_US") (at 154.94 99.06 0)
     (in_bom yes) (on_board yes) (fields_autoplaced)
-    (property "Reference" "R67" (id 0) (at 157.48 97.7899 0)
+    (property "Reference" "R?" (id 0) (at 157.48 97.7899 0)
       (effects (font (size 1.27 1.27)) (justify left))
     )
@@
   (symbol (lib_id "Connector:TestPoint") (at 165.735 104.14 0)
     (in_bom yes) (on_board yes) (fields_autoplaced)
-    (property "Reference" "TP20" (id 0) (at 168.275 99.5679 0)
+    (property "Reference" "TP?" (id 0) (at 168.275 99.5679 0)
       (effects (font (size 1.27 1.27)) (justify left))
     )
@@
   (symbol (lib_id "Device:R_US") (at 142.24 110.49 90)
     (in_bom yes) (on_board yes)
-    (property "Reference" "R66" (id 0) (at 142.24 113.03 90))
+    (property "Reference" "R?" (id 0) (at 142.24 113.03 90))
     (property "Value" "DNP" (id 1) (at 142.24 115.57 90))
     (property "Footprint" "Resistor_SMD:R_0603_1608Metric" (id 2) (at 142.494 109.474 90)
@@
   (symbol (lib_id "Connector:TestPoint") (at 119.38 104.14 0)
     (in_bom yes) (on_board yes) (fields_autoplaced)
-    (property "Reference" "TP19" (id 0) (at 121.92 99.5679 0)
+    (property "Reference" "TP?" (id 0) (at 121.92 99.5679 0)
       (effects (font (size 1.27 1.27)) (justify left))
     )
@@
   (symbol (lib_id "Device:R_US") (at 129.54 99.06 0)
     (in_bom yes) (on_board yes) (fields_autoplaced)
-    (property "Reference" "R65" (id 0) (at 132.08 97.7899 0)
+    (property "Reference" "R?" (id 0) (at 132.08 97.7899 0)
       (effects (font (size 1.27 1.27)) (justify left))
     )
@@
   (symbol (lib_id "Device:Q_NMOS_GSD") (at 142.24 101.6 90) (mirror x)
     (in_bom yes) (on_board yes)
-    (property "Reference" "Q9" (id 0) (at 139.7 99.06 90))
+    (property "Reference" "Q?" (id 0) (at 139.7 99.06 90))
     (property "Value" "Q_NMOS_GSD" (id 1) (at 142.24 107.95 90)
       (effects (font (size 1.27 1.27)) hide)

Commit message: design updates
Parts:
- Q27: renamed from Q?; value Q_NMOS_GSD -> BSS138
- TP40, TP41: renamed from TP?; footprint TestPoint:TestPoint_Pad_2.5x2.5mm -> TestPoint:TestPoint_Pad_D1.0mm
- gave numbers to parts that had none: 3
Changed lines of the file:
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@@
     (effects (font (size 1.27 1.27)) (justify right))
   )
-  (symbol (lib_id "Device:R_US") (at 154.94 99.06 0)
+  (symbol (lib_id "Device:R_US") (at 154.94 99.06 0) (unit 1)
     (in_bom yes) (on_board yes) (fields_autoplaced)
-    (property "Reference" "R?" (id 0) (at 157.48 97.7899 0)
+    (property "Reference" "R119" (id 0) (at 157.48 97.7899 0)
       (effects (font (size 1.27 1.27)) (justify left))
     )
@@
     (pin "2")
   )
-  (symbol (lib_id "Connector:TestPoint") (at 165.735 104.14 0)
+  (symbol (lib_id "Connector:TestPoint") (at 165.735 104.14 0) (unit 1)
     (in_bom yes) (on_board yes) (fields_autoplaced)
-    (property "Reference" "TP?" (id 0) (at 168.275 99.5679 0)
+    (property "Reference" "TP41" (id 0) (at 168.275 99.5679 0)
       (effects (font (size 1.27 1.27)) (justify left))
     )
@@
       (effects (font (size 1.27 1.27)) (justify left) hide)
     )
-    (property "Footprint" "TestPoint:TestPoint_Pad_2.5x2.5mm" (id 2) (at 170.815 104.14 0)
+    (property "Footprint" "TestPoint:TestPoint_Pad_D1.0mm" (id 2) (at 170.815 104.14 0)
       (effects (font (size 1.27 1.27)) hide)
     )
@@
     (pin "1")
   )
-  (symbol (lib_id "Device:R_US") (at 142.24 110.49 90)
+  (symbol (lib_id "Device:R_US") (at 142.24 110.49 90) (unit 1)
     (in_bom yes) (on_board yes)
-    (property "Reference" "R?" (id 0) (at 142.24 113.03 90))
+    (property "Reference" "R118" (id 0) (at 142.24 113.03 90))
     (property "Value" "DNP" (id 1) (at 142.24 115.57 90))
     (property "Footprint" "Resistor_SMD:R_0603_1608Metric" (id 2) (at 142.494 109.474 90)
@@
     (pin "2")
   )
-  (symbol (lib_id "Connector:TestPoint") (at 119.38 104.14 0)
+  (symbol (lib_id "Connector:TestPoint") (at 119.38 104.14 0) (unit 1)
     (in_bom yes) (on_board yes) (fields_autoplaced)
-    (property "Reference" "TP?" (id 0) (at 121.92 99.5679 0)
+    (property "Reference" "TP40" (id 0) (at 121.92 99.5679 0)
       (effects (font (size 1.27 1.27)) (justify left))
     )
@@
       (effects (font (size 1.27 1.27)) (justify left) hide)
     )
-    (property "Footprint" "TestPoint:TestPoint_Pad_2.5x2.5mm" (id 2) (at 124.46 104.14 0)
+    (property "Footprint" "TestPoint:TestPoint_Pad_D1.0mm" (id 2) (at 124.46 104.14 0)
       (effects (font (size 1.27 1.27)) hide)
     )
@@
     (pin "1")
   )
-  (symbol (lib_id "Device:R_US") (at 129.54 99.06 0)
+  (symbol (lib_id "Device:R_US") (at 129.54 99.06 0) (unit 1)
     (in_bom yes) (on_board yes) (fields_autoplaced)
-    (property "Reference" "R?" (id 0) (at 132.08 97.7899 0)
+    (property "Reference" "R117" (id 0) (at 132.08 97.7899 0)
       (effects (font (size 1.27 1.27)) (justify left))
     )
@@
     (pin "2")
   )
-  (symbol (lib_id "Device:Q_NMOS_GSD") (at 142.24 101.6 90) (mirror x)
+  (symbol (lib_id "Device:Q_NMOS_GSD") (at 142.24 101.6 90) (mirror x) (unit 1)
     (in_bom yes) (on_board yes)
-    (property "Reference" "Q?" (id 0) (at 139.7 99.06 90))
-    (property "Value" "Q_NMOS_GSD" (id 1) (at 142.24 107.95 90)
+    (property "Reference" "Q27" (id 0) (at 139.7 99.06 90))
+    (property "Value" "BSS138" (id 1) (at 142.24 107.95 90)
       (effects (font (size 1.27 1.27)) hide)
     )

Commit message: friday changes
Parts:
- renumbered Q27 to Q26, R117 to R114, R118 to R115, R119 to R116, TP40 to TP38, TP41 to TP39
Changed lines of the file:
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@@
   (symbol (lib_id "Device:R_US") (at 154.94 99.06 0) (unit 1)
     (in_bom yes) (on_board yes) (fields_autoplaced)
-    (property "Reference" "R119" (id 0) (at 157.48 97.7899 0)
+    (property "Reference" "R116" (id 0) (at 157.48 97.7899 0)
       (effects (font (size 1.27 1.27)) (justify left))
     )
@@
   (symbol (lib_id "Connector:TestPoint") (at 165.735 104.14 0) (unit 1)
     (in_bom yes) (on_board yes) (fields_autoplaced)
-    (property "Reference" "TP41" (id 0) (at 168.275 99.5679 0)
+    (property "Reference" "TP39" (id 0) (at 168.275 99.5679 0)
       (effects (font (size 1.27 1.27)) (justify left))
     )
@@
   (symbol (lib_id "Device:R_US") (at 142.24 110.49 90) (unit 1)
     (in_bom yes) (on_board yes)
-    (property "Reference" "R118" (id 0) (at 142.24 113.03 90))
+    (property "Reference" "R115" (id 0) (at 142.24 113.03 90))
     (property "Value" "DNP" (id 1) (at 142.24 115.57 90))
     (property "Footprint" "Resistor_SMD:R_0603_1608Metric" (id 2) (at 142.494 109.474 90)
@@
   (symbol (lib_id "Connector:TestPoint") (at 119.38 104.14 0) (unit 1)
     (in_bom yes) (on_board yes) (fields_autoplaced)
-    (property "Reference" "TP40" (id 0) (at 121.92 99.5679 0)
+    (property "Reference" "TP38" (id 0) (at 121.92 99.5679 0)
       (effects (font (size 1.27 1.27)) (justify left))
     )
@@
   (symbol (lib_id "Device:R_US") (at 129.54 99.06 0) (unit 1)
     (in_bom yes) (on_board yes) (fields_autoplaced)
-    (property "Reference" "R117" (id 0) (at 132.08 97.7899 0)
+    (property "Reference" "R114" (id 0) (at 132.08 97.7899 0)
       (effects (font (size 1.27 1.27)) (justify left))
     )
@@
   (symbol (lib_id "Device:Q_NMOS_GSD") (at 142.24 101.6 90) (mirror x) (unit 1)
     (in_bom yes) (on_board yes)
-    (property "Reference" "Q27" (id 0) (at 139.7 99.06 90))
+    (property "Reference" "Q26" (id 0) (at 139.7 99.06 90))
     (property "Value" "BSS138" (id 1) (at 142.24 107.95 90)
       (effects (font (size 1.27 1.27)) hide)
