File: pico.kicad_sch (KiCad schematic)
At the start: 8 parts

Commit message: friday changes
Parts:
- D8: renamed from D?; value SBR1A20T5-7 -> S1G; footprint Diode_SMD:D_SOD-523 -> Diode_SMD:D_SMA
- gave numbers to parts that had none: 7
Changed lines of the file:
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@@
   (symbol (lib_id "power:GND") (at 212.09 85.09 0) (unit 1)
     (in_bom yes) (on_board yes) (fields_autoplaced)
-    (property "Reference" "#PWR?" (id 0) (at 212.09 91.44 0)
+    (property "Reference" "#PWR0120" (id 0) (at 212.09 91.44 0)
       (effects (font (size 1.27 1.27)) hide)
     )
@@
   (symbol (lib_id "power:GND") (at 212.09 72.39 0) (unit 1)
     (in_bom yes) (on_board yes) (fields_autoplaced)
-    (property "Reference" "#PWR?" (id 0) (at 212.09 78.74 0)
+    (property "Reference" "#PWR0109" (id 0) (at 212.09 78.74 0)
       (effects (font (size 1.27 1.27)) hide)
     )
@@
   (symbol (lib_id "power:GND") (at 212.09 110.49 0) (unit 1)
     (in_bom yes) (on_board yes) (fields_autoplaced)
-    (property "Reference" "#PWR?" (id 0) (at 212.09 116.84 0)
+    (property "Reference" "#PWR0118" (id 0) (at 212.09 116.84 0)
       (effects (font (size 1.27 1.27)) hide)
     )
@@
   (symbol (lib_id "power:GND") (at 44.45 97.79 0) (mirror y) (unit 1)
     (in_bom yes) (on_board yes) (fields_autoplaced)
-    (property "Reference" "#PWR?" (id 0) (at 44.45 104.14 0)
+    (property "Reference" "#PWR0126" (id 0) (at 44.45 104.14 0)
       (effects (font (size 1.27 1.27)) hide)
     )
@@
   (symbol (lib_id "Device:R_US") (at 149.86 24.13 0) (unit 1)
     (in_bom yes) (on_board yes) (fields_autoplaced)
-    (property "Reference" "R?" (id 0) (at 152.4 22.8599 0)
+    (property "Reference" "R92" (id 0) (at 152.4 22.8599 0)
       (effects (font (size 1.27 1.27)) (justify left))
     )
@@
   (symbol (lib_id "Device:D") (at 160.02 64.77 0) (unit 1)
     (in_bom yes) (on_board yes) (fields_autoplaced)
-    (property "Reference" "D?" (id 0) (at 160.02 58.42 0))
-    (property "Value" "SBR1A20T5-7" (id 1) (at 160.02 60.96 0))
-    (property "Footprint" "Diode_SMD:D_SOD-523" (id 2) (at 160.02 64.77 0)
+    (property "Reference" "D8" (id 0) (at 160.02 58.42 0))
+    (property "Value" "S1G" (id 1) (at 160.02 60.96 0))
+    (property "Footprint" "Diode_SMD:D_SMA" (id 2) (at 160.02 64.77 0)
       (effects (font (size 1.27 1.27)) hide)
     )
@@
   (symbol (lib_id "power:GND") (at 212.09 97.79 0) (unit 1)
     (in_bom yes) (on_board yes) (fields_autoplaced)
-    (property "Reference" "#PWR?" (id 0) (at 212.09 104.14 0)
+    (property "Reference" "#PWR0115" (id 0) (at 212.09 104.14 0)
       (effects (font (size 1.27 1.27)) hide)
     )
@@
   (symbol (lib_id "power:GND") (at 149.86 45.72 0) (mirror y) (unit 1)
     (in_bom yes) (on_board yes)
-    (property "Reference" "#PWR?" (id 0) (at 149.86 52.07 0)
+    (property "Reference" "#PWR0114" (id 0) (at 149.86 52.07 0)
       (effects (font (size 1.27 1.27)) hide)
     )
@@
   (symbol (lib_id "power:GND") (at 44.45 85.09 0) (mirror y) (unit 1)
     (in_bom yes) (on_board yes) (fields_autoplaced)
-    (property "Reference" "#PWR?" (id 0) (at 44.45 91.44 0)
+    (property "Reference" "#PWR0125" (id 0) (at 44.45 91.44 0)
       (effects (font (size 1.27 1.27)) hide)
     )
@@
   (symbol (lib_id "power:GND") (at 44.45 72.39 0) (mirror y) (unit 1)
     (in_bom yes) (on_board yes) (fields_autoplaced)
-    (property "Reference" "#PWR?" (id 0) (at 44.45 78.74 0)
+    (property "Reference" "#PWR0129" (id 0) (at 44.45 78.74 0)
       (effects (font (size 1.27 1.27)) hide)
     )
@@
   (symbol (lib_id "Device:Q_NPN_BEC") (at 147.32 38.1 0) (unit 1)
     (in_bom yes) (on_board yes) (fields_autoplaced)
-    (property "Reference" "Q?" (id 0) (at 152.4 36.8299 0)
+    (property "Reference" "Q20" (id 0) (at 152.4 36.8299 0)
       (effects (font (size 1.27 1.27)) (justify left))
     )
@@
   (symbol (lib_id "Device:C") (at 191.77 63.5 0) (unit 1)
     (in_bom yes) (on_board yes) (fields_autoplaced)
-    (property "Reference" "C?" (id 0) (at 195.58 62.2299 0)
+    (property "Reference" "C72" (id 0) (at 195.58 62.2299 0)
       (effects (font (size 1.27 1.27)) (justify left))
     )
@@
   (symbol (lib_id "power:+5V") (at 139.7 20.32 0) (unit 1)
     (in_bom yes) (on_board yes) (fields_autoplaced)
-    (property "Reference" "#PWR?" (id 0) (at 139.7 24.13 0)
+    (property "Reference" "#PWR0108" (id 0) (at 139.7 24.13 0)
       (effects (font (size 1.27 1.27)) hide)
     )
@@
   (symbol (lib_id "power:GND") (at 128.27 127 0) (unit 1)
     (in_bom yes) (on_board yes) (fields_autoplaced)
-    (property "Reference" "#PWR?" (id 0) (at 128.27 133.35 0)
+    (property "Reference" "#PWR0123" (id 0) (at 128.27 133.35 0)
       (effects (font (size 1.27 1.27)) hide)
     )
@@
   (symbol (lib_id "Device:R_US") (at 128.27 41.91 0) (unit 1)
     (in_bom yes) (on_board yes) (fields_autoplaced)
-    (property "Reference" "R?" (id 0) (at 130.81 40.6399 0)
+    (property "Reference" "R90" (id 0) (at 130.81 40.6399 0)
       (effects (font (size 1.27 1.27)) (justify left))
     )
@@
   (symbol (lib_id "RPi_Pico:Pico") (at 128.27 88.9 0) (unit 1)
     (in_bom yes) (on_board yes) (fields_autoplaced)
-    (property "Reference" "U?" (id 0) (at 128.27 57.15 0))
+    (property "Reference" "U25" (id 0) (at 128.27 57.15 0))
     (property "Value" "Pico" (id 1) (at 128.27 59.69 0))
     (property "Footprint" "RPi_Pico:RPi_Pico_SMD_TH" (id 2) (at 128.27 88.9 90)
@@
   (symbol (lib_id "power:GND") (at 128.27 45.72 0) (mirror y) (unit 1)
     (in_bom yes) (on_board yes)
-    (property "Reference" "#PWR?" (id 0) (at 128.27 52.07 0)
+    (property "Reference" "#PWR0128" (id 0) (at 128.27 52.07 0)
       (effects (font (size 1.27 1.27)) hide)
     )
@@
   (symbol (lib_id "SLI-Backplane-Blank-Card-KiCad:IRF7404TRPBF") (at 162.56 27.94 0) (mirror x) (unit 1)
     (in_bom yes) (on_board yes) (fields_autoplaced)
-    (property "Reference" "Q?" (id 0) (at 168.91 26.6699 0)
+    (property "Reference" "Q21" (id 0) (at 168.91 26.6699 0)
       (effects (font (size 1.27 1.27)) (justify left))
     )
@@
   (symbol (lib_id "power:GND") (at 44.45 110.49 0) (mirror y) (unit 1)
     (in_bom yes) (on_board yes) (fields_autoplaced)
-    (property "Reference" "#PWR?" (id 0) (at 44.45 116.84 0)
+    (property "Reference" "#PWR0127" (id 0) (at 44.45 116.84 0)
       (effects (font (size 1.27 1.27)) hide)
     )
@@
   (symbol (lib_id "Device:R_US") (at 135.89 38.1 90) (unit 1)
     (in_bom yes) (on_board yes) (fields_autoplaced)
-    (property "Reference" "R?" (id 0) (at 135.89 31.75 90))
+    (property "Reference" "R91" (id 0) (at 135.89 31.75 90))
     (property "Value" "10k" (id 1) (at 135.89 34.29 90))
     (property "Footprint" "Resistor_SMD:R_0603_1608Metric" (id 2) (at 136.144 37.084 90)
