File: FP Interface Card.kicad_pcb (KiCad board)
At the start: 6 copper layers, 90.2 x 101.1 mm, 40 parts, among them J100 ZX62-AB-5PA(31), P1 Card Edge for HSEC8-160-01-S-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, Q100 BC847BM3T5G, Q101 BC847BM3T5G, Q102 BC847BM3T5G, Q103 BC847BM3T5G, SW100 SW_Push_SPST, U100 AP2161W

Commit message: 1
Connections:
- net /~BUS_RESET renamed /~{BUS_RESET}
- net /~USB_EN renamed /~{USB_EN}
- net /~USB_FLAG renamed /~{USB_FLAG}
Other:
- net class Default removed

Commit message: 1
Parts:
- added G***: LOGO, payload-interface-board:Sierra_Lobo_Logo, F.Cu at (18.4, -4.55)
- added J1: T2M-105-01-X-D-TH-DS, payload-interface-board:SAMTEC_T2M-105-01-X-D-TH-DS, F.Cu at (46.0, -9.50)
- added Q1: Q_NMOS_GSD, Package_TO_SOT_SMD:SOT-23, F.Cu at (36.5, -39.5)
- added Q2: Q_NMOS_GSD, Package_TO_SOT_SMD:SOT-23, F.Cu at (50.5, -39.5)
- added Q3: Q_NMOS_GSD, Package_TO_SOT_SMD:SOT-23, F.Cu at (43.5, -39.5)
- added Q4: Q_NMOS_GSD, Package_TO_SOT_SMD:SOT-23, F.Cu at (57.5, -39.5)
- added R1: 10k, Resistor_SMD:R_0603_1608Metric_Pad0.98x0.95mm_HandSolder, F.Cu at (35.5, -43.0)
- added R10: 10k, Resistor_SMD:R_0603_1608Metric_Pad0.98x0.95mm_HandSolder, F.Cu at (57.5, -35.5)
- added R11: 0, Resistor_SMD:R_0603_1608Metric_Pad0.98x0.95mm_HandSolder, F.Cu at (46.5, -39.5)
- added R12: 0, Resistor_SMD:R_0603_1608Metric_Pad0.98x0.95mm_HandSolder, F.Cu at (60.5, -39.5)
- added R2: 10k, Resistor_SMD:R_0603_1608Metric_Pad0.98x0.95mm_HandSolder, F.Cu at (36.5, -35.5)
- added R3: 10k, Resistor_SMD:R_0603_1608Metric_Pad0.98x0.95mm_HandSolder, F.Cu at (49.5, -43.0)
- added R4: 10k, Resistor_SMD:R_0603_1608Metric_Pad0.98x0.95mm_HandSolder, F.Cu at (50.5, -35.5)
- added R5: 0, Resistor_SMD:R_0603_1608Metric_Pad0.98x0.95mm_HandSolder, F.Cu at (39.5, -39.5)
- added R6: 0, Resistor_SMD:R_0603_1608Metric_Pad0.98x0.95mm_HandSolder, F.Cu at (53.5, -39.5)
- added R7: 10k, Resistor_SMD:R_0603_1608Metric_Pad0.98x0.95mm_HandSolder, F.Cu at (42.5, -43.0)
- added R8: 10k, Resistor_SMD:R_0603_1608Metric_Pad0.98x0.95mm_HandSolder, F.Cu at (43.5, -35.5)
- added R9: 10k, Resistor_SMD:R_0603_1608Metric_Pad0.98x0.95mm_HandSolder, F.Cu at (56.5, -43.0)
- added TP1: TestPoint, TestPoint:TestPoint_Pad_2.5x2.5mm, F.Cu at (43.5, -48.0)
- added TP2: TestPoint, TestPoint:TestPoint_Pad_2.5x2.5mm, F.Cu at (36.5, -48.0)
- added TP3: TestPoint, TestPoint:TestPoint_Pad_2.5x2.5mm, F.Cu at (43.5, -30.5)
- added TP4: TestPoint, TestPoint:TestPoint_Pad_2.5x2.5mm, F.Cu at (36.5, -30.5)
- added TP5: TestPoint, TestPoint:TestPoint_Pad_2.5x2.5mm, F.Cu at (50.5, -48.0)
- added TP6: TestPoint, TestPoint:TestPoint_Pad_2.5x2.5mm, F.Cu at (57.5, -48.0)
- added TP7: TestPoint, TestPoint:TestPoint_Pad_2.5x2.5mm, F.Cu at (50.5, -30.5)
- added TP8: TestPoint, TestPoint:TestPoint_Pad_2.5x2.5mm, F.Cu at (57.5, -30.5)
- renumbered C102 to C1, C109 to C10, C103 to C2, C100 to C3, C101 to C4, C104 to C5, C105 to C6, C106 to C7, C107 to C8, C108 to C9, D100 to D1, D101 to D2, D102 to D3, D103 to D4, H100 to H1, H101 to H2, H102 to H3, H103 to H4, J100 to J2, Q100 to Q5, Q101 to Q6, Q102 to Q7, Q103 to Q8, R100 to R13, R111 to R14, R101 to R15, R102 to R16, R103 to R17, R104 to R18, R105 to R19, R106 to R20, R107 to R21, R108 to R22, R109 to R23, R110 to R24, SW100 to SW1, U100 to U1, Z100 to Z1, Z101 to Z2
Connections:
- net /SCK0 renamed /H1-21
- net /SDI0 renamed /H1-22
- net /SDO0 renamed /H1-23
- net /VCC_sys renamed +3V3
- C1 pad 2: /Blank-Card-Default/GND -> GND
- C10 pad 1: /Blank-Card-Default/GND -> GND
- C2 pad 2: /Blank-Card-Default/GND -> GND
- C3 pad 2: /Blank-Card-Default/GND -> GND
- C4 pad 2: /Blank-Card-Default/GND -> GND
- C5 pad 2: /Blank-Card-Default/GND -> GND
- C6 pad 2: /Blank-Card-Default/GND -> GND
- C7 pad 1: /Blank-Card-Default/GND -> GND
- C8 pad 1: /Blank-Card-Default/GND -> GND
- C9 pad 1: /Blank-Card-Default/GND -> GND
- J2 pad 4: Net-(J100-Pad4) -> unconnected-(J2-Pad4)
- J2 pad 5: /Blank-Card-Default/GND -> GND
- P1 pad 103: /GND -> GND
- P1 pad 104: /GND -> GND
- P1 pad 45: /URx0 -> /H1-19
- P1 pad 46: /UTx0 -> /H1-20
- P1 pad 59: /H2-25 -> +5V
- P1 pad 60: /H2-26 -> +5V
- P1 pad 67: /GND -> GND
- P1 pad 68: /GND -> GND
- P1 pad 72: /GND -> GND
- Q5 pad 2: /Blank-Card-Default/GND -> GND
- Q6 pad 2: /Blank-Card-Default/GND -> GND
- Q7 pad 2: /Blank-Card-Default/GND -> GND
- Q8 pad 2: /Blank-Card-Default/GND -> GND
- R14 pad 2: /Blank-Card-Default/GND -> GND
- R15 pad 2: /Blank-Card-Default/GND -> GND
- R20 pad 2: /USB_D+ -> /H1-19
- R21 pad 2: /USB_D- -> /H1-20
- R23 pad 2: /ORG_LED -> /H2-6
- SW1 pad 2: /GND -> GND
- U1 pad 2: /Blank-Card-Default/GND -> GND
- Z1 pad 2: /Blank-Card-Default/GND -> GND
- Z2 pad 2: /Blank-Card-Default/GND -> GND
Routing:
- net /H1-20: track 0.00 -> 98.0 mm, vias 0 -> 3
- net /H1-19: track 0.00 -> 97.2 mm, vias 0 -> 4
- net /H2-6: track 0.00 -> 80.6 mm, vias 0 -> 1
- net /5V_USB: track 22.5 -> 103.0 mm, vias 3 -> 7
- net GND: track 0.00 -> 70.9 mm, vias 0 -> 14
- net /H1-6: track 0.00 -> 68.7 mm, vias 0 -> 2
- net /RESET: track 0.00 -> 37.6 mm, vias 0 -> 1
- net /RXD: track 0.00 -> 37.3 mm, vias 0 -> 1
- net /Blank-Card-Default/GND: track 34.5 -> 0.00 mm, vias 5 -> 0
- net /SERVO_PWR_CTRL: track 0.00 -> 33.6 mm
- net /TXD: track 0.00 -> 32.4 mm
- net +3V3: track 0.00 -> 26.9 mm, vias 0 -> 5
- net /GND: track 20.9 -> 0.00 mm, vias 3 -> 0
- net +5V: track 0.00 -> 11.5 mm, vias 0 -> 5
- net /USB_D-: track 4.30 -> 1.82 mm, vias 1 -> 0
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- added copper zone on B.Cu, net +3V3
- added copper zone on In1.Cu, net +5V
- added copper zone on In2.Cu, net GND
Other:
- copper layers 6 -> 4
- board text added: "3.3V IO"
- board text added: "5V IO"
- board text added: "Foras Promineo Payload Interface Board C.Hillis 2/21"
- board text added: "PAYLOAD_RX"
- board text added: "PAYLOAD_TX"
- board text added: "RESET"
- board text added: "SERVO_PWR_CTRL"

Commit message: generated fab files
Connections:
- J1 pad 10: Net-(J1-Pad10) -> +5V
- J1 pad 8: Net-(J1-Pad10) -> +5V
- J1 pad 9: Net-(J1-Pad10) -> +5V
Routing:
- net /CHS: track 50.3 -> 48.1 mm
- net GND: track 70.9 -> 69.8 mm
- net /SW_NO: track 4.34 -> 3.29 mm
- net /5V_USB: track 103.0 -> 102.2 mm, vias 7 -> 6
- net /RESET: track 37.6 -> 37.5 mm, vias 1 -> 0
- net /RXD: vias 1 -> 0

Commit message: majority of routing completed
Parts:
- removed the Q1 at (36.5, -39.5)
- removed the Q2 at (50.5, -39.5)
- removed the Q3 at (43.5, -39.5)
- removed the Q4 at (57.5, -39.5)
- removed the R10 at (57.5, -35.5)
- removed the R11 at (46.5, -39.5)
- removed the R12 at (60.5, -39.5)
- removed the R4 at (50.5, -35.5)
- removed the R5 at (39.5, -39.5)
- removed the R6 at (53.5, -39.5)
- removed the R7 at (42.5, -43.0)
- removed the R8 at (43.5, -35.5)
- removed the R9 at (56.5, -43.0)
- removed TP1, TP2, TP3, TP4, TP5, TP6, TP7, TP8: TestPoint, TestPoint:TestPoint_Pad_2.5x2.5mm
- added C1: 0.1uF, Capacitor_SMD:C_0603_1608Metric, F.Cu at (53.8, -32.4)
- added C14: 2.2uF, Capacitor_SMD:C_0805_2012Metric, F.Cu at (7.90, -39.6)
- added C15: 2.2uF, Capacitor_SMD:C_0805_2012Metric, F.Cu at (7.90, -49.5)
- added C16: 0.1uF, Capacitor_SMD:C_0603_1608Metric, F.Cu at (21.6, -54.6)
- added C17: 0.1uF, Capacitor_SMD:C_0603_1608Metric, F.Cu at (8.15, -37.6)
- added C18: 0.1uF, Capacitor_SMD:C_0603_1608Metric, F.Cu at (8.15, -47.5)
- added C19: 10nF, Capacitor_SMD:C_0603_1608Metric, F.Cu at (6.88, -34.0)
- added C2: 0.1uF, Capacitor_SMD:C_0603_1608Metric, F.Cu at (57.1, -31.1)
- added C20: 10nF, Capacitor_SMD:C_0603_1608Metric, F.Cu at (6.88, -43.9)
- added C21: 0.47uF, Capacitor_SMD:C_0603_1608Metric, F.Cu at (11.5, -37.6)
- added C22: 0.47uF, Capacitor_SMD:C_0603_1608Metric, F.Cu at (11.5, -47.5)
- added C23: 1uF, Capacitor_SMD:C_0603_1608Metric, F.Cu at (14.5, -38.4)
- added C24: 1uF, Capacitor_SMD:C_0603_1608Metric, F.Cu at (14.5, -48.3)
- added C25: 10uF, Capacitor_SMD:C_0805_2012Metric, F.Cu at (17.3, -37.8)
- added C26: 10uF, Capacitor_SMD:C_0805_2012Metric, F.Cu at (17.3, -47.8)
- added C27: 1uF, Capacitor_SMD:C_0603_1608Metric, F.Cu at (21.4, -37.1)
- added C28: 1uF, Capacitor_SMD:C_0603_1608Metric, F.Cu at (21.4, -47.0)
- added C29: 0.1uF, Capacitor_SMD:C_0603_1608Metric, F.Cu at (37.9, -54.9)
- added C3: 4.7uF, Capacitor_SMD:C_0805_2012Metric, F.Cu at (56.9, -29.4)
- added C30: 10uF, Capacitor_SMD:C_0805_2012Metric, F.Cu at (38.9, -48.3)
- added C31: 0.1uF, Capacitor_SMD:C_0603_1608Metric, F.Cu at (40.9, -48.5)
- added C32: 0.1uF, Capacitor_SMD:C_0603_1608Metric, F.Cu at (48.5, -37.8)
- added C33: 0.1uF, Capacitor_SMD:C_0603_1608Metric, F.Cu at (48.5, -39.4)
- added C34: 560pF, Capacitor_SMD:C_0603_1608Metric, F.Cu at (58.9, -53.3)
- added C35: 10uF, Capacitor_SMD:C_0805_2012Metric, F.Cu at (61.0, -63.5)
- added C36: 10uF, Capacitor_SMD:C_0805_2012Metric, F.Cu at (55.9, -59.9)
- added C37: 560pF, Capacitor_SMD:C_0603_1608Metric, F.Cu at (66.3, -57.1)
- added C38: 0.1uF, Capacitor_SMD:C_0603_1608Metric, F.Cu at (48.5, -23.1)
- added C39: 0.1uF, Capacitor_SMD:C_0603_1608Metric, F.Cu at (61.2, -61.5)
- added C40: 0.1uF, Capacitor_SMD:C_0603_1608Metric, F.Cu at (57.9, -59.7)
- added C41: 0.1uF, Capacitor_SMD:C_0603_1608Metric, F.Cu at (48.5, -24.6)
- added C42: 560pF, Capacitor_SMD:C_0603_1608Metric, F.Cu at (62.5, -53.3)
- added C43: 0.1uF, Capacitor_SMD:C_0603_1608Metric, F.Cu at (73.4, -55.4)
- added C44: 0.1uF, Capacitor_SMD:C_0603_1608Metric, F.Cu at (73.4, -60.5)
- added C45: 2.2uF, Capacitor_SMD:C_0805_2012Metric, F.Cu at (56.9, -55.1)
- added C46: 2.2uF, Capacitor_SMD:C_0805_2012Metric, F.Cu at (56.9, -57.1)
- added C47: 10nF, Capacitor_SMD:C_0603_1608Metric, F.Cu at (21.6, -73.7)
- added C48: 10nF, Capacitor_SMD:C_0603_1608Metric, F.Cu at (21.6, -78.2)
- added C49: 0.1uF, Capacitor_SMD:C_0603_1608Metric, F.Cu at (53.8, -42.5)
- added C50: 0.1uF, Capacitor_SMD:C_0603_1608Metric, F.Cu at (57.1, -41.4)
- added C51: 4.7uF, Capacitor_SMD:C_0805_2012Metric, F.Cu at (56.9, -39.6)
- added C52: 1uF, Capacitor_SMD:C_0603_1608Metric, F.Cu at (74.9, -47.0)
- added C53: 0.1uF, Capacitor_SMD:C_0603_1608Metric, F.Cu at (73.4, -47.0)
- added C54: 1uF, Capacitor_SMD:C_0603_1608Metric, F.Cu at (74.9, -36.8)
- added C55: 0.1uF, Capacitor_SMD:C_0603_1608Metric, F.Cu at (73.4, -36.8)
- added C56: 0.1uF, Capacitor_SMD:C_0603_1608Metric, F.Cu at (53.8, -22.1)
- added C57: 0.1uF, Capacitor_SMD:C_0603_1608Metric, F.Cu at (57.1, -20.8)
- added C58: 4.7uF, Capacitor_SMD:C_0805_2012Metric, F.Cu at (56.9, -18.8)
- added C59: 1uF, Capacitor_SMD:C_0603_1608Metric, F.Cu at (74.9, -26.4)
- added C60: 0.1uF, Capacitor_SMD:C_0603_1608Metric, F.Cu at (73.4, -26.4)
- added C61: 0.1uF, Capacitor_SMD:C_0603_1608Metric, F.Cu at (34.0, -31.5)
- added C62: 0.1uF, Capacitor_SMD:C_0603_1608Metric, F.Cu at (30.5, -37.6)
- added C63: 0.1uF, Capacitor_SMD:C_0603_1608Metric, F.Cu at (34.0, -37.6)
- added C64: 0.1uF, Capacitor_SMD:C_0603_1608Metric, F.Cu at (34.0, -39.1)
- added C65: 0.1uF, Capacitor_SMD:C_0603_1608Metric, F.Cu at (30.5, -45.2)
- added C66: 0.1uF, Capacitor_SMD:C_0603_1608Metric, F.Cu at (34.0, -45.2)
- added C67: 0.1uF, Capacitor_SMD:C_0603_1608Metric, F.Cu at (34.1, -21.1)
- added C68: 0.1uF, Capacitor_SMD:C_0603_1608Metric, F.Cu at (30.5, -27.4)
- added C69: 0.1uF, Capacitor_SMD:C_0603_1608Metric, F.Cu at (34.1, -27.4)
- added C70: 10nF, Capacitor_SMD:C_0603_1608Metric, F.Cu at (21.6, -64.9)
- added C71: 10nF, Capacitor_SMD:C_0603_1608Metric, F.Cu at (21.6, -69.1)
- added D1: TPSMF4L6.0A, Diode_SMD:D_SOD-123F, F.Cu at (61.2, -33.0)
- added D6: TPSMF4L6.0A, Diode_SMD:D_SOD-123F, F.Cu at (61.2, -43.2)
- added D7: TPSMF4L6.0A, Diode_SMD:D_SOD-123F, F.Cu at (61.2, -22.9)
- added J2: T2M-105-01-X-D-TH-DS, payload-interface-board:SAMTEC_T2M-105-01-X-D-TH-DS, B.Cu at (83.8, -24.1)
- added Q10: Q_NMOS_GSD, Package_TO_SOT_SMD:SOT-23, F.Cu at (18.3, -4.32)
- added Q11: Q_NMOS_GSD, Package_TO_SOT_SMD:SOT-23, F.Cu at (18.3, -10.2)
- added Q12: Q_NMOS_GSD, Package_TO_SOT_SMD:SOT-23, F.Cu at (18.3, -16.0)
- added Q13: BSS138DWQ-7, Package_TO_SOT_SMD:SOT-363_SC-70-6, F.Cu at (19.6, -64.9)
- added Q14: MMDT5551-7-F, Package_TO_SOT_SMD:SOT-363_SC-70-6, F.Cu at (14.0, -64.9)
- added Q15: BSS138DWQ-7, Package_TO_SOT_SMD:SOT-363_SC-70-6, F.Cu at (19.6, -69.1)
- added Q16: MMDT5551-7-F, Package_TO_SOT_SMD:SOT-363_SC-70-6, F.Cu at (14.0, -69.1)
- added Q5: BSS138DWQ-7, Package_TO_SOT_SMD:SOT-363_SC-70-6, F.Cu at (19.6, -73.7)
- added Q6: MMDT5551-7-F, Package_TO_SOT_SMD:SOT-363_SC-70-6, F.Cu at (14.0, -73.7)
- added Q7: BSS138DWQ-7, Package_TO_SOT_SMD:SOT-363_SC-70-6, F.Cu at (19.6, -78.2)
- added Q8: MMDT5551-7-F, Package_TO_SOT_SMD:SOT-363_SC-70-6, F.Cu at (14.0, -78.2)
- added Q9: Q_NMOS_GSD, Package_TO_SOT_SMD:SOT-23, F.Cu at (18.0, -22.1)
- added R16: 100k, Resistor_SMD:R_0603_1608Metric, F.Cu at (7.62, -54.6)
- added R17: 100k, Resistor_SMD:R_0603_1608Metric, F.Cu at (7.62, -58.7)
- added R18: 100k, Resistor_SMD:R_0603_1608Metric, F.Cu at (9.40, -58.7)
- added R19: 10k, Resistor_SMD:R_0603_1608Metric, F.Cu at (13.0, -58.7)
- added R20: 100k, Resistor_SMD:R_0603_1608Metric, F.Cu at (21.6, -58.7)
- added R21: 10k, Resistor_SMD:R_0603_1608Metric, F.Cu at (11.2, -58.7)
- added R22: 100k, Resistor_SMD:R_0603_1608Metric, F.Cu at (13.0, -54.6)
- added R23: 10k, Resistor_SMD:R_0603_1608Metric, F.Cu at (9.40, -54.6)
- added R24: 10k, Resistor_SMD:R_0603_1608Metric, F.Cu at (11.2, -54.6)
- added R25: 100k, Resistor_SMD:R_0603_1608Metric, F.Cu at (48.0, -57.1)
- added R26: 51, Resistor_SMD:R_0603_1608Metric, F.Cu at (33.0, -58.4)
- added R27: 51, Resistor_SMD:R_0603_1608Metric, F.Cu at (33.0, -56.9)
- added R28: 51, Resistor_SMD:R_0603_1608Metric, F.Cu at (47.5, -52.3)
- added R29: 51, Resistor_SMD:R_0603_1608Metric, F.Cu at (46.0, -52.3)
- added R30: 100, Resistor_SMD:R_0603_1608Metric, F.Cu at (44.5, -52.3)
- added R31: 100, Resistor_SMD:R_0603_1608Metric, F.Cu at (42.9, -52.3)
- added R32: 200mR, Resistor_SMD:R_0805_2012Metric, F.Cu at (63.8, -43.7)
- added R33: 200mR, Resistor_SMD:R_0805_2012Metric, F.Cu at (64.0, -33.5)
- added R34: 91mR, Resistor_SMD:R_0805_2012Metric, F.Cu at (63.8, -23.4)
- added R35: 100k, Resistor_SMD:R_0603_1608Metric, F.Cu at (39.9, -33.8)
- added R36: 33, Resistor_SMD:R_0603_1608Metric, F.Cu at (58.9, -51.8)
- added R37: 33, Resistor_SMD:R_0603_1608Metric, F.Cu at (67.8, -57.1)
- added R38: 33, Resistor_SMD:R_0603_1608Metric, F.Cu at (62.5, -51.8)
- added R39: 100k, Resistor_SMD:R_0603_1608Metric, F.Cu at (40.1, -19.3)
- added R40: 100k, Resistor_SMD:R_0603_1608Metric, F.Cu at (43.4, -19.3)
- added R41: 100, Resistor_SMD:R_0603_1608Metric, F.Cu at (56.6, -62.7)
- added R42: 100k, Resistor_SMD:R_0603_1608Metric, F.Cu at (39.9, -29.2)
- added R43: 100, Resistor_SMD:R_0603_1608Metric, F.Cu at (67.1, -54.1)
- added R44: 100, Resistor_SMD:R_0603_1608Metric, F.Cu at (67.1, -63.0)
- added R45: 51, Resistor_SMD:R_0603_1608Metric, F.Cu at (67.1, -59.9)
- added R46: 51, Resistor_SMD:R_0603_1608Metric, F.Cu at (67.1, -61.5)
- added R47: 100k, Resistor_SMD:R_0603_1608Metric, F.Cu at (17.5, -73.7)
- added R48: 680, Resistor_SMD:R_0603_1608Metric, F.Cu at (11.9, -73.7)
- added R49: 10k, Resistor_SMD:R_0603_1608Metric, F.Cu at (8.89, -73.7)
- added R50: 10k, Resistor_SMD:R_0603_1608Metric, F.Cu at (7.37, -73.7)
- added R51: 200K, Resistor_SMD:R_0603_1608Metric, F.Cu at (16.0, -73.7)
- added R52: 100k, Resistor_SMD:R_0603_1608Metric, F.Cu at (17.5, -78.2)
- added R53: 680, Resistor_SMD:R_0603_1608Metric, F.Cu at (11.9, -78.2)
- added R54: 10k, Resistor_SMD:R_0603_1608Metric, F.Cu at (8.89, -78.2)
- added R55: 10k, Resistor_SMD:R_0603_1608Metric, F.Cu at (7.37, -78.2)
- added R56: 200K, Resistor_SMD:R_0603_1608Metric, F.Cu at (16.0, -78.2)
- added R57: 0, Resistor_SMD:R_0603_1608Metric, F.Cu at (10.4, -73.7)
- added R58: 0, Resistor_SMD:R_0603_1608Metric, F.Cu at (10.4, -78.2)
- added R59: 100, Resistor_SMD:R_0603_1608Metric, F.Cu at (53.1, -45.0)
- added R60: 100, Resistor_SMD:R_0603_1608Metric, F.Cu at (53.1, -46.5)
- added R61: 100, Resistor_SMD:R_0603_1608Metric, F.Cu at (53.1, -48.0)
- added R62: 100, Resistor_SMD:R_0603_1608Metric, F.Cu at (53.1, -24.4)
- added R63: 100, Resistor_SMD:R_0603_1608Metric, F.Cu at (53.1, -25.9)
- added R64: 100, Resistor_SMD:R_0603_1608Metric, F.Cu at (53.1, -27.4)
- added R65: 10k, Resistor_SMD:R_0603_1608Metric, F.Cu at (15.2, -22.1)
- added R66: DNP, Resistor_SMD:R_0603_1608Metric, F.Cu at (20.8, -22.1)
- added R67: 10k, Resistor_SMD:R_0603_1608Metric, F.Cu at (22.6, -22.1)
- added R68: 10k, Resistor_SMD:R_0603_1608Metric, F.Cu at (15.5, -4.32)
- added R69: DNP, Resistor_SMD:R_0603_1608Metric, F.Cu at (21.1, -4.32)
- added R70: 10k, Resistor_SMD:R_0603_1608Metric, F.Cu at (22.9, -4.32)
- added R71: 10k, Resistor_SMD:R_0603_1608Metric, F.Cu at (15.5, -10.2)
- added R72: DNP, Resistor_SMD:R_0603_1608Metric, F.Cu at (21.1, -10.2)
- added R73: 10k, Resistor_SMD:R_0603_1608Metric, F.Cu at (22.9, -10.2)
- added R74: 10k, Resistor_SMD:R_0603_1608Metric, F.Cu at (15.5, -16.0)
- added R75: DNP, Resistor_SMD:R_0603_1608Metric, F.Cu at (21.1, -16.0)
- added R76: 10k, Resistor_SMD:R_0603_1608Metric, F.Cu at (22.9, -16.0)
- added R77: 100k, Resistor_SMD:R_0603_1608Metric, F.Cu at (17.5, -64.9)
- added R78: 680, Resistor_SMD:R_0603_1608Metric, F.Cu at (11.9, -64.9)
- added R79: 10k, Resistor_SMD:R_0603_1608Metric, F.Cu at (8.89, -64.9)
- added R80: 10k, Resistor_SMD:R_0603_1608Metric, F.Cu at (7.37, -64.9)
- added R81: 200K, Resistor_SMD:R_0603_1608Metric, F.Cu at (16.0, -64.9)
- added R82: 100k, Resistor_SMD:R_0603_1608Metric, F.Cu at (17.5, -69.1)
- added R83: 680, Resistor_SMD:R_0603_1608Metric, F.Cu at (11.9, -69.1)
- added R84: 10k, Resistor_SMD:R_0603_1608Metric, F.Cu at (8.89, -69.1)
- added R85: 10k, Resistor_SMD:R_0603_1608Metric, F.Cu at (7.37, -69.1)
- added R86: 200K, Resistor_SMD:R_0603_1608Metric, F.Cu at (16.0, -69.1)
- added R87: 0, Resistor_SMD:R_0603_1608Metric, F.Cu at (10.4, -64.9)
- added R88: 0, Resistor_SMD:R_0603_1608Metric, F.Cu at (10.4, -69.1)
- added RN1: MAX5490GC01000+T, Package_TO_SOT_SMD:SOT-23, F.Cu at (30.5, -34.5)
- added RN2: MAX5490GC01000+T, Package_TO_SOT_SMD:SOT-23, F.Cu at (30.5, -42.2)
- added RN3: MAX5490GC01000+T, Package_TO_SOT_SMD:SOT-23, F.Cu at (30.5, -24.1)
- added U1: DRV8838DSGT, Package_SON:WSON-8-1EP_2x2mm_P0.5mm_EP0.9x1.6mm, F.Cu at (57.1, -34.2)
- added U10: MAX7311AAG+, Package_SO:SSOP-24_5.3x8.2mm_P0.65mm, F.Cu at (40.6, -60.7)
- added U11: MCP47FVB24-E/MQ, payload-interface-board:MCP47FVB24EMQ, F.Cu at (45.2, -46.5)
- added U12: ALM2402QPWPRQ1, Package_SO:HTSSOP-14-1EP_4.4x5mm_P0.65mm_EP3.4x5mm_Mask3x3.1mm, F.Cu at (41.9, -38.6)
- added U13: OPA340MDBVTEP, Package_TO_SOT_SMD:SOT-23-5, F.Cu at (73.4, -57.9)
- added U14: AD7091R-5BCPZ-RL7, Package_DFN_QFN:QFN-20-1EP_4x4mm_P0.5mm_EP2.5x2.5mm, F.Cu at (62.2, -57.4)
- added U15: ALM2402QPWPRQ1, Package_SO:HTSSOP-14-1EP_4.4x5mm_P0.65mm_EP3.4x5mm_Mask3x3.1mm, F.Cu at (41.9, -23.9)
- added U16: DRV8838DSGT, Package_SON:WSON-8-1EP_2x2mm_P0.5mm_EP0.9x1.6mm, F.Cu at (57.1, -44.3)
- added U17: INA240A3EDRQ1, Package_SO:SOIC-8_3.9x4.9mm_P1.27mm, F.Cu at (68.8, -43.7)
- added U18: INA240A3EDRQ1, Package_SO:SOIC-8_3.9x4.9mm_P1.27mm, F.Cu at (68.8, -33.5)
- added U19: DRV8838DSGT, Package_SON:WSON-8-1EP_2x2mm_P0.5mm_EP0.9x1.6mm, F.Cu at (57.1, -23.9)
- added U20: INA240A3EDRQ1, Package_SO:SOIC-8_3.9x4.9mm_P1.27mm, F.Cu at (68.8, -23.4)
- added U21: OPA340MDBVTEP, Package_TO_SOT_SMD:SOT-23-5, F.Cu at (34.0, -34.5)
- added U22: OPA340MDBVTEP, Package_TO_SOT_SMD:SOT-23-5, F.Cu at (34.0, -42.2)
- added U23: OPA340MDBVTEP, Package_TO_SOT_SMD:SOT-23-5, F.Cu at (34.0, -24.1)
- added U3: IAM-20380, payload-interface-board:IAM-20380, F.Cu at (10.2, -34.3)
- added U4: IAM-20380, payload-interface-board:IAM-20380, F.Cu at (10.2, -44.2)
- added U5: PCA9543APW,118, Package_SO:TSSOP-14_4.4x5mm_P0.65mm, F.Cu at (17.3, -56.6)
- added U6: MMC5983MA, payload-interface-board:MMC5983MA, F.Cu at (16.0, -34.3)
- added U7: MMC5983MA, payload-interface-board:MMC5983MA, F.Cu at (16.0, -44.2)
- added U8: MXC6655XA, payload-interface-board:MXC6655XA, F.Cu at (21.4, -34.3)
- added U9: MXC6655XA, payload-interface-board:MXC6655XA, F.Cu at (21.4, -44.2)
- R1, R2, R3: value 10k -> 100; footprint Resistor_SMD:R_0603_1608Metric_Pad0.98x0.95mm_HandSolder -> Resistor_SMD:R_0603_1608Metric
- moved G*** 37.0 mm to (-18.6, -7.14)
- moved R1 19.4 mm to (53.1, -34.7)
- moved R2 16.6 mm to (53.1, -36.2)
- moved R3 6.36 mm to (53.1, -37.7)
- renumbered C3 to C10, C4 to C11, C1 to C12, C2 to C13, C7 to C4, C8 to C5, C9 to C6, C10 to C7, C5 to C8, C6 to C9, D1 to D2, D2 to D3, D3 to D4, D4 to D5, J2 to J3, Q5 to Q1, Q6 to Q2, Q7 to Q3, Q8 to Q4, R14 to R10, R22 to R11, R18 to R12, R23 to R14, R19 to R15, R20 to R4, R15 to R5, R24 to R6, R16 to R7, R21 to R8, R17 to R9, U1 to U2
Connections:
- R1 pad 1: +3V3 -> /Magnetotorquer Drivers/~{DRV_SLP_Y}
- R1 pad 2: /H2-6 -> Net-(R1-Pad2)
- R2 pad 1: +5V -> /Magnetotorquer Drivers/DRV_PH_Y
- R2 pad 2: /SERVO_PWR_CTRL -> Net-(R2-Pad2)
- R3 pad 1: +3V3 -> /Magnetotorquer Drivers/DRV_EN_Y
- R3 pad 2: /H1-19 -> Net-(R3-Pad2)
Routing:
- net GND: track 69.8 -> 205.6 mm, vias 14 -> 106
- net /Magnetotorquer Drivers/2.5V_Vref: track 0.00 -> 98.9 mm, vias 0 -> 6
- net /SDA_Magnetotorquers: track 0.00 -> 87.5 mm, vias 0 -> 4
- net /SCL_Magnetotorquers: track 0.00 -> 85.7 mm, vias 0 -> 4
- net /5V_USB: track 102.2 -> 31.5 mm, vias 6 -> 2
- net +3V3: track 26.9 -> 97.5 mm, vias 5 -> 41
- net /Magnetotorquer Drivers/DRV_EN_Z: track 0.00 -> 61.5 mm, vias 0 -> 2
- net /Magnetotorquer Drivers/~{DRV_SLP_Z}: track 0.00 -> 58.8 mm, vias 0 -> 2
- net /Magnetotorquer Drivers/DRV_PH_Z: track 0.00 -> 57.5 mm, vias 0 -> 2
- net /Magnetotorquer Drivers/ADC_ALERT/BUSY: track 0.00 -> 54.6 mm, vias 0 -> 2
- net /Magnetotorquer Drivers/~{DRV_SLP_Y}: track 0.00 -> 53.7 mm, vias 0 -> 2
- net /IMU/SCL_IMU2: track 0.00 -> 53.6 mm, vias 0 -> 4
- net /Magnetotorquer Drivers/DRV_EN_Y: track 0.00 -> 53.0 mm, vias 0 -> 2
- net /IMU/SDA_IMU2: track 0.00 -> 48.3 mm, vias 0 -> 4
- net /Magnetotorquer Drivers/~{AMP_SHDN_Z}: track 0.00 -> 46.2 mm, vias 0 -> 3
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- added copper zone on F.Cu, net +3V3
- added copper zone on In3.Cu, net +3V3
- added copper zone on B.Cu, net +5V
- added copper zone on F.Cu, net /Magnetotorquer Drivers/Full Bridge 1/OUT2
- added copper zone on F.Cu, net /Magnetotorquer Drivers/Full Bridge 2/OUT2
- added copper zone on F.Cu, net /Magnetotorquer Drivers/Full Bridge 3/OUT2
- added copper zone on F.Cu, net /Magnetotorquer Drivers/X_Drive
- added copper zone on F.Cu, net /Magnetotorquer Drivers/Y_Drive
- added copper zone on F.Cu, net /Magnetotorquer Drivers/Z_drive
- added copper zone on F.Cu, net /X+
- added copper zone on F.Cu, net /Y+
- added copper zone on F.Cu, net /Z+
- added copper zone on F.Cu, net GND
- added copper zone on In1.Cu, net GND
- added copper zone on In4.Cu, net GND
- removed copper zone on B.Cu, net +3V3
- removed copper zone on In1.Cu, net +5V
- removed copper zone on In2.Cu, net GND
Other:
- copper layers 4 -> 6
- board text removed: "3.3V IO"
- board text removed: "5V IO"
- board text removed: "PAYLOAD_RX"
- board text removed: "PAYLOAD_TX"
- board text removed: "RESET"
- board text removed: "SERVO_PWR_CTRL"

Commit message: updated board
Parts:
- moved J2 24.1 mm to (83.1, -48.3)
- moved J1 16.0 mm to (46.0, -25.5)
- moved C1 15.1 mm to (53.7, -47.5)
- moved C29 15.1 mm to (37.7, -70.0)
- moved C32 15.1 mm to (48.4, -53.0)
- moved C37 15.1 mm to (66.2, -72.3)
- moved C46 15.1 mm to (56.8, -72.3)
- moved R25 15.1 mm to (47.9, -72.3)
- moved R35 15.1 mm to (39.8, -48.9)
- moved R37 15.1 mm to (67.7, -72.3)
- moved R43 15.1 mm to (66.9, -69.2)
- moved R44 15.1 mm to (66.9, -78.1)
- moved U13 15.1 mm to (73.3, -73.0)
- moved C3 15.1 mm to (56.8, -44.5)
- moved C57 15.1 mm to (57.0, -35.9)
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Routing:
- net /X+: track 38.7 -> 24.3 mm
- net /X-: track 36.9 -> 25.7 mm
- net /Y+: track 30.5 -> 20.0 mm
- net /Z+: track 28.9 -> 18.4 mm
- net /Z-: track 28.4 -> 19.9 mm
- net /Y-: track 29.3 -> 21.9 mm
Other:
- outline, holes or cut-outs redrawn

Commit message: design updates
Parts:
- added J4: T1M-6-F-SV-L, payload-interface-board:SAMTEC_T1M-06-F-SV-L, F.Cu at (43.0, -33.5)
- added J5: T1M-10-F-SV-L, payload-interface-board:SAMTEC_T1M-10-F-SV-L, F.Cu at (14.6, -20.3)
- added Q17: MMBT4401-7-F, Package_TO_SOT_SMD:SOT-23, F.Cu at (35.1, -73.2)
- added Q18: MMBT4401-7-F, Package_TO_SOT_SMD:SOT-23, F.Cu at (29.5, -55.6)
- added Q19: IRF7404TRPBF, Package_SO:SO-8_3.9x4.9mm_P1.27mm, F.Cu at (34.6, -52.1)
- added Q20: MMBT4401-7-F, Package_TO_SOT_SMD:SOT-23, F.Cu at (73.4, -24.4)
- added Q21: IRF7404TRPBF, Package_SO:SO-8_3.9x4.9mm_P1.27mm, F.Cu at (68.8, -17.5)
- added Q22: MMBT4401-7-F, Package_TO_SOT_SMD:SOT-23, F.Cu at (30.0, -24.0)
- added Q23: IRF7404TRPBF, Package_SO:SO-8_3.9x4.9mm_P1.27mm, F.Cu at (25.0, -17.5)
- added Q24: BSS138, Package_TO_SOT_SMD:SOT-23, F.Cu at (31.8, -67.1)
- added Q25: BSS138, Package_TO_SOT_SMD:SOT-23, F.Cu at (44.7, -25.1)
- added Q26: BSS138, Package_TO_SOT_SMD:SOT-23, F.Cu at (36.6, -67.1)
- added Q27: BSS138, Package_TO_SOT_SMD:SOT-23, F.Cu at (44.7, -14.0)
- added Q28: BSS138, Package_TO_SOT_SMD:SOT-23, F.Cu at (44.7, -19.8)
- added R100: 10k, Resistor_SMD:R_0603_1608Metric, F.Cu at (26.7, -53.3)
- added R101: 3.3k, Resistor_SMD:R_0603_1608Metric, F.Cu at (33.0, -57.1)
- added R102: 100k, Resistor_SMD:R_0603_1608Metric, F.Cu at (70.9, -21.6)
- added R103: 10k, Resistor_SMD:R_0603_1608Metric, F.Cu at (70.1, -24.4)
- added R104: 3.3k, Resistor_SMD:R_0603_1608Metric, F.Cu at (74.4, -19.1)
- added R105: 100k, Resistor_SMD:R_0603_1608Metric, F.Cu at (27.3, -21.2)
- added R106: 10k, Resistor_SMD:R_0603_1608Metric, F.Cu at (26.5, -24.0)
- added R107: 3.3k, Resistor_SMD:R_0603_1608Metric, F.Cu at (31.0, -19.0)
- added R108: 10k, Resistor_SMD:R_0603_1608Metric, F.Cu at (31.8, -69.6)
- added R109: DNP, Resistor_SMD:R_0603_1608Metric, F.Cu at (31.8, -64.5)
- added R110: 10k, Resistor_SMD:R_0603_1608Metric, F.Cu at (31.8, -62.7)
- added R111: 10k, Resistor_SMD:R_0603_1608Metric, F.Cu at (41.9, -25.1)
- added R112: DNP, Resistor_SMD:R_0603_1608Metric, F.Cu at (48.8, -25.1)
- added R113: 10k, Resistor_SMD:R_0603_1608Metric, F.Cu at (47.2, -25.1)
- added R114: 10k, Resistor_SMD:R_0603_1608Metric, F.Cu at (36.6, -69.6)
- added R115: DNP, Resistor_SMD:R_0603_1608Metric, F.Cu at (36.6, -64.5)
- added R116: 10k, Resistor_SMD:R_0603_1608Metric, F.Cu at (36.6, -62.7)
- added R117: 10k, Resistor_SMD:R_0603_1608Metric, F.Cu at (41.9, -14.0)
- added R118: DNP, Resistor_SMD:R_0603_1608Metric, F.Cu at (47.2, -14.0)
- added R119: 10k, Resistor_SMD:R_0603_1608Metric, F.Cu at (48.8, -14.0)
- added R120: 10k, Resistor_SMD:R_0603_1608Metric, F.Cu at (41.9, -19.8)
- added R121: DNP, Resistor_SMD:R_0603_1608Metric, F.Cu at (47.2, -19.8)
- added R122: 10k, Resistor_SMD:R_0603_1608Metric, F.Cu at (48.8, -19.8)
- added R89: 10k, Resistor_SMD:R_0603_1608Metric, F.Cu at (32.5, -73.4)
- added R90: 0, Resistor_SMD:R_0603_1608Metric, F.Cu at (52.6, -23.4)
- added R91: 0, Resistor_SMD:R_0603_1608Metric, F.Cu at (51.1, -23.4)
- added R92: 0, Resistor_SMD:R_0603_1608Metric, F.Cu at (52.6, -19.8)
- added R93: 0, Resistor_SMD:R_0603_1608Metric, F.Cu at (51.1, -19.8)
- added R94: 100k, Resistor_SMD:R_0603_1608Metric, F.Cu at (37.6, -73.2)
- added R95: 0, Resistor_SMD:R_0603_1608Metric, F.Cu at (34.8, -59.2)
- added R96: 0, Resistor_SMD:R_0603_1608Metric, F.Cu at (34.8, -61.0)
- added R97: 0, Resistor_SMD:R_0603_1608Metric, F.Cu at (31.8, -59.2)
- added R98: 0, Resistor_SMD:R_0603_1608Metric, F.Cu at (31.7, -60.9)
- added R99: 100k, Resistor_SMD:R_0603_1608Metric, F.Cu at (29.5, -52.3)
- added TP19: TestPoint, TestPoint:TestPoint_Pad_D1.0mm, F.Cu at (2.29, -32.3)
- added TP20: TestPoint, TestPoint:TestPoint_Pad_D1.0mm, F.Cu at (9.65, -26.4)
- added TP28: TestPoint, TestPoint:TestPoint_Pad_D1.0mm, F.Cu at (70.1, -85.9)
- added TP38: TestPoint, TestPoint:TestPoint_Pad_D1.0mm, F.Cu at (39.6, -69.6)
- added TP39: TestPoint, TestPoint:TestPoint_Pad_D1.0mm, F.Cu at (37.3, -60.9)
- added U24: RockBlock_9603, payload-interface-board:RockBlock_9603, B.Cu at (56.5, -25.4)
- H1: value MountingHole_Pad -> SLI-Backplane-Blank-Card-KiCad:125mil_hole
- J1: value T2M-105-01-X-D-TH-DS -> T1M-10-F-SV-L; footprint payload-interface-board:SAMTEC_T2M-105-01-X-D-TH-DS -> payload-interface-board:SAMTEC_T1M-10-F-SV-L; moved to B.Cu
- J2: value T2M-105-01-X-D-TH-DS -> T1M-10-F-SV-L; footprint payload-interface-board:SAMTEC_T2M-105-01-X-D-TH-DS -> payload-interface-board:SAMTEC_T1M-10-F-SV-L; moved to F.Cu
- Q10, Q11, Q12, Q9: value Q_NMOS_GSD -> BSS138
- R44: value 100 -> 100k
- moved RN3 50.2 mm to (46.6, -86.7), turned to 180 degrees
- moved R26 49.2 mm to (80.9, -84.2), turned to -90 degrees
- moved C68 48.3 mm to (49.9, -86.7), turned to 90 degrees
- moved R27 48.1 mm to (79.4, -84.2), turned to -90 degrees
- moved C67 48.0 mm to (43.6, -83.2), turned to 90 degrees
- moved R39 47.1 mm to (42.0, -81.5), turned to -90 degrees
- moved C65 45.8 mm to (67.7, -86.7), turned to 90 degrees
- moved U23 45.8 mm to (46.6, -83.2), turned to 180 degrees
- moved RN1 45.7 mm to (57.0, -86.7), turned to 180 degrees
- moved RN2 45.2 mm to (64.7, -86.7), turned to 180 degrees
- moved C62 45.2 mm to (60.1, -86.7), turned to 90 degrees
- moved R40 43.8 mm to (42.0, -78.2), turned to -90 degrees
- moved C69 43.7 mm to (49.9, -83.2), turned to 90 degrees
- moved U10 42.7 mm to (83.2, -76.6), turned to 90 degrees
- moved C61 41.7 mm to (54.0, -83.2), turned to 90 degrees
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Connections:
- J1 pad 1: GND -> /RB_RxD
- J1 pad 10: +5V -> GND
- J1 pad 2: GND -> /RB_CTS
- J1 pad 3: GND -> /RB_RTS
- J1 pad 4: /SERVO_PWR_CTRL -> /RB_NetAv
- J1 pad 5: /RXD -> /RB_RI
- J1 pad 6: /TXD -> /RB_TxD
- J1 pad 7: /RESET -> /RB_OnOff
- J1 pad 8: +5V -> /RB_5V_IN
- J1 pad 9: +5V -> /RB_Li-iON
- J2 pad 1: /X+ -> /ST_5V
- J2 pad 10: /Z- -> GND
- J2 pad 2: /X- -> /ST_5V
- J2 pad 3: unconnected-(J2-Pad3) -> /ST_5V
- J2 pad 4: unconnected-(J2-Pad4) -> /ST_RST
- J2 pad 5: /Y+ -> /ST_TXD
- J2 pad 6: /Y- -> /ST_RXD
- J2 pad 8: unconnected-(J2-Pad8) -> GND
- J2 pad 9: /Z+ -> GND
- P1 pad 73: /H1-33 -> 5V_RF
- Q10 pad 3: /H2-6 -> /H1-5
- Q11 pad 2: /TXD -> /P_TXD
- Q12 pad 2: /RXD -> /P_RXD
- Q9 pad 2: /RESET -> /P_RESET
- R44 pad 1: Net-(R44-Pad1) -> /H1-08
- R44 pad 2: /Magnetotorquer Drivers/ADC_CONVST -> GND
- R66 pad 2: /RESET -> /P_RESET
- R67 pad 2: /RESET -> /P_RESET
- R68 pad 2: /H2-6 -> /H1-5
- R69 pad 1: /H2-6 -> /H1-5
- R72 pad 2: /TXD -> /P_TXD
- R73 pad 2: /TXD -> /P_TXD
- R75 pad 2: /RXD -> /P_RXD
- R76 pad 2: /RXD -> /P_RXD
- U10 pad 19: /Magnetotorquer Drivers/ADC_CONVST -> /Magnetotorquer Drivers/~{ADC_RST}
- U10 pad 20: unconnected-(U10-Pad20) -> /Ball_Deploy
- U14 pad 17: Net-(R44-Pad1) -> unconnected-(U14-Pad17)
Routing:
- net /Magnetotorquer Drivers/ADC_CONVST: track 44.8 -> 0.00 mm, vias 2 -> 0
- net /Magnetotorquer Drivers/ADC_ALERT/BUSY: track 54.6 -> 9.86 mm
- net /RESET: track 37.7 -> 0.00 mm
- net /RXD: track 32.8 -> 0.00 mm
- net /H2-6: track 100.0 -> 68.3 mm, vias 1 -> 0
- net /TXD: track 30.3 -> 0.00 mm
- net /SERVO_PWR_CTRL: track 29.5 -> 3.51 mm
- net /H1-19: track 100.7 -> 81.6 mm
- net /SDA_Magnetotorquers: track 87.5 -> 72.2 mm
- net GND: track 205.6 -> 191.4 mm, vias 106 -> 103
- net /H1-20: track 94.0 -> 80.5 mm
- net /SCL_Magnetotorquers: track 85.7 -> 72.8 mm
- net /P_RESET: track 0.00 -> 10.8 mm
- net /Magnetotorquer Drivers/2.5V_ADCout: track 33.0 -> 23.7 mm
- net /H1-6: track 75.9 -> 68.6 mm
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Other:
- outline, holes or cut-outs redrawn

Commit message: friday changes
Parts:
- removed J2: T1M-10-F-SV-L, payload-interface-board:SAMTEC_T1M-10-F-SV-L
- removed Q25, Q27, Q28: BSS138, Package_TO_SOT_SMD:SOT-23
- removed R102: 100k, Resistor_SMD:R_0603_1608Metric
- removed R103, R111, R113, R117, R119, R120, R122: 10k, Resistor_SMD:R_0603_1608Metric
- removed R104: 3.3k, Resistor_SMD:R_0603_1608Metric
- removed R112, R118, R121: DNP, Resistor_SMD:R_0603_1608Metric
- removed R93: 0, Resistor_SMD:R_0603_1608Metric
- added C72: 1uF, Capacitor_SMD:C_0603_1608Metric, B.Cu at (61.5, -10.9)
- added D8: S1G, Diode_SMD:D_SMA, B.Cu at (60.2, -14.2)
- added U25: Pico, RPi_Pico:RPi_Pico_SMD_TH, B.Cu at (26.9, -24.1)
- C1, C2, C29, C3, C30, C31, C32, C33, C34, C35, C36, C37, C38, C39, C40, C41, C42, C43, C44, C45, C46, C49, C50, C51, C52, C53, C54, C55, C56, C57, C58, C59, C60, C61, C62, C63, C64, C65, C66, C67, C68, C69, D1, D6, D7, J4, Q17, Q18, Q19, Q20, Q21, Q22, Q24, Q26, R1, R100, R101, R105, R106, R108, R109, R110, R114, R115, R116, R2, R25, R26, R27, R28, R29, R3, R30, R31, R32, R33, R34, R35, R36, R37, R38, R39, R40, R41, R42, R43, R44, R45, R46, R59, R60, R61, R62, R63, R64, R89, R94, R95, R96, R97, R98, R99, RN1, RN2, RN3, TP28, TP38, TP39, U1, U10, U11, U12, U13, U14, U15, U16, U17, U18, U19, U20, U21, U22, U23: moved to B.Cu
- J1, U24: moved to F.Cu
- R90: value 0 -> 100k; moved to B.Cu
- R91: value 0 -> 10k; moved to B.Cu
- R92: value 0 -> 3.3k; moved to B.Cu
- moved TP19 84.9 mm to (87.1, -33.6), turned to -90 degrees
- moved R65 82.1 mm to (84.2, -33.7), turned to 0 degrees
- moved C35 81.9 mm to (4.13, -56.3)
- moved R41 80.3 mm to (4.89, -60.6)
- moved G*** 80.0 mm to (35.3, -66.3)
- moved Q9 79.2 mm to (84.2, -30.9), turned to 0 degrees
- moved C39 77.8 mm to (6.16, -56.0)
- moved R46 77.8 mm to (6.16, -50.2)
- moved R66 76.4 mm to (84.2, -28.1), turned to 180 degrees
- moved R74 76.3 mm to (78.1, -33.5), turned to 0 degrees
- moved U10 76.3 mm to (6.93, -76.6)
- moved C44 75.8 mm to (7.18, -43.9)
- moved C36 74.8 mm to (7.69, -61.4), turned to 180 degrees
- moved R45 74.8 mm to (7.69, -50.2)
- moved R67 74.7 mm to (84.2, -26.4), turned to 180 degrees
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Connections:
- net /ST_5V renamed Net-(C72-Pad1)
- Q20 pad 1: /PAYLOAD_PWR_SW -> /Pico/RB_PWR_SW_B
- R90 pad 1: /Level Shifter 7/io_hi -> /H2-22
- R90 pad 2: /ST_TXD -> GND
- R91 pad 1: /Level Shifter 7/io_hi -> /H2-22
- R91 pad 2: /ST_RXD -> /Pico/RB_PWR_SW_B
- R92 pad 1: /Level Shifter 8/io_hi -> +5V
- R92 pad 2: /ST_TXD -> Net-(Q20-Pad3)
Routing:
- net /H1-20: track 80.5 -> 12.7 mm
- net /H1-19: track 81.6 -> 14.7 mm
- net /H1-6: track 68.6 -> 5.98 mm
- net /H2-6: track 68.3 -> 6.40 mm
- net /SDA_SYS: track 42.9 -> 26.0 mm, vias 3 -> 2
- net /SCL_SYS: track 45.9 -> 29.9 mm, vias 4 -> 3
- net /RB_RxD: track 2.67 -> 0.00 mm, vias 2 -> 0
- net GND: track 191.4 -> 194.0 mm, vias 103 -> 105
- net /RB_Li-iON: track 1.34 -> 0.00 mm, vias 1 -> 0
- net /Magnetotorquer Drivers/Z_sen: track 22.2 -> 23.5 mm, vias 1 -> 2
- added copper zone on B.Cu, net +3V3
- added copper zone on B.Cu, net /Magnetotorquer Drivers/Full Bridge 1/OUT2
- added copper zone on B.Cu, net /Magnetotorquer Drivers/Full Bridge 2/OUT2
- added copper zone on B.Cu, net /Magnetotorquer Drivers/Full Bridge 3/OUT2
- added copper zone on B.Cu, net /Magnetotorquer Drivers/X_Drive
- added copper zone on B.Cu, net /Magnetotorquer Drivers/Y_Drive
- added copper zone on B.Cu, net /Magnetotorquer Drivers/Z_drive
- added copper zone on B.Cu, net /X+
- added copper zone on B.Cu, net /Y+
- added copper zone on B.Cu, net /Z+
- added copper zone on B.Cu, net GND
- removed copper zone on F.Cu, net +3V3
- removed copper zone on B.Cu, net +5V
- removed copper zone on F.Cu, net /Magnetotorquer Drivers/Full Bridge 1/OUT2
- removed copper zone on F.Cu, net /Magnetotorquer Drivers/Full Bridge 2/OUT2
- removed copper zone on F.Cu, net /Magnetotorquer Drivers/Full Bridge 3/OUT2
- removed copper zone on F.Cu, net /Magnetotorquer Drivers/X_Drive
- removed copper zone on F.Cu, net /Magnetotorquer Drivers/Y_Drive
- removed copper zone on F.Cu, net /Magnetotorquer Drivers/Z_drive
- removed copper zone on F.Cu, net /X+
- removed copper zone on F.Cu, net /Y+
- removed copper zone on F.Cu, net /Z+
- removed copper zone on F.Cu, net GND
