File: FP Interface Card.kicad_pcb (KiCad board)
At the start: 6 copper layers, 90.2 x 101.1 mm, 260 parts, among them J1 T1M-10-F-SV-L, J3 ZX62-AB-5PA(31), J4 T1M-6-F-SV-L, J5 T1M-10-F-SV-L, P1 Card Edge for HSEC8-160-01-S-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, Q1 BC847BM3T5G, Q10 BSS138, Q11 BSS138, Q12 BSS138, Q13 BSS138DWQ-7, Q14 MMDT5551-7-F, Q15 BSS138DWQ-7, Q16 MMDT5551-7-F, Q17 MMBT4401-7-F, Q18 MMBT4401-7-F, Q19 IRF7404TRPBF, Q2 BC847BM3T5G, Q20 MMBT4401-7-F, Q21 IRF7404TRPBF, Q22 MMBT4401-7-F, Q23 IRF7404TRPBF, Q24 BSS138, Q26 BSS138, Q3 BC847BM3T5G, Q4 BC847BM3T5G, Q5 BSS138DWQ-7, Q6 MMDT5551-7-F, Q7 BSS138DWQ-7, Q8 MMDT5551-7-F, Q9 BSS138, SW1 SW_Push_SPST, U1 DRV8838DSGT, U10 MAX7311AAG+, U11 MCP47FVB24-E/MQ, U12 ALM2402QPWPRQ1, U13 OPA340MDBVTEP, U14 AD7091R-5BCPZ-RL7, U15 ALM2402QPWPRQ1, U16 DRV8838DSGT, U17 INA240A3EDRQ1, U18 INA240A3EDRQ1, U19 DRV8838DSGT, U2 AP2161W, U20 INA240A3EDRQ1, U21 OPA340MDBVTEP, U22 OPA340MDBVTEP, U23 OPA340MDBVTEP, U24 RockBlock_9603, U25 Pico, U3 IAM-20380, U4 IAM-20380, U5 PCA9543APW,118, U6 MMC5983MA, U7 MMC5983MA, U8 MXC6655XA, U9 MXC6655XA

Commit message: finished routing
Parts:
- removed TP19, TP20, TP28, TP38, TP39: TestPoint, TestPoint:TestPoint_Pad_D1.0mm
- added R93: 100k, Resistor_SMD:R_0603_1608Metric, B.Cu at (18.6, -54.7)
- C1, C29, C49, C56, Q17, Q18, Q19, Q24, Q26, R1, R100, R101, R108, R109, R110, R114, R115, R116, R2, R25, R26, R27, R3, R35, R39, R40, R41, R42, R43, R44, R45, R46, R59, R60, R61, R62, R63, R64, R89, R94, R95, R96, R97, R98, R99, U10: moved to F.Cu
- Q23, R107: moved to B.Cu
- moved C72 33.9 mm to (28.0, -5.72)
- moved D8 33.9 mm to (26.7, -9.02)
- moved Q21 33.9 mm to (35.1, -7.50)
- moved R92 33.5 mm to (40.7, -7.63)
- moved Q20 33.4 mm to (44.2, -6.81)
- moved R91 30.1 mm to (48.0, -6.98), turned to -90 degrees
- moved R90 28.5 mm to (50.3, -6.98), turned to -90 degrees
- moved R97 22.0 mm to (51.5, -80.1), turned to -90 degrees
- moved R98 19.9 mm to (53.3, -80.1), turned to -90 degrees
- moved J4 19.3 mm to (51.4, -58.3), turned to 90 degrees
- moved R70 18.5 mm to (77.7, -11.4)
- moved Q10 18.5 mm to (77.7, -16.0)
- moved R68 18.5 mm to (77.7, -18.8)
- moved R69 18.5 mm to (77.7, -13.2)
- moved R95 18.3 mm to (51.5, -77.1), turned to 90 degrees
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Connections:
- R100 pad 1: /H1-07 -> /H1-7
- R11 pad 2: /5V_USB -> /H1-11
- R14 pad 2: /H2-6 -> /H1-7
- R4 pad 2: /H1-19 -> /H1-5
- R44 pad 1: /H1-08 -> /H1-8
- R8 pad 2: /H1-20 -> /H2-22
- R89 pad 1: /H1-08 -> /H1-8
- R99 pad 1: /H1-07 -> /H1-7
- U10 pad 20: /Ball_Deploy -> unconnected-(U10-Pad20)
- U13 pad 3: /Magnetotorquer Drivers/2.5V_ADCout -> Net-(R93-Pad2)
- U13 pad 4: /Magnetotorquer Drivers/2.5V_Vref -> Net-(R102-Pad1)
Routing:
- net /H2-22: track 0.00 -> 145.3 mm, vias 0 -> 4
- net /H1-5: track 5.98 -> 144.7 mm, vias 1 -> 3
- net /H1-11: track 0.00 -> 132.4 mm, vias 0 -> 4
- net /H1-6: track 5.98 -> 111.1 mm, vias 1 -> 2
- net /H1-20: track 12.7 -> 114.0 mm
- net /SDA_IMU: track 28.9 -> 120.4 mm, vias 2 -> 4
- net /H1-19: track 14.7 -> 104.8 mm
- net /SCL_IMU: track 24.5 -> 112.2 mm, vias 2 -> 4
- net /H1-7: track 0.00 -> 81.5 mm, vias 0 -> 3
- net /5V_USB: track 31.5 -> 111.5 mm, vias 2 -> 5
- net /SDA_Magnetotorquers: track 72.2 -> 137.4 mm
- net /SCL_Magnetotorquers: track 72.8 -> 133.6 mm
- net /H1-8: track 0.00 -> 51.1 mm, vias 0 -> 2
- net GND: track 194.0 -> 238.8 mm, vias 105 -> 125
- net /RB_OnOff: track 0.00 -> 32.2 mm
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- added copper zone on B.Cu, net +5V
- added copper zone on In1.Cu, net +5V
- added copper zone on B.Cu, net /PAYLOAD_5V
- added copper zone on F.Cu, net /PAYLOAD_5V
- added copper zone on F.Cu, net /RB_5V_IN
- added copper zone on B.Cu, net 5V_RF
- added copper zone on F.Cu, net 5V_RF
- added copper zone on F.Cu, net GND
- added copper zone on B.Cu, net Net-(C72-Pad1)
