File: magnetotorquer-driver.kicad_sch (KiCad schematic)
At the start: 62 parts

Commit message: majority of routing completed
Parts:
- removed C? (x9): 0.1uF, Capacitor_SMD:C_0805_2012Metric, symbol Device:C
- removed C? (x3): 1uF, Capacitor_SMD:C_0805_2012Metric, symbol Device:C
- removed C? (x2): 560pF, symbol Device:C
- removed R? (x3): 33, symbol Device:R_US
- removed R? (x3): R_US, symbol Device:R_US
- removed R? (x9): 100, Resistor_SMD:R_0805_2012Metric, symbol Device:R_US
- removed U? (x3): INA240A3EDRQ1, Package_SO:SOIC-8_3.9x4.9mm_P1.27mm, symbol Amplifier_Current:INA240A3PW
- removed U? (x3): DRV8838DSGT, Package_SON:WSON-8-1EP_2x2mm_P0.5mm_EP0.9x1.6mm, symbol magnetotorquer-test-board:DRV8838DSGT
- added C29, C43, C44: 0.1uF, Capacitor_SMD:C_0603_1608Metric, symbol Device:C
- added C37, C42: 560pF, Capacitor_SMD:C_0603_1608Metric, symbol Device:C
- added R25: 100k, Resistor_SMD:R_0603_1608Metric, symbol Device:R_US
- added R26, R27: 51, Resistor_SMD:R_0603_1608Metric, symbol Device:R_US
- added R32, R33: 200mR, Resistor_SMD:R_0805_2012Metric, symbol Device:R_US
- added R34: 91mR, Resistor_SMD:R_0805_2012Metric, symbol Device:R_US
- added R36, R37, R38: 33, Resistor_SMD:R_0603_1608Metric, symbol Device:R_US
- added R41, R43, R44: 100, Resistor_SMD:R_0603_1608Metric, symbol Device:R_US
- added TP1, TP10, TP11, TP12, TP13, TP14, TP2, TP3, TP4, TP5, TP6, TP7, TP8, TP9: TestPoint, TestPoint:TestPoint_Pad_2.5x2.5mm, symbol Connector:TestPoint
- added U10: MAX7311AAG+, Package_SO:SSOP-24_5.3x8.2mm_P0.65mm, symbol FP-Interface-Card:MAX7311AAG+
- added U13: OPA340MDBVTEP, Package_TO_SOT_SMD:SOT-23-5, symbol Amplifier_Operational:OPA340NA
- C31, C32, C33, C38, C41: renamed from C?; footprint Capacitor_SMD:C_0805_2012Metric -> Capacitor_SMD:C_0603_1608Metric
- C34, C39, C40: renamed from C?; footprint (none) -> Capacitor_SMD:C_0603_1608Metric
- C35, C36, C45, C46: renamed from C?; footprint (none) -> Capacitor_SMD:C_0805_2012Metric
- R28, R29, R35, R42, R45, R46: renamed from R?; footprint Resistor_SMD:R_0805_2012Metric -> Resistor_SMD:R_0603_1608Metric
- R30, R31: renamed from R?; value 0 -> 100; footprint Resistor_SMD:R_0805_2012Metric -> Resistor_SMD:R_0603_1608Metric
- R39, R40: renamed from R?; footprint (none) -> Resistor_SMD:R_0603_1608Metric
- U11: renamed from U?; footprint (none) -> payload-interface-board:MCP47FVB24EMQ
- U14: renamed from U?; footprint (none) -> Package_DFN_QFN:QFN-20-1EP_4x4mm_P0.5mm_EP2.5x2.5mm
- gave numbers to parts that had none: 3
Connections:
- net Torquer_1_sen is gone; now on net GND: C34.1
- net +3V3: now also C36.1, C40.1, U14.1 (VDD), C29.1, C43.1, R25.1, U10.24 (V+), U13.5 (V+)
- net +5V: no longer C36.1, C40.1, U14.1 (VDD)
- net GND: now also U11.1 (A0), U11.15 (A1), U11.21 (EP), U14.14 (AS1), U14.19 (AS0), U14.21 (GND), C29.2, C37.1, C42.1, C43.2, C44.2, U10.12 (GND), U10.2 (AD1), U10.21 (AD0), U10.3 (AD2), U13.2 (V-); no longer C34.2, R30.1, R31.1
- net SCL: now also R46.1, R26.1
- net SDA: now also R45.1, R27.1
- net at U14.11 (Vin1): now also C37.2, R37.1
- net at U14.7 (Vin2): now also C42.2, R38.1
- net 2.5V_Vref: now reaches U11.14 (Vref1)
- net 2.5V_Vref: now also U11.2 (Vref0), C44.1, TP14.1, U13.1, U13.4 (-)
- net at U14.17 (CONVST/GPO1): now also R44.1
- net at U14.20 (~{RST}): now also R41.2
- net 2.5V_ADCout: now reaches C45.1, U14.3 (REFin/REFout)
- net 2.5V_ADCout: now also TP13.1, U13.3 (+)
- net at U14.6 (Vin0): now also C34.2, R36.1
- net at U14.8 (ALERT/BUSY/GPO0): now also R43.2
- removed net DAC_vout0: U11.3 (Vout0), U12.2 (IN1+), U15.2 (IN1+)
- net DAC_vout1 renamed Y_Vs_2.5V
- net Y_Vs_2.5V: now also TP2.1; no longer U12.4 (IN2+)
- net DAC_vout2 renamed Z_Vs_2.5V
- net Z_Vs_2.5V: now also TP3.1
- net SHDN renamed ~{AMP_SHDN_XY}
- net ~{AMP_SHDN_XY}: now also U10.6 (IO_2); no longer R42.2, U15.3 (OTF/SH_DM)
- net Torquer_Drive_1 renamed X_Drive
- net X_Drive: now also TP4.1
- net Torquer_Drive_2 renamed Y_Drive
- net Y_Drive: now also TP5.1
- net Torquer_Drive_3 renamed Z_drive
- net Z_drive: now also TP6.1
- new net: R27.2, U10.23 (SDA)
- new net: R25.2, U10.1 (~{INT})
- new net: R26.2, U10.22 (SCL)
- new net ADC_ALERT/BUSY: R43.1, U10.18 (IO_13)
- new net ADC_CONVST: R44.2, U10.19 (IO_14)
- new net DRV_EN_X: U10.9 (IO_5)
- new net DRV_EN_Y: U10.13 (IO_8)
- new net DRV_EN_Z: U10.16 (IO_11)
- new net DRV_PH_X: U10.8 (IO_4)
- new net DRV_PH_Y: U10.11 (IO_7)
- new net DRV_PH_Z: U10.15 (IO_10)
- new net Full Bridge 1/OUT2: R32.1
- new net Full Bridge 2/OUT2: R33.1
- new net Full Bridge 3/OUT2: R34.1
- new net X+: TP7.1
- new net X-: R32.2, TP8.1
- new net X_Vs_2.5V: TP1.1, U11.3 (Vout0)
- new net X_Vs_5V: U12.2 (IN1+)
- new net X_sen: R36.2
- new net Y+: TP9.1
- new net Y-: R33.2, TP10.1
- new net Y_Vs_5V: U12.4 (IN2+)
- new net Y_sen: R37.2
- new net Z+: TP11.1
- new net Z-: R34.2, TP12.1
- new net Z_Vs_5V: U15.2 (IN1+)
- new net Z_sen: R38.2
- new net ~{ADC_RST}: R41.1
- new net ~{AMP_SHDN_Z}: R42.2, U10.7 (IO_3), U15.3 (OTF/SH_DM)
- new net ~{DAC_LAT0}: R30.1, U10.4 (IO_0)
- new net ~{DAC_LAT1}: R31.1, U10.5 (IO_1)
- new net ~{DRV_SLP_X}: U10.10 (IO_6)
- new net ~{DRV_SLP_Y}: U10.14 (IO_9)
- new net ~{DRV_SLP_Z}: U10.17 (IO_12)
- no-connect marks 2 -> 3
Other:
- added sheet 5V Amp 1 (5V_amp.kicad_sch)
- added sheet 5V Amp 2 (5V_amp.kicad_sch)
- added sheet 5V Amp 3 (5V_amp.kicad_sch)
- added sheet Full Bridge 1 (Full_Bridge.kicad_sch)
- added sheet Full Bridge 2 (Full_Bridge.kicad_sch)
- added sheet Full Bridge 3 (Full_Bridge.kicad_sch)
- added sheet Sense Amp 1 (Sense_Amp.kicad_sch)
- added sheet Sense Amp 2 (Sense_Amp.kicad_sch)
- added sheet Sense Amp 3 (Sense_Amp.kicad_sch)
- note added: "0-2.5Vout"
- note added: "0-5Vout"
- note added: "2.5V vref buffer"
- note added: "5V AMPLIFIER"
- note added: "CURRENT SENSE ADC"
- note added: "DRIVE AMPLIFIER"
- note added: "HALF BRIDGE DRIVER & CURRENT SENSE"
- note added: "IO EXPANDER"
- note added: "addr. 0x2F"
- note added: "addr. 0x40"
- note added: "addr. 0x60"
- note added: "any way to get a super accurate 5V reference? always a dropout voltage"
- note added: "generated by ADC"
- note added: "lets say current will cause a +/- 1.0v defelection"
- note added: "r_rod = 1/(50mA)/100 = 200mR r_air = 1/110mA/100 = 91mR"
- note added: "take 0-2.5V DAC signal to 0-5V"
- note added: "update me!"
- note removed: "100v/v gain"
- note removed: "CURRENT SENSE"
- note removed: "CURRENT SENSE DAC"
- note removed: "DAC for unity gain buffer (driver voltage source)"
- note removed: "DRIVER STAGE"
- note removed: "FULL BRDIGE OUTPUT STAGE"
- note removed: "TBR"
- note removed: "current sense amplifier"
- note removed: "figure out what tobreakout IO w/ on this? thinking shift register"
- note removed: "half bridge driver"
- note removed: "lets say current will cause a +/- 1.5v defelection"
- note removed: "or a max7329 IO exp?"
- note removed: "r_rod = 1.5/(50mA)/100 = 300mR r_air = 1.5/110mA/100 = 136mR"
- note removed: "torque rods vs air core torqer sadly require different currents :("
- moved on the sheet: C30, C31, C32, C33, C34, C35, C36, C38, C39, C40, C41, C45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

Commit message: working on sch changes
Connections:
- net Ball_Deploy: now reaches U10.20 (IO_15)
- no-connect marks 3 -> 2
Other:
- note added: "snagging this off here saves mainboard IO"
Changed lines of the file:
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@@
   )
   (no_connect (at 344.17 151.13))
-  (no_connect (at 96.52 162.56))
   (no_connect (at 92.71 49.53))
   (wire (pts (xy 45.72 41.91) (xy 45.72 43.18))
@@
     (effects (font (size 2.54 2.54) (thickness 0.508) bold) (justify left bottom))
   )
+  (text "snagging this off here saves mainboard IO" (at 95.25 165.1 0)
+    (effects (font (size 1.27 1.27)) (justify left bottom))
+  )
   (text "update me!" (at 245.11 223.52 0)
     (effects (font (size 1.27 1.27)) (justify left bottom))
@@
     (effects (font (size 1.27 1.27)) (justify right bottom))
   )
+  (hierarchical_label "Ball_Deploy" (shape input) (at 96.52 162.56 0)
+    (effects (font (size 1.27 1.27)) (justify left))
+  )
   (hierarchical_label "SCL" (shape input) (at 24.13 104.14 180)

Commit message: working on EM
Parts:
- removed R44: 100, Resistor_SMD:R_0603_1608Metric, symbol Device:R_US
Connections:
- net ADC_CONVST is gone; now on net ~{ADC_RST}: U10.19 (IO_14)
Other:
- note added: "<- input"
- note added: "output ->"
- moved on the sheet: R41
Changed lines of the file:
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@@
     (stroke (width 0) (type default) (color 0 0 0 0))
   )
-  (wire (pts (xy 317.5 172.72) (xy 320.04 172.72))
+  (wire (pts (xy 309.88 172.72) (xy 312.42 172.72))
     (stroke (width 0) (type default) (color 0 0 0 0))
   )
@@
     (stroke (width 0) (type default) (color 0 0 0 0))
   )
-  (wire (pts (xy 387.35 142.24) (xy 389.89 142.24))
-    (stroke (width 0) (type default) (color 0 0 0 0))
-  )
   (wire (pts (xy 67.31 134.62) (xy 69.85 134.62))
     (stroke (width 0) (type default) (color 0 0 0 0))
   )
-  (wire (pts (xy 327.66 172.72) (xy 344.17 172.72))
-    (stroke (width 0) (type default) (color 0 0 0 0))
-  )
   (wire (pts (xy 95.25 72.39) (xy 95.25 74.93))
     (stroke (width 0) (type default) (color 0 0 0 0))
@@
     (stroke (width 0) (type default) (color 0 0 0 0))
   )
+  (wire (pts (xy 320.04 172.72) (xy 344.17 172.72))
+    (stroke (width 0) (type default) (color 0 0 0 0))
+  )
   (wire (pts (xy 209.55 158.75) (xy 209.55 173.99))
     (stroke (width 0) (type default) (color 0 0 0 0))
@@
     (stroke (width 0) (type default) (color 0 0 0 0))
   )
-  (wire (pts (xy 377.19 142.24) (xy 379.73 142.24))
-    (stroke (width 0) (type default) (color 0 0 0 0))
-  )
   (wire (pts (xy 209.55 143.51) (xy 223.52 143.51))
     (stroke (width 0) (type default) (color 0 0 0 0))
@@
     )
   )
+  (text "output ->" (at 114.3 139.7 0)
+    (effects (font (size 1.27 1.27)) (justify left bottom))
+  )
+  (text "output ->" (at 114.3 137.16 0)
+    (effects (font (size 1.27 1.27)) (justify left bottom))
+  )
   (text "lets say current will cause a +/- 1.0v defelection"
     (at 186.69 224.79 0)
@@
     (effects (font (size 1.27 1.27)) (justify left bottom))
   )
+  (text "output ->" (at 114.3 144.78 0)
+    (effects (font (size 1.27 1.27)) (justify left bottom))
+  )
   (text "update me!" (at 245.11 223.52 0)
     (effects (font (size 1.27 1.27)) (justify left bottom))
   )
+  (text "output ->" (at 114.3 142.24 0)
+    (effects (font (size 1.27 1.27)) (justify left bottom))
+  )
+  (text "output ->" (at 114.3 152.4 0)
+    (effects (font (size 1.27 1.27)) (justify left bottom))
+  )
   (text "r_rod = 1/(50mA)/100 = 200mR\nr_air = 1/110mA/100 = 91mR"
     (at 186.69 229.87 0)
@@
     (effects (font (size 1.27 1.27)) (justify left bottom))
   )
+  (text "output ->" (at 114.3 154.94 0)
+    (effects (font (size 1.27 1.27)) (justify left bottom))
+  )
+  (text "output ->" (at 114.3 147.32 0)
+    (effects (font (size 1.27 1.27)) (justify left bottom))
+  )
   (text "2.5V vref buffer" (at 303.53 193.04 0)
     (effects (font (size 2.54 2.54) (thickness 0.508) bold) (justify left bottom))
@@
     (effects (font (size 2.54 2.54) (thickness 0.508) bold) (justify left bottom))
   )
+  (text "output ->" (at 114.3 149.86 0)
+    (effects (font (size 1.27 1.27)) (justify left bottom))
+  )
+  (text "output ->" (at 113.665 160.02 0)
+    (effects (font (size 1.27 1.27)) (justify left bottom))
+  )
+  (text "output ->" (at 114.3 129.54 0)
+    (effects (font (size 1.27 1.27)) (justify left bottom))
+  )
   (text "0-5Vout" (at 147.32 39.37 0)
     (effects (font (size 1.27 1.27)) (justify left bottom))
   )
+  (text "output ->" (at 114.3 127 0)
+    (effects (font (size 1.27 1.27)) (justify left bottom))
+  )
+  (text "<- input " (at 113.665 157.48 0)
+    (effects (font (size 1.27 1.27)) (justify left bottom))
+  )
   (text "max rod current = 50mA\nmax air core current = 110mA"
     (at 186.69 218.44 0)
@@
     (effects (font (size 2.54 2.54) (thickness 0.508) bold) (justify left bottom))
   )
+  (text "output ->" (at 114.3 132.08 0)
+    (effects (font (size 1.27 1.27)) (justify left bottom))
+  )
+  (text "output ->" (at 114.3 134.62 0)
+    (effects (font (size 1.27 1.27)) (justify left bottom))
+  )
   (text "CURRENT SENSE ADC" (at 332.74 102.87 0)
     (effects (font (size 2.54 2.54) (thickness 0.508) bold) (justify left bottom))
   )
+  (text "output ->" (at 114.3 124.46 0)
+    (effects (font (size 1.27 1.27)) (justify left bottom))
+  )
   (text "check for pulldowns on DAC lines" (at 97.79 29.21 0)
     (effects (font (size 1.27 1.27)) (justify left bottom))
@@
     (effects (font (size 1.27 1.27)) (justify right bottom))
   )
-  (label "ADC_CONVST" (at 96.52 160.02 0)
-    (effects (font (size 1.27 1.27)) (justify left bottom))
-  )
   (label "Y_Drive" (at 251.46 76.2 180)
     (effects (font (size 1.27 1.27)) (justify right bottom))
@@
     (effects (font (size 1.27 1.27)) (justify left bottom))
   )
-  (label "ADC_CONVST" (at 389.89 142.24 0)
-    (effects (font (size 1.27 1.27)) (justify left bottom))
-  )
   (label "~{DAC_LAT0}" (at 59.69 66.04 180)
     (effects (font (size 1.27 1.27)) (justify right bottom))
@@
     (effects (font (size 1.27 1.27)) (justify left bottom))
   )
-  (label "~{ADC_RST}" (at 317.5 172.72 180)
+  (label "~{ADC_RST}" (at 309.88 172.72 180)
     (effects (font (size 1.27 1.27)) (justify right bottom))
   )
@@
     (effects (font (size 1.27 1.27)) (justify right bottom))
   )
+  (label "~{ADC_RST}" (at 96.52 160.02 0)
+    (effects (font (size 1.27 1.27)) (justify left bottom))
+  )
   (label "SDA" (at 57.15 134.62 180)
     (effects (font (size 1.27 1.27)) (justify right bottom))
@@
     (pin "9")
   )
-  (symbol (lib_id "Device:R_US") (at 383.54 142.24 90) (unit 1)
-    (in_bom yes) (on_board yes)
-    (property "Reference" "R44" (id 0) (at 379.73 140.97 90))
-    (property "Value" "100" (id 1) (at 387.35 140.97 90))
-    (property "Footprint" "Resistor_SMD:R_0603_1608Metric" (id 2) (at 383.794 141.224 90)
-      (effects (font (size 1.27 1.27)) hide)
-    )
-    (property "Datasheet" "~" (id 3) (at 383.54 142.24 0)
-      (effects (font (size 1.27 1.27)) hide)
-    )
-    (pin "1")
-    (pin "2")
-  )
   (symbol (lib_id "Device:C") (at 219.71 46.99 0) (unit 1)
     (in_bom yes) (on_board yes) (fields_autoplaced)
@@
     (pin "1")
   )
-  (symbol (lib_id "Device:R_US") (at 323.85 172.72 90) (unit 1)
+  (symbol (lib_id "Device:R_US") (at 316.23 172.72 90) (unit 1)
     (in_bom yes) (on_board yes)
-    (property "Reference" "R41" (id 0) (at 320.04 171.45 90))
-    (property "Value" "100" (id 1) (at 327.66 171.45 90))
-    (property "Footprint" "Resistor_SMD:R_0603_1608Metric" (id 2) (at 324.104 171.704 90)
+    (property "Reference" "R41" (id 0) (at 312.42 171.45 90))
+    (property "Value" "100" (id 1) (at 320.04 171.45 90))
+    (property "Footprint" "Resistor_SMD:R_0603_1608Metric" (id 2) (at 316.484 171.704 90)
       (effects (font (size 1.27 1.27)) hide)
     )
-    (property "Datasheet" "~" (id 3) (at 323.85 172.72 0)
+    (property "Datasheet" "~" (id 3) (at 316.23 172.72 0)
       (effects (font (size 1.27 1.27)) hide)
     )
@@
   )
   (symbol (lib_id "power:GND") (at 332.105 156.21 0) (unit 1)
-    (in_bom yes) (on_board yes) (fields_autoplaced)
+    (in_bom yes) (on_board yes)
     (property "Reference" "#PWR032" (id 0) (at 332.105 162.56 0)
       (effects (font (size 1.27 1.27)) hide)

Commit message: design updates
Parts:
- TP1, TP10, TP11, TP12, TP13, TP14, TP2, TP3, TP4, TP5, TP6, TP7, TP8, TP9: footprint TestPoint:TestPoint_Pad_2.5x2.5mm -> TestPoint:TestPoint_Pad_D1.0mm
Changed lines of the file:
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@@
       (effects (font (size 1.27 1.27)) (justify left) hide)
     )
-    (property "Footprint" "TestPoint:TestPoint_Pad_2.5x2.5mm" (id 2) (at 189.23 151.13 0)
+    (property "Footprint" "TestPoint:TestPoint_Pad_D1.0mm" (id 2) (at 189.23 151.13 0)
       (effects (font (size 1.27 1.27)) hide)
     )
@@
       (effects (font (size 1.27 1.27)) (justify left) hide)
     )
-    (property "Footprint" "TestPoint:TestPoint_Pad_2.5x2.5mm" (id 2) (at 113.03 41.91 0)
+    (property "Footprint" "TestPoint:TestPoint_Pad_D1.0mm" (id 2) (at 113.03 41.91 0)
       (effects (font (size 1.27 1.27)) hide)
     )
@@
       (effects (font (size 1.27 1.27)) (justify left) hide)
     )
-    (property "Footprint" "TestPoint:TestPoint_Pad_2.5x2.5mm" (id 2) (at 189.23 120.65 0)
+    (property "Footprint" "TestPoint:TestPoint_Pad_D1.0mm" (id 2) (at 189.23 120.65 0)
       (effects (font (size 1.27 1.27)) hide)
     )
@@
       (effects (font (size 1.27 1.27)) (justify left) hide)
     )
-    (property "Footprint" "TestPoint:TestPoint_Pad_2.5x2.5mm" (id 2) (at 224.79 158.75 0)
+    (property "Footprint" "TestPoint:TestPoint_Pad_D1.0mm" (id 2) (at 224.79 158.75 0)
       (effects (font (size 1.27 1.27)) hide)
     )
@@
       (effects (font (size 1.27 1.27)) (justify left) hide)
     )
-    (property "Footprint" "TestPoint:TestPoint_Pad_2.5x2.5mm" (id 2) (at 224.79 184.15 0)
+    (property "Footprint" "TestPoint:TestPoint_Pad_D1.0mm" (id 2) (at 224.79 184.15 0)
       (effects (font (size 1.27 1.27)) hide)
     )
@@
       (effects (font (size 1.27 1.27)) (justify left) hide)
     )
-    (property "Footprint" "TestPoint:TestPoint_Pad_2.5x2.5mm" (id 2) (at 224.79 123.19 0)
+    (property "Footprint" "TestPoint:TestPoint_Pad_D1.0mm" (id 2) (at 224.79 123.19 0)
       (effects (font (size 1.27 1.27)) hide)
     )
@@
       (effects (font (size 1.27 1.27)) (justify left) hide)
     )
-    (property "Footprint" "TestPoint:TestPoint_Pad_2.5x2.5mm" (id 2) (at 224.79 128.27 0)
+    (property "Footprint" "TestPoint:TestPoint_Pad_D1.0mm" (id 2) (at 224.79 128.27 0)
       (effects (font (size 1.27 1.27)) hide)
     )
@@
       (effects (font (size 1.27 1.27)) (justify left) hide)
     )
-    (property "Footprint" "TestPoint:TestPoint_Pad_2.5x2.5mm" (id 2) (at 344.17 200.66 0)
+    (property "Footprint" "TestPoint:TestPoint_Pad_D1.0mm" (id 2) (at 344.17 200.66 0)
       (effects (font (size 1.27 1.27)) hide)
     )
@@
       (effects (font (size 1.27 1.27)) (justify left) hide)
     )
-    (property "Footprint" "TestPoint:TestPoint_Pad_2.5x2.5mm" (id 2) (at 189.23 181.61 0)
+    (property "Footprint" "TestPoint:TestPoint_Pad_D1.0mm" (id 2) (at 189.23 181.61 0)
       (effects (font (size 1.27 1.27)) hide)
     )
@@
       (effects (font (size 1.27 1.27)) (justify left) hide)
     )
-    (property "Footprint" "TestPoint:TestPoint_Pad_2.5x2.5mm" (id 2) (at 120.65 46.99 0)
+    (property "Footprint" "TestPoint:TestPoint_Pad_D1.0mm" (id 2) (at 120.65 46.99 0)
       (effects (font (size 1.27 1.27)) hide)
     )
@@
       (effects (font (size 1.27 1.27)) (justify left) hide)
     )
-    (property "Footprint" "TestPoint:TestPoint_Pad_2.5x2.5mm" (id 2) (at 116.84 44.45 0)
+    (property "Footprint" "TestPoint:TestPoint_Pad_D1.0mm" (id 2) (at 116.84 44.45 0)
       (effects (font (size 1.27 1.27)) hide)
     )
@@
       (effects (font (size 1.27 1.27)) (justify left) hide)
     )
-    (property "Footprint" "TestPoint:TestPoint_Pad_2.5x2.5mm" (id 2) (at 374.65 203.2 0)
+    (property "Footprint" "TestPoint:TestPoint_Pad_D1.0mm" (id 2) (at 374.65 203.2 0)
       (effects (font (size 1.27 1.27)) hide)
     )
@@
       (effects (font (size 1.27 1.27)) (justify left) hide)
     )
-    (property "Footprint" "TestPoint:TestPoint_Pad_2.5x2.5mm" (id 2) (at 224.79 189.23 0)
+    (property "Footprint" "TestPoint:TestPoint_Pad_D1.0mm" (id 2) (at 224.79 189.23 0)
       (effects (font (size 1.27 1.27)) hide)
     )
@@
       (effects (font (size 1.27 1.27)) (justify left) hide)
     )
-    (property "Footprint" "TestPoint:TestPoint_Pad_2.5x2.5mm" (id 2) (at 224.79 153.67 0)
-      (effects (font (size 1.27 1.27)) hide)
-    )
+    (property "Footprint" "TestPoint:TestPoint_Pad_D1.0mm" (id 2) (at 224.79 153.67 0)
+      (effects (font (size 1.27 1.27)) hide)
+    )

Commit message: friday changes
Connections:
- net Ball_Deploy: no longer names the net of U10.20 (IO_15)
- no-connect marks 2 -> 3
Other:
- note removed: "snagging this off here saves mainboard IO"
Changed lines of the file:
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@@
   (junction (at 209.55 158.75) (diameter 0) (color 0 0 0 0)
   )
+  (no_connect (at 96.52 162.56))
   (no_connect (at 344.17 151.13))
   (no_connect (at 92.71 49.53))
@@
     (effects (font (size 2.54 2.54) (thickness 0.508) bold) (justify left bottom))
   )
-  (text "snagging this off here saves mainboard IO" (at 95.25 165.1 0)
-    (effects (font (size 1.27 1.27)) (justify left bottom))
-  )
   (text "output ->" (at 114.3 144.78 0)
     (effects (font (size 1.27 1.27)) (justify left bottom))
@@
     (effects (font (size 1.27 1.27)) (justify right bottom))
   )
-  (hierarchical_label "Ball_Deploy" (shape input) (at 96.52 162.56 0)
-    (effects (font (size 1.27 1.27)) (justify left))
-  )
   (hierarchical_label "SCL" (shape input) (at 24.13 104.14 180)
