File: magnetotorquer-driver.kicad_sch (KiCad schematic)
At the start: 62 parts, among them U10 MAX7311AAG+, U11 MCP47FVB24-E/MQ, U12 ALM2402QPWPRQ1, U13 OPA340MDBVTEP, U14 AD7091R-5BCPZ-RL7, U15 ALM2402QPWPRQ1

Commit message: updates
Parts:
- gave numbers to parts that had none: 1
Other:
- note added: "add i/p resistors to all sense line destinations!!"
- note added: "make FP for this guys' pads larger!!@!"
- note removed: "any way to get a super accurate 5V reference? always a dropout voltage"
Changed lines of the file:
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@@
+    (effects (font (size 1.27 1.27)) (justify left bottom))
+  )
+  (text "add i/p resistors to all sense line destinations!!"
+    (at 287.02 207.01 0)
     (effects (font (size 1.27 1.27)) (justify left bottom))
   )
@@
     (effects (font (size 1.27 1.27)) (justify left bottom))
   )
+  (text "make FP for this guys' pads larger!!@!" (at 92.71 57.15 0)
+    (effects (font (size 1.27 1.27)) (justify left bottom))
+  )
   (text "0-5Vout" (at 147.32 39.37 0)
     (effects (font (size 1.27 1.27)) (justify left bottom))
@@
   )
   (text "0-2.5Vout" (at 63.5 29.21 0)
-    (effects (font (size 1.27 1.27)) (justify left bottom))
-  )
-  (text "any way to get a super accurate 5V reference?\nalways a dropout voltage "
-    (at 55.88 92.71 0)
     (effects (font (size 1.27 1.27)) (justify left bottom))
   )
@@
   (symbol (lib_id "Device:R_US") (at 316.23 168.91 180) (unit 1)
     (in_bom yes) (on_board yes) (fields_autoplaced)
-    (property "Reference" "R?" (id 0) (at 318.77 167.6399 0)
+    (property "Reference" "R104" (id 0) (at 318.77 167.6399 0)
       (effects (font (size 1.27 1.27)) (justify right))
     )
@@
   (symbol (lib_id "power:GND") (at 232.41 60.96 0) (unit 1)
     (in_bom yes) (on_board yes) (fields_autoplaced)
-    (property "Reference" "#PWR?" (id 0) (at 232.41 67.31 0)
+    (property "Reference" "#PWR0133" (id 0) (at 232.41 67.31 0)
       (effects (font (size 1.27 1.27)) hide)
     )
@@
   (symbol (lib_id "power:+3.3V") (at 316.23 165.1 0) (unit 1)
     (in_bom yes) (on_board yes) (fields_autoplaced)
-    (property "Reference" "#PWR?" (id 0) (at 316.23 168.91 0)
+    (property "Reference" "#PWR0132" (id 0) (at 316.23 168.91 0)
       (effects (font (size 1.27 1.27)) hide)
     )
@@
   (symbol (lib_id "power:GND") (at 331.47 62.23 0) (unit 1)
     (in_bom yes) (on_board yes) (fields_autoplaced)
-    (property "Reference" "#PWR?" (id 0) (at 331.47 68.58 0)
-      (effects (font (size 1.27 1.27)) hide)
-    )
+    (property "Reference" "#PWR0134" (id 0) (at 331.47 68.58 0)
+      (effects (font (size 1.27 1.27)) hide)
+    )
