File: I2C-Protection.kicad_sch (KiCad schematic)
At the start: 22 parts

Commit message: majority of routing completed
Parts:
- added TP15, TP16, TP17, TP18: TestPoint, TestPoint:TestPoint_Pad_2.5x2.5mm, symbol Connector:TestPoint
- Q5, Q7: renamed from Q?; Flight BSS138DWQ-7 -> (none); Manufacturer_Name Diodes Incorporated -> (none); Manufacturer_Part_Number BSS138DWQ-7 -> (none); Proto BSS138DWQ-7 -> (none)
- Q6, Q8: renamed from Q?; Flight MMDT5551-7-F -> (none)
- Q8: renamed from Q?; Flight MBT2222ADW1T1G -> (none); Manufacturer_Name ON Semiconductor -> (none); Manufacturer_Part_Number MBT2222ADW1T1G -> (none); Proto MBT2222ADW1T1G -> (none)
- R47, R52: renamed from R?; value 100K -> 100k
- R49, R50, R54, R55: renamed from R?; value 10K -> 10k
- gave numbers to parts that had none: 9
Connections:
- net GND: now also Q5.1 (S2), Q7.1 (S2); no longer Q5.4 (S1), Q7.4 (S1)
- net SCL_IN: now also Q6.6 (C1), TP15.1; no longer Q6.3 (C2)
- net SCL_PROT: now also Q6.1 (E1), TP17.1; no longer Q6.4 (E2)
- net SDA_IN: now also Q8.6 (C1), TP16.1; no longer Q8.3 (C2)
- net SDA_PROT: now also Q8.1 (E1), TP18.1; no longer Q8.4 (E2)
- net at Q7.2 (G2), R52.2: now also Q7.6 (D1); no longer Q7.3 (D2)
- net at C48.1, R56.2: now also Q7.2 (G2); no longer Q7.5 (G1)
- net at C47.1, R51.2: now also Q5.2 (G2); no longer Q5.5 (G1)
- net at Q5.6 (D1), R48.2, R49.2: now also Q6.2 (B1); no longer Q6.5 (B2)
- net at Q5.2 (G2), R47.2: now also Q5.6 (D1); no longer Q5.3 (D2)
- net at Q7.6 (D1), R53.2, R54.2: now also Q8.2 (B1); no longer Q8.5 (B2)

Commit message: design updates
Parts:
- TP30: renamed from TP15; footprint TestPoint:TestPoint_Pad_2.5x2.5mm -> TestPoint:TestPoint_Pad_D1.0mm
- TP31: renamed from TP16; footprint TestPoint:TestPoint_Pad_2.5x2.5mm -> TestPoint:TestPoint_Pad_D1.0mm
- TP32: renamed from TP17; footprint TestPoint:TestPoint_Pad_2.5x2.5mm -> TestPoint:TestPoint_Pad_D1.0mm
- TP33: renamed from TP18; footprint TestPoint:TestPoint_Pad_2.5x2.5mm -> TestPoint:TestPoint_Pad_D1.0mm
- renumbered C47 to C70, C48 to C71, Q5 to Q13, Q6 to Q14, Q7 to Q15, Q8 to Q16, R47 to R77, R48 to R78, R49 to R79, R50 to R80, R51 to R81, R52 to R82, R53 to R83, R54 to R84, R55 to R85, R56 to R86, R57 to R87, R58 to R88
Connections:
- net GND: now also Q13.4 (S1), Q15.4 (S1); no longer Q13.1 (S2), Q15.1 (S2)
- net SCL_IN: now also Q14.3 (C2); no longer Q14.6 (C1)
- net SCL_PROT: now also Q14.4 (E2); no longer Q14.1 (E1)
- net SDA_IN: now also Q16.3 (C2); no longer Q16.6 (C1)
- net SDA_PROT: now also Q16.4 (E2); no longer Q16.1 (E1)
- net at C71.1, R86.2: now also Q15.5 (G1); no longer Q15.2 (G2)
- net at Q15.2 (G2), R82.2: now also Q15.3 (D2); no longer Q15.6 (D1)
- net at C70.1, R81.2: now also Q13.5 (G1); no longer Q13.2 (G2)
- net at Q13.6 (D1), R78.2, R79.2: now also Q14.5 (B2); no longer Q14.2 (B1)
- net at Q13.2 (G2), R77.2: now also Q13.3 (D2); no longer Q13.6 (D1)
- net at Q15.6 (D1), R83.2, R84.2: now also Q16.5 (B2); no longer Q16.2 (B1)

Commit message: updates
Parts:
- C70, C71: symbol mainboard-rescue:C-Device-mainboard-rescue -> Device:C
- R77, R78, R79, R80, R81, R82, R83, R84, R85, R86, R87, R88: symbol mainboard-rescue:R_US-Device-mainboard-rescue -> Device:R_US
Changed lines of the file:
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@@
     (effects (font (size 1.27 1.27)) (justify right))
   )
-  (symbol (lib_id "mainboard-rescue:R_US-Device-mainboard-rescue") (at 172.72 78.74 0) (unit 1)
+  (symbol (lib_id "Device:R_US") (at 172.72 78.74 0) (unit 1)
     (in_bom yes) (on_board yes)
     (property "Reference" "R85" (id 0) (at 174.4472 77.5716 0)
@@
     (pin "5")
   )
-  (symbol (lib_id "mainboard-rescue:C-Device-mainboard-rescue") (at 130.81 118.11 0) (unit 1)
+  (symbol (lib_id "Device:C") (at 130.81 118.11 0) (unit 1)
     (in_bom yes) (on_board yes)
     (property "Reference" "C70" (id 0) (at 133.731 116.9416 0)
@@
     (pin "5")
   )
-  (symbol (lib_id "mainboard-rescue:R_US-Device-mainboard-rescue") (at 119.38 93.98 270) (unit 1)
+  (symbol (lib_id "Device:R_US") (at 119.38 93.98 270) (unit 1)
     (in_bom yes) (on_board yes)
     (property "Reference" "R78" (id 0) (at 118.11 88.9 90))
@@
     (pin "2")
   )
-  (symbol (lib_id "mainboard-rescue:R_US-Device-mainboard-rescue") (at 130.81 78.74 0) (unit 1)
+  (symbol (lib_id "Device:R_US") (at 130.81 78.74 0) (unit 1)
     (in_bom yes) (on_board yes)
     (property "Reference" "R80" (id 0) (at 132.5372 77.5716 0)
@@
     (pin "1")
   )
-  (symbol (lib_id "mainboard-rescue:R_US-Device-mainboard-rescue") (at 130.81 107.95 0) (unit 1)
+  (symbol (lib_id "Device:R_US") (at 130.81 107.95 0) (unit 1)
     (in_bom yes) (on_board yes)
     (property "Reference" "R81" (id 0) (at 132.5372 106.7816 0)
@@
     (pin "2")
   )
-  (symbol (lib_id "mainboard-rescue:R_US-Device-mainboard-rescue") (at 125.73 72.39 0) (unit 1)
+  (symbol (lib_id "Device:R_US") (at 125.73 72.39 0) (unit 1)
     (in_bom yes) (on_board yes)
     (property "Reference" "R79" (id 0) (at 124.0282 71.2216 0)
@@
     (pin "5")
   )
-  (symbol (lib_id "mainboard-rescue:R_US-Device-mainboard-rescue") (at 167.64 72.39 0) (unit 1)
+  (symbol (lib_id "Device:R_US") (at 167.64 72.39 0) (unit 1)
     (in_bom yes) (on_board yes)
     (property "Reference" "R84" (id 0) (at 165.9382 71.2216 0)
@@
     (pin "2")
   )
-  (symbol (lib_id "mainboard-rescue:R_US-Device-mainboard-rescue") (at 118.11 105.41 0) (unit 1)
+  (symbol (lib_id "Device:R_US") (at 118.11 105.41 0) (unit 1)
     (in_bom yes) (on_board yes)
     (property "Reference" "R77" (id 0) (at 114.3 102.87 0)
@@
     (pin "2")
   )
-  (symbol (lib_id "mainboard-rescue:C-Device-mainboard-rescue") (at 172.72 118.11 0) (unit 1)
+  (symbol (lib_id "Device:C") (at 172.72 118.11 0) (unit 1)
     (in_bom yes) (on_board yes)
     (property "Reference" "C71" (id 0) (at 175.641 116.9416 0)
@@
     (pin "1")
   )
-  (symbol (lib_id "mainboard-rescue:R_US-Device-mainboard-rescue") (at 215.9 116.84 270) (unit 1)
+  (symbol (lib_id "Device:R_US") (at 215.9 116.84 270) (unit 1)
     (in_bom yes) (on_board yes)
     (property "Reference" "R87" (id 0) (at 212.09 115.57 90))
@@
     (pin "5")
   )
-  (symbol (lib_id "mainboard-rescue:R_US-Device-mainboard-rescue") (at 215.9 120.65 270) (unit 1)
+  (symbol (lib_id "Device:R_US") (at 215.9 120.65 270) (unit 1)
     (in_bom yes) (on_board yes)
     (property "Reference" "R88" (id 0) (at 212.09 119.38 90))
@@
     (pin "2")
   )
-  (symbol (lib_id "mainboard-rescue:R_US-Device-mainboard-rescue") (at 160.02 105.41 0) (unit 1)
+  (symbol (lib_id "Device:R_US") (at 160.02 105.41 0) (unit 1)
     (in_bom yes) (on_board yes)
     (property "Reference" "R82" (id 0) (at 156.21 102.87 0)
@@
     (pin "2")
   )
-  (symbol (lib_id "mainboard-rescue:R_US-Device-mainboard-rescue") (at 161.29 93.98 270) (unit 1)
+  (symbol (lib_id "Device:R_US") (at 161.29 93.98 270) (unit 1)
     (in_bom yes) (on_board yes)
     (property "Reference" "R83" (id 0) (at 160.02 88.9 90))
@@
     (pin "1")
   )
-  (symbol (lib_id "mainboard-rescue:R_US-Device-mainboard-rescue") (at 172.72 107.95 0) (unit 1)
+  (symbol (lib_id "Device:R_US") (at 172.72 107.95 0) (unit 1)
     (in_bom yes) (on_board yes)
     (property "Reference" "R86" (id 0) (at 174.4472 106.7816 0)
