File: IMU.kicad_sch (KiCad schematic)
At the start: 31 parts

Commit message: majority of routing completed
Parts:
- C14, C15: renamed from C?; footprint Capacitor_SMD:C_0603_1608Metric -> Capacitor_SMD:C_0805_2012Metric
- R20: renamed from R?; value 10k -> 100k
- U6, U7: renamed from U?; footprint payload-interface-boardI:MMC5983MA -> payload-interface-board:MMC5983MA
- U8, U9: renamed from U?; footprint payload-interface-boardI:MXC6655XA -> payload-interface-board:MXC6655XA
- gave numbers to parts that had none: 24
Other:
- note added: "i2c mux addr = 0x7A"
- note removed: "i2c mux addr = 0x72"

Commit message: updates
Parts:
- C14, C15, C16, C17, C18, C19, C20, C21, C22, C23, C24, C25, C26, C27, C28: symbol mainboard-rescue:C-Device-mainboard-rescue -> Device:C
- R16, R17, R18, R19, R20, R21, R22, R23, R24: symbol mainboard-rescue:R_US-Device-mainboard-rescue -> Device:R_US
Changed lines of the file:
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@@
     (pin "1")
   )
-  (symbol (lib_id "mainboard-rescue:C-Device-mainboard-rescue") (at 43.18 106.68 0) (unit 1)
+  (symbol (lib_id "Device:C") (at 43.18 106.68 0) (unit 1)
     (in_bom yes) (on_board yes)
     (property "Reference" "C17" (id 0) (at 46.101 105.5116 0)
@@
     (pin "9")
   )
-  (symbol (lib_id "mainboard-rescue:C-Device-mainboard-rescue") (at 104.14 43.18 0) (unit 1)
+  (symbol (lib_id "Device:C") (at 104.14 43.18 0) (unit 1)
     (in_bom yes) (on_board yes)
     (property "Reference" "C24" (id 0) (at 107.061 42.0116 0)
@@
     (pin "2")
   )
-  (symbol (lib_id "mainboard-rescue:R_US-Device-mainboard-rescue") (at 146.05 157.48 0) (unit 1)
+  (symbol (lib_id "Device:R_US") (at 146.05 157.48 0) (unit 1)
     (in_bom yes) (on_board yes)
     (property "Reference" "R23" (id 0) (at 147.7772 156.3116 0)
@@
     (pin "9")
   )
-  (symbol (lib_id "mainboard-rescue:C-Device-mainboard-rescue") (at 31.75 106.68 0) (unit 1)
+  (symbol (lib_id "Device:C") (at 31.75 106.68 0) (unit 1)
     (in_bom yes) (on_board yes)
     (property "Reference" "C14" (id 0) (at 34.671 105.5116 0)
@@
     (pin "1")
   )
-  (symbol (lib_id "mainboard-rescue:C-Device-mainboard-rescue") (at 157.48 45.72 0) (unit 1)
+  (symbol (lib_id "Device:C") (at 157.48 45.72 0) (unit 1)
     (in_bom yes) (on_board yes)
     (property "Reference" "C28" (id 0) (at 160.401 44.5516 0)
@@
     (pin "1")
   )
-  (symbol (lib_id "mainboard-rescue:R_US-Device-mainboard-rescue") (at 138.43 154.94 0) (unit 1)
+  (symbol (lib_id "Device:R_US") (at 138.43 154.94 0) (unit 1)
     (in_bom yes) (on_board yes)
     (property "Reference" "R22" (id 0) (at 140.1572 153.7716 0)
@@
     (pin "2")
   )
-  (symbol (lib_id "mainboard-rescue:C-Device-mainboard-rescue") (at 53.34 33.02 0) (unit 1)
+  (symbol (lib_id "Device:C") (at 53.34 33.02 0) (unit 1)
     (in_bom yes) (on_board yes)
     (property "Reference" "C20" (id 0) (at 56.261 31.8516 0)
@@
     (pin "1")
   )
-  (symbol (lib_id "mainboard-rescue:R_US-Device-mainboard-rescue") (at 110.49 144.78 0) (unit 1)
+  (symbol (lib_id "Device:R_US") (at 110.49 144.78 0) (unit 1)
     (in_bom yes) (on_board yes)
     (property "Reference" "R18" (id 0) (at 112.2172 143.6116 0)
@@
     (pin "2")
   )
-  (symbol (lib_id "mainboard-rescue:R_US-Device-mainboard-rescue") (at 124.46 179.07 0) (unit 1)
+  (symbol (lib_id "Device:R_US") (at 124.46 179.07 0) (unit 1)
     (in_bom yes) (on_board yes)
     (property "Reference" "R20" (id 0) (at 126.1872 177.9016 0)
@@
     (pin "1")
   )
-  (symbol (lib_id "mainboard-rescue:R_US-Device-mainboard-rescue") (at 55.88 161.29 0) (unit 1)
+  (symbol (lib_id "Device:R_US") (at 55.88 161.29 0) (unit 1)
     (in_bom yes) (on_board yes)
     (property "Reference" "R16" (id 0) (at 49.53 160.02 0)
@@
     (pin "2")
   )
-  (symbol (lib_id "mainboard-rescue:C-Device-mainboard-rescue") (at 53.34 110.49 0) (unit 1)
+  (symbol (lib_id "Device:C") (at 53.34 110.49 0) (unit 1)
     (in_bom yes) (on_board yes)
     (property "Reference" "C21" (id 0) (at 56.261 109.3216 0)
@@
     (pin "1")
   )
-  (symbol (lib_id "mainboard-rescue:R_US-Device-mainboard-rescue") (at 60.96 161.29 0) (unit 1)
+  (symbol (lib_id "Device:R_US") (at 60.96 161.29 0) (unit 1)
     (in_bom yes) (on_board yes)
     (property "Reference" "R17" (id 0) (at 62.6872 160.1216 0)
@@
     (pin "1")
   )
-  (symbol (lib_id "mainboard-rescue:C-Device-mainboard-rescue") (at 54.61 52.07 0) (unit 1)
+  (symbol (lib_id "Device:C") (at 54.61 52.07 0) (unit 1)
     (in_bom yes) (on_board yes)
     (property "Reference" "C22" (id 0) (at 57.531 50.9016 0)
@@
     (pin "2")
   )
-  (symbol (lib_id "mainboard-rescue:C-Device-mainboard-rescue") (at 33.02 48.26 0) (unit 1)
+  (symbol (lib_id "Device:C") (at 33.02 48.26 0) (unit 1)
     (in_bom yes) (on_board yes)
     (property "Reference" "C15" (id 0) (at 35.941 47.0916 0)
@@
     (pin "2")
   )
-  (symbol (lib_id "mainboard-rescue:C-Device-mainboard-rescue") (at 44.45 48.26 0) (unit 1)
+  (symbol (lib_id "Device:C") (at 44.45 48.26 0) (unit 1)
     (in_bom yes) (on_board yes)
     (property "Reference" "C18" (id 0) (at 47.371 47.0916 0)
@@
     (pin "2")
   )
-  (symbol (lib_id "mainboard-rescue:C-Device-mainboard-rescue") (at 114.3 49.53 0) (unit 1)
+  (symbol (lib_id "Device:C") (at 114.3 49.53 0) (unit 1)
     (in_bom yes) (on_board yes)
     (property "Reference" "C26" (id 0) (at 117.221 48.3616 0)
@@
     (pin "1")
   )
-  (symbol (lib_id "mainboard-rescue:C-Device-mainboard-rescue") (at 52.07 91.44 0) (unit 1)
+  (symbol (lib_id "Device:C") (at 52.07 91.44 0) (unit 1)
     (in_bom yes) (on_board yes)
     (property "Reference" "C19" (id 0) (at 54.991 90.2716 0)
@@
     (pin "1")
   )
-  (symbol (lib_id "mainboard-rescue:C-Device-mainboard-rescue") (at 113.03 107.95 0) (unit 1)
+  (symbol (lib_id "Device:C") (at 113.03 107.95 0) (unit 1)
     (in_bom yes) (on_board yes)
     (property "Reference" "C25" (id 0) (at 115.951 106.7816 0)
@@
     (pin "1")
   )
-  (symbol (lib_id "mainboard-rescue:C-Device-mainboard-rescue") (at 102.87 101.6 0) (unit 1)
+  (symbol (lib_id "Device:C") (at 102.87 101.6 0) (unit 1)
     (in_bom yes) (on_board yes)
     (property "Reference" "C23" (id 0) (at 105.791 100.4316 0)
@@
     (pin "9")
   )
-  (symbol (lib_id "mainboard-rescue:R_US-Device-mainboard-rescue") (at 125.73 149.86 0) (unit 1)
+  (symbol (lib_id "Device:R_US") (at 125.73 149.86 0) (unit 1)
     (in_bom yes) (on_board yes)
     (property "Reference" "R21" (id 0) (at 127.4572 148.6916 0)
@@
     (pin "1")
   )
-  (symbol (lib_id "mainboard-rescue:C-Device-mainboard-rescue") (at 156.21 104.14 0) (unit 1)
+  (symbol (lib_id "Device:C") (at 156.21 104.14 0) (unit 1)
     (in_bom yes) (on_board yes)
     (property "Reference" "C27" (id 0) (at 159.131 102.9716 0)
@@
     (pin "2")
   )
-  (symbol (lib_id "mainboard-rescue:R_US-Device-mainboard-rescue") (at 153.67 160.02 0) (unit 1)
+  (symbol (lib_id "Device:R_US") (at 153.67 160.02 0) (unit 1)
     (in_bom yes) (on_board yes)
     (property "Reference" "R24" (id 0) (at 155.3972 158.8516 0)
@@
     (pin "1")
   )
-  (symbol (lib_id "mainboard-rescue:C-Device-mainboard-rescue") (at 40.64 158.75 0) (unit 1)
+  (symbol (lib_id "Device:C") (at 40.64 158.75 0) (unit 1)
     (in_bom yes) (on_board yes)
     (property "Reference" "C16" (id 0) (at 43.561 157.5816 0)
@@
     (pin "1")
   )
-  (symbol (lib_id "mainboard-rescue:R_US-Device-mainboard-rescue") (at 118.11 147.32 0) (unit 1)
+  (symbol (lib_id "Device:R_US") (at 118.11 147.32 0) (unit 1)
     (in_bom yes) (on_board yes)
     (property "Reference" "R19" (id 0) (at 119.8372 146.1516 0)
