File: Sense_Amp.kicad_sch (KiCad schematic)
At the start: 3 parts, among them U20 INA240A3EDRQ1

Commit message: design updates
Parts:
- renumbered C59 to C52, C60 to C53, U20 to U17
Changed lines of the file:
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@@
     (effects (font (size 1.27 1.27)) (justify right))
   )
-  (symbol (lib_id "Device:C") (at 121.92 71.12 0)
+  (symbol (lib_id "Device:C") (at 121.92 71.12 0) (unit 1)
     (in_bom yes) (on_board yes) (fields_autoplaced)
-    (property "Reference" "C59" (id 0) (at 124.841 70.2115 0)
+    (property "Reference" "C52" (id 0) (at 124.841 70.2115 0)
       (effects (font (size 1.27 1.27)) (justify left))
     )
@@
     (pin "2")
   )
-  (symbol (lib_id "power:GND") (at 144.78 109.22 0)
+  (symbol (lib_id "power:GND") (at 144.78 109.22 0) (unit 1)
     (in_bom yes) (on_board yes) (fields_autoplaced)
-    (property "Reference" "#PWR058" (id 0) (at 144.78 115.57 0)
+    (property "Reference" "#PWR049" (id 0) (at 144.78 115.57 0)
       (effects (font (size 1.27 1.27)) hide)
     )
@@
     (pin "1")
   )
-  (symbol (lib_id "Device:C") (at 130.81 71.12 0)
+  (symbol (lib_id "Device:C") (at 130.81 71.12 0) (unit 1)
     (in_bom yes) (on_board yes) (fields_autoplaced)
-    (property "Reference" "C60" (id 0) (at 133.731 70.2115 0)
+    (property "Reference" "C53" (id 0) (at 133.731 70.2115 0)
       (effects (font (size 1.27 1.27)) (justify left))
     )
@@
     (pin "2")
   )
-  (symbol (lib_id "Amplifier_Current:INA240A3PW") (at 147.32 97.79 0)
+  (symbol (lib_id "Amplifier_Current:INA240A3PW") (at 147.32 97.79 0) (unit 1)
     (in_bom yes) (on_board yes)
-    (property "Reference" "U20" (id 0) (at 152.4 91.44 0))
+    (property "Reference" "U17" (id 0) (at 152.4 91.44 0))
     (property "Value" "INA240A3EDRQ1" (id 1) (at 157.48 93.98 0))
     (property "Footprint" "Package_SO:SOIC-8_3.9x4.9mm_P1.27mm" (id 2) (at 147.32 114.3 0)
@@
     (pin "8")
   )
-  (symbol (lib_id "power:GND") (at 121.92 76.2 0)
+  (symbol (lib_id "power:GND") (at 121.92 76.2 0) (unit 1)
     (in_bom yes) (on_board yes) (fields_autoplaced)
-    (property "Reference" "#PWR057" (id 0) (at 121.92 82.55 0)
+    (property "Reference" "#PWR048" (id 0) (at 121.92 82.55 0)
       (effects (font (size 1.27 1.27)) hide)
     )

Commit message: updates
Parts:
- U17: symbol Amplifier_Current:INA240A3PW -> FP-Interface-Card:INA240AxxD
Connections:
- net GND: now also U17.2 (GND), U17.3 (REF2); no longer U17.1 (GND), U17.7 (REF1)
- net Sense_+: now also U17.8 (+); no longer U17.2 (+)
- net Sense_-: now also U17.1 (-); no longer U17.3 (-)
- net Sense_Out: now also U17.5; no longer U17.8
- net V+: now also U17.7 (REF1); no longer U17.5 (V+)
Changed lines of the file:
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@@
+    (stroke (width 0) (type default) (color 0 0 0 0))
+  )
+  (wire (pts (xy 144.78 106.68) (xy 144.78 109.22))
     (stroke (width 0) (type default) (color 0 0 0 0))
   )
   (wire (pts (xy 121.92 67.31) (xy 121.92 66.04))
-    (stroke (width 0) (type default) (color 0 0 0 0))
-  )
-  (wire (pts (xy 149.86 106.68) (xy 144.78 106.68))
     (stroke (width 0) (type default) (color 0 0 0 0))
   )
@@
     (stroke (width 0) (type default) (color 0 0 0 0))
   )
-  (wire (pts (xy 144.78 106.68) (xy 144.78 109.22))
+  (wire (pts (xy 149.86 106.68) (xy 158.75 106.68))
     (stroke (width 0) (type default) (color 0 0 0 0))
   )
@@
     (stroke (width 0) (type default) (color 0 0 0 0))
   )
+  (wire (pts (xy 144.78 106.68) (xy 147.32 106.68))
+    (stroke (width 0) (type default) (color 0 0 0 0))
+  )
+  (wire (pts (xy 147.32 105.41) (xy 147.32 106.68))
+    (stroke (width 0) (type default) (color 0 0 0 0))
+  )
   (wire (pts (xy 147.32 60.96) (xy 144.78 60.96))
     (stroke (width 0) (type default) (color 0 0 0 0))
@@
     (stroke (width 0) (type default) (color 0 0 0 0))
   )
-  (wire (pts (xy 147.32 105.41) (xy 147.32 107.95))
-    (stroke (width 0) (type default) (color 0 0 0 0))
-  )
   (wire (pts (xy 121.92 76.2) (xy 130.81 76.2))
-    (stroke (width 0) (type default) (color 0 0 0 0))
-  )
-  (wire (pts (xy 147.32 107.95) (xy 158.75 107.95))
     (stroke (width 0) (type default) (color 0 0 0 0))
   )
@@
     (effects (font (size 1.27 1.27)) (justify left bottom))
   )
-  (hierarchical_label "V+" (shape input) (at 158.75 107.95 0)
+  (hierarchical_label "V+" (shape input) (at 158.75 106.68 0)
     (effects (font (size 1.27 1.27)) (justify left))
   )
@@
     (pin "2")
   )
-  (symbol (lib_id "Amplifier_Current:INA240A3PW") (at 147.32 97.79 0) (unit 1)
+  (symbol (lib_id "FP-Interface-Card:INA240AxxD") (at 147.32 97.79 0) (unit 1)
     (in_bom yes) (on_board yes)
     (property "Reference" "U17" (id 0) (at 152.4 91.44 0))
