File: hardware/revA/5V_amp.kicad_sch (KiCad schematic)
At the start: 6 parts, among them U22 OPA340MDBVTEP

Commit message: working revB
Parts:
- removed C65, C66: 0.1uF, Capacitor_SMD:C_0603_1608Metric, symbol Device:C
- removed TP28: TestPoint, TestPoint:TestPoint_Pad_D1.0mm, symbol Connector:TestPoint
- added R67: 33, symbol Device:R_US
Connections:
- net OUT_5V: now also R67.2; no longer RN2.1, U22.1
- new net: R67.1, RN2.1, U22.1
Other:
- company: (none) -> Sierra Lobo INC
- moved on the sheet: RN2
