File: hardware/revA/Blank-Card-Default.kicad_sch (KiCad schematic)
At the start: 39 parts, among them J3 ZX62-AB-5PA(31), Q1 BC847BM3T5G, Q2 BC847BM3T5G, Q3 BC847BM3T5G, Q4 BC847BM3T5G, SW1 SW_Push_SPST, U2 AP2161W

Commit message: working revB
Other:
- company: (none) -> Sierra Lobo INC
