File: hardware/revA/FP Interface Card.kicad_sch (KiCad schematic)
At the start: 27 parts, among them J1 T1M-10-F-SV-L, J4 T1M-6-F-SV-L, J5 T1M-10-F-SV-L, P1 Card Edge for HSEC8-160-01-S-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, Q17 MMBT4401-7-F, Q18 MMBT4401-7-F, Q19 IRF7404TRPBF, Q22 MMBT4401-7-F, Q23 IRF7404TRPBF, U24 RockBlock_9603, U26 LTC4307

Commit message: working revB
Parts:
- removed J4: T1M-6-F-SV-L, payload-interface-board:SAMTEC_T1M-06-F-SV-L, symbol Connector_Generic:Conn_01x06
- removed R105, R99: 100k, Resistor_SMD:R_0603_1608Metric, symbol Device:R_US
- added C32 (x2): 0.1uF, Capacitor_SMD:C_0603_1608Metric, symbol Device:C
- added C35: 10uF, Capacitor_SMD:C_0805_2012Metric, symbol Device:C
- added Q25: MMBT4401-7-F, Package_TO_SOT_SMD:SOT-23, symbol Device:Q_NPN_BEC
- added R16: 10k, symbol Device:R_US
- added R17: 10k, Resistor_SMD:R_0603_1608Metric, symbol Device:R_US
- added R18, R19, R20: R_US, symbol Device:R_US
- added R21, R22, R23, R24, R26, R27, R28, R29, R45, R46, R72, R73, R74, R75, R76: 1k, symbol Device:R_US
- added U3: imu-stamp-revA, payload-interface-board:imu-stamp-revA-SMD, symbol FP-Interface-Card:imu-stamp-revA
- added U4, U5: SN74LVCH245APWR, Package_SO:TSSOP-20_4.4x6.5mm_P0.65mm, symbol FP-Interface-Card:SN74LVCH245APWR
- R44: value 100k -> 1k; footprint Resistor_SMD:R_0603_1608Metric -> (none)
- R94: value 100k -> 10k
- R95, R96, R97, R98: value 0 -> 1k; footprint Resistor_SMD:R_0603_1608Metric -> (none)
Connections:
- net AGND is gone; now on net GND: P1.71 (Pin_71)
- net H1-26 is gone; now on net +3V3: P1.58 (Pin_58)
- net Level Shifter 6/io_hi is gone; now on net GND: R95.1, R96.1
- net P_RESET is gone; now on net H1-6: J5.4 (Pin_4)
- net SERVO_PWR_CTRL is gone; now on net H1-5: J5.7 (Pin_7)
- net +3V3: now also C32.1, C32.1, C35.1, R16.1, R24.2, U3.1 (VCC), U4.20 (V_{CC}), U5.20 (V_{CC})
- net GND: now also R97.2, R98.2, C32.2, C32.2, C35.2, Q25.2 (E), R20.2, R26.2, R27.2, R28.2, R29.2, R45.2, R46.2, R73.1, R75.1, R76.1, U3.10 (GND), U3.2 (GND), U3.9 (GND), U4.10 (GND), U5.10 (GND); no longer R44.2
- net H1-17: now also U4.14 (B5)
- net H1-18: now also R21.1
- net H1-19: now also U4.18 (B1)
- net H1-20: now also R22.1
- net H1-39: now also U4.16 (B3)
- net H1-40: now also R74.1
- net H1-8: no longer R44.1, R89.1
- net RB_RxD: now also U5.4 (A3); no longer R95.2, R97.2
- net RB_TxD: now also R72.2; no longer R96.2, R98.2
- net SCL_IMU: now also U3.3 (SCL)
- net SDA_IMU: now also U3.4 (SDA)
- net H1-51 renamed SEP1_RET
- net H1-52 renamed SEP2_RET
- net H2-51 renamed SEP3_RET
- net H2-52 renamed SEP4_RET
- net I2C-Protection-1/SCL_IN renamed SCL_PIB
- net I2C-Protection-1/SDA_IN renamed SDA_PIB
- net Level Shifter 5/io_hi: no longer names the net of R97.1
- net Level Shifter 5/io_hi: now also U5.1 (DIR); no longer R98.1
- net PAYLOAD_5V renamed 5V_PYLD
- net PAYLOAD_PWR_SW: no longer names the net of Q22.1 (B), R106.2
- net P_RXD renamed PYLD_RXD
- net PYLD_RXD: now also U5.2 (A1)
- net P_TXD renamed PYLD_TXD
- net PYLD_TXD: now also R23.2
- net RB_PWR_SW_B: no longer names the net of Q18.1 (B), R100.2
- net ~{BUS_RESET} renamed ~{RESET}
- new net: R45.1, U4.8 (A7)
- new net: R18.1, U3.6 (XOR_REF)
- new net: R18.2, R19.1, U3.7 (XORL2)
- new net: R96.2, U5.11 (B8)
- new net: Q25.1 (B), R17.2
- new net: R44.1, U4.6 (A5)
- new net: R29.1, U4.3 (A2)
- new net: R72.1, U4.4 (A3)
- new net: R95.2, U5.12 (B7)
- new net: R76.2, U5.13 (B6)
- new net: R21.2, U5.14 (B5)
- new net: R75.2, U5.15 (B4)
- new net: R74.2, U5.16 (B3)
- new net: R73.2, U5.17 (B2)
- new net: R22.2, U5.18 (B1)
- new net: R98.1, U5.19 (~{OE})
- new net: R26.1, U4.19 (~{OE})
- new net: Q25.3 (C), R16.2, U3.5 (EN)
- new net: R19.2, R20.1, U3.8 (XORL1)
- new net: R23.1, U4.2 (A1)
- new net: R27.1, U4.7 (A6)
- new net: R28.1, U4.5 (A4)
- new net: R24.1, U4.1 (DIR)
- new net: R46.1, U4.9 (A8)
- new net PICO_RxD: U5.6 (A5)
- new net PICO_TxD: R44.2
- new net ~{IMU_EN}: R17.1
- new net ~{RB_OnOff_IN}: R89.1
- no-connect marks 5 -> 20
Other:
- sheet Blank-Card-Default renamed Backplane Card Interface
- sheet Magnetotorquer Drivers renamed MT Drivers
- removed sheet IMU
- removed sheet Level Shifter 1
- removed sheet Level Shifter 2
- removed sheet Level Shifter 3
- removed sheet Level Shifter 4
- removed sheet Level Shifter 5
- removed sheet Level Shifter 6
- sheet MT Drivers ports: added none; removed Ball_Deploy, X+, X-, Y+, Y-, Z+, Z-
- sheet Pico ports: added Pico_Rx, Pico_Tx; removed I2C1_SCL, I2C1_SDA
- note added: "Card Edge to PIB Signals"
- note added: "Edge Connector"
- note added: "I2C Buffer"
- note added: "IN"
- note added: "OUT"
- note added: "RX_MCU_2"
- note added: "RX_MCU_3"
- note added: "RX_MCU_4"
- note added: "Serial IO Buffers"
- note added: "TO FORAS PROMINEO PAYLOAD"
- note added: "TODO: CALCULATE XOR VALUE RESISTORS FOR I2C"
- note added: "TX_MCU_2"
- note added: "TX_MCU_3"
- note added: "TX_MCU_4"
- note removed: "End of CSK Bus Pins"
- note removed: "I2C PROTECTION"
- note removed: "MAGNETORQUER DRIVERS"
- note removed: "MAKE A UART PROTECTION CIRCUIT"
- note removed: "PAYLOAD LEVEL SHIFTERS"
- note removed: "PICO"
- note removed: "ROCKBLOCK LEVEL SHIFTERS & POWER SW"
- note removed: "SLI Backplane Card Default Circuitry"
- note removed: "SLI Backplane Card Default Edge Connector"
- note removed: "TO FORAS PROMINEO PAB"
- note removed: "TO MAGNETOTORQUERS"
- note removed: "UART_2_Rx"
- note removed: "UART_2_Tx"
- note removed: "UART_3_Rx"
- note removed: "UART_3_Tx"
- note removed: "USB 2.0 microB"
- note removed: "main i2c bus, pycubed processor is master."
- note removed: "mainboard PA19"
- note removed: "mainboard PC05"
- note removed: "mainboard PC06"
- note removed: "mainboard PC07"
- note removed: "mainboard PC10"
- note removed: "openMV MISO"
- note removed: "openMV MOSI"
- note removed: "openMV RST"
- moved on the sheet: C73, J1, J5, P1, Q17, Q18, Q19, Q22, Q23, R100, R101, R106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
