File: hardware/revA/Full_Bridge.kicad_sch (KiCad schematic)
At the start: 9 parts, among them U16 DRV8838DSGT

Commit message: working revB
Parts:
- removed C50: 0.1uF, Capacitor_SMD:C_0603_1608Metric, symbol Device:C
- removed C51: 4.7uF, Capacitor_SMD:C_0805_2012Metric, symbol Device:C
- R59, R60, R61: value 100 -> 1k
Other:
- company: (none) -> Sierra Lobo INC
