File: hardware/revA/I2C-Protection.kicad_sch (KiCad schematic)
At the start: 22 parts, among them Q13 BSS138DWQ-7, Q14 MMDT5551-7-F, Q15 BSS138DWQ-7, Q16 MMDT5551-7-F

Commit message: working revB
Other:
- company: (none) -> Sierra Lobo INC
