File: hardware/revA/magnetotorquer-driver.kicad_sch (KiCad schematic)
At the start: 62 parts, among them U10 MAX7311AAG+, U11 MCP47FVB24-E/MQ, U12 ALM2402QPWPRQ1, U13 OPA340MDBVTEP, U14 AD7091R-5BCPZ-RL7, U15 ALM2402QPWPRQ1

Commit message: working revB
Parts:
- removed C44: 0.1uF, Capacitor_SMD:C_0603_1608Metric, symbol Device:C
- removed R102: 100k, symbol Device:R_US
- removed R26, R27, R28, R29, R45, R46: 51, Resistor_SMD:R_0603_1608Metric, symbol Device:R_US
- removed TP10, TP11, TP12, TP13, TP2, TP3, TP5, TP6, TP9: TestPoint, TestPoint:TestPoint_Pad_D1.0mm, symbol Connector:TestPoint
- added J4: T1M-6-F-SV-L, payload-interface-board:SAMTEC_T1M-06-F-SV-L, symbol Connector_Generic:Conn_01x06
- added R65: 33, Resistor_SMD:R_0603_1608Metric, symbol Device:R_US
- added R69, R70, R71: 33, symbol Device:R_US
- R104, R25, R35, R42: value 100k -> 10k
- R30, R31, R41, R43: value 100 -> 1k
- R93: value 100k -> 33
Connections:
- net 2.5V_Vref: now also R65.2; no longer U13.1
- net SCL: now also U10.22 (SCL), U11.16 (SCL), U14.16 (SCL)
- net SDA: now also U10.23 (SDA), U11.17 (SDA), U14.15 (SDA)
- net X+: now also J4.2 (Pin_2)
- net X-: now also J4.1 (Pin_1)
- net X_Vs_5V: now also R69.1; no longer U12.2 (IN1+)
- net Y+: now also J4.4 (Pin_4)
- net Y-: now also J4.3 (Pin_3)
- net Y_Vs_5V: now also R70.1; no longer U12.4 (IN2+)
- net Z+: now also J4.6 (Pin_6)
- net Z-: now also J4.5 (Pin_5)
- net Z_Vs_5V: now also R71.1; no longer U15.2 (IN1+)
- net at U13.4 (-): now also U13.1, R65.1
- net ~{IMU_EN}: now reaches U10.20 (IO_15)
- new net: R70.2, U12.4 (IN2+)
- new net: R69.2, U12.2 (IN1+)
- new net: R71.2, U15.2 (IN1+)
- no-connect marks 3 -> 2
Other:
- note added: "2.5V generated by ADC"
- note added: "To MTs"
- note removed: "add i/p resistors to all sense line destinations!!"
- note removed: "generated by ADC"
- note removed: "make FP for this guys' pads larger!!@!"
- company: (none) -> Sierra Lobo INC
- moved on the sheet: C34, C35, C36, C37, C39, C40, C42, C43, C45, C46, R104, R32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
