File: hardware/revB/5V_amp.kicad_sch (KiCad schematic)
At the start: 4 parts, among them U22 OPA340MDBVTEP

Commit message: working revB
Parts:
- R67: value 33 -> 1k; footprint (none) -> Resistor_SMD:R_0603_1608Metric
Changed lines of the file:
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@@
       (effects (font (size 1.27 1.27)))
     )
-    (property "Value" "33" (at 151.13 87.63 90)
+    (property "Value" "1k" (at 151.13 87.63 90)
       (effects (font (size 1.27 1.27)))
     )
-    (property "Footprint" "" (at 151.384 89.154 90)
+    (property "Footprint" "Resistor_SMD:R_0603_1608Metric" (at 151.384 89.154 90)
       (effects (font (size 1.27 1.27)) hide)
     )

Commit message: working revB
Parts:
- renumbered C64 to C44, R67 to R77, RN2 to RN6, U22 to U20

Commit message: updated files
Parts:
- renumbered C44 to C42, R77 to R53, RN6 to RN10, U20 to U18

Commit message: working
Parts:
- removed C42: 0.1uF, Capacitor_SMD:C_0603_1608Metric, symbol Device:C
- removed R53: 1k, Resistor_SMD:R_0603_1608Metric, symbol Device:R_US
- removed RN10: MAX5490GC01000+T, Package_TO_SOT_SMD:SOT-23, symbol FP-Interface-Card:MAX5490GC01000+T
- removed U18: OPA340MDBVTEP, Package_TO_SOT_SMD:SOT-23-5, symbol Amplifier_Operational:OPA340NA
- added C46: 100pF, Capacitor_SMD:C_0603_1608Metric, symbol Device:C
- added R25, R26: 220k, Resistor_SMD:R_0603_1608Metric, symbol Device:R_US
- added R84: 110k, Resistor_SMD:R_0603_1608Metric, symbol Device:R_US
- added U32: LT6004CMS8#PBF, Package_SO:MSOP-8_3x3mm_P0.65mm, symbol SierraLobo:LT6004CMS8#PBF
Connections:
- net GND: now also C46.2, R26.2
- net IN_2.5V: now also R84.1
- new net: R25.1, U32.1
- new net: C46.1, R25.2, R26.1, U32.2 (-)
- new net: R84.2, U32.3 (+)
Other:
- note added: "Gain of 2 amp"
- company: Sierra Lobo INC -> (none)
- title: (none) -> Foras Promineo Payload Interface Board
