File: hardware/revB/Blank-Card-Default.kicad_sch (KiCad schematic)
At the start: 39 parts, among them J3 ZX62-AB-5PA(31), Q1 BC847BM3T5G, Q2 BC847BM3T5G, Q3 BC847BM3T5G, Q4 BC847BM3T5G, SW1 SW_Push_SPST, U2 AP2161W

Commit message: working revB
Parts:
- removed C12, C8: 0.1uF, Capacitor_SMD:C_0402_1005Metric, symbol Device:C
- removed C13: 47uF, Capacitor_SMD:C_1206_3216Metric, symbol Device:C
- removed C9: 1nF, Capacitor_SMD:C_0402_1005Metric, symbol Device:C
- removed J3: ZX62-AB-5PA(31), SLI-Backplane-Blank-Card-KiCad:ZX62-AB-5PA(31), symbol Connector:USB_B_Micro
- removed R10, R13, R6: 10k, Resistor_SMD:R_0402_1005Metric, symbol Device:R_US
- removed R5: 1Meg, Resistor_SMD:R_0402_1005Metric, symbol Device:R_US
- removed SW1: SW_Push_SPST, SLI-Backplane-Blank-Card-KiCad:EVQP7C01P, symbol Switch:SW_Push
- removed U2: AP2161W, Package_TO_SOT_SMD:SOT-23-5, symbol Power_Management:AP2161W
- removed Z1, Z2: CG0402MLU-05G, Capacitor_SMD:C_0402_1005Metric, symbol Device:Varistor
- added D208 (x2): SK68XX-EC3210R, payload-interface-board:SK6812-EC3210F-RA, symbol FP-Interface-Card:SK6812-EC321F_4
- C10: value 10uF -> 0.1uF; footprint Capacitor_SMD:C_0603_1608Metric -> Capacitor_SMD:C_0402_1005Metric
- renumbered C4 to C6, C5 to C7, C6 to C8, C7 to C9, Q4 to Q10, Q1 to Q7, Q2 to Q8, Q3 to Q9, R4 to R24, R7 to R27, R8 to R28, R9 to R29, R11 to R31, R12 to R32, R14 to R34, R15 to R35
Connections:
- net GND: now also D208.1 (VSS), D208.1 (VSS)
- net LED_VCC: now also C10.1, C11.1, D208.4 (VDD), D208.4 (VDD)
- new net: D208.2 (DOUT), D208.3 (DIN)
- new net DIN: D208.3 (DIN)
- new net DOUT: D208.2 (DOUT)
- no-connect marks 1 -> 0
Other:
- note removed: "Switch"
- note removed: "USB protection and power switch"
- note removed: "do we even need power thru usb? usb data transmission only needs a common ground"

Commit message: updated files
Parts:
- added R81: 1k, Resistor_SMD:R_0603_1608Metric, symbol Device:R_US
- D208: value SK68XX-EC3210R -> SK6805-EC3210R
- renumbered C9 to C10, C10 to C5, C11 to C6, C6 to C7, C7 to C8, C8 to C9, D2 to D4, D3 to D5, D4 to D6, D5 to D7, Q7 to Q4, Q8 to Q5, Q9 to Q6, Q10 to Q7, R27 to R13, R29 to R14, R32 to R15, R35 to R16, R24 to R17, R28 to R18, R31 to R19, R34 to R20
Connections:
- net DIN: now also R81.2; no longer D208.3 (DIN)
- new net: D208.3 (DIN), R81.1

Commit message: working
Parts:
- renumbered C7 to C10, C8 to C11, C9 to C12, C10 to C13, C5 to C8, C6 to C9, R81 to R14, R13 to R15, R14 to R16, R15 to R17, R16 to R18, R17 to R19, R18 to R20, R19 to R21, R20 to R22
Connections:
- removed net CHS: C10.2, C11.2, C12.2, C13.2, H1.1, H2.1, H3.1, H4.1
- new net: C10.2, H1.1
- new net: C11.2, H2.1
- new net: C12.2, H3.1
- new net: C13.2, H4.1
Other:
- note added: "Chassis"
- company: Sierra Lobo INC -> (none)
- title: (none) -> Foras Promineo Payload Interface Board
- moved on the sheet: C8, C9
