File: hardware/revB/Full_Bridge.kicad_sch (KiCad schematic)
At the start: 7 parts, among them U16 DRV8838DSGT

Commit message: working revB
Parts:
- R111: value 100k -> 10Meg
Changed lines of the file:
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@@
       (effects (font (size 1.27 1.27)) (justify left))
     )
-    (property "Value" "100k" (at 101.6 93.9799 0)
+    (property "Value" "10Meg" (at 101.6 93.9799 0)
       (effects (font (size 1.27 1.27)) (justify left))
     )

Commit message: working revB
Parts:
- removed R59, R60, R61: 1k, Resistor_SMD:R_0603_1608Metric, symbol Device:R_US
- renumbered C49 to C35, R111 to R68, U16 to U14
Connections:
- net EN: now also U14.5 (EN)
- net PH: now also U14.6 (PH)
- net ~{SLEEP}: now also U14.7 (~{SLEEP})

Commit message: updated files
Parts:
- renumbered C35 to C33, D6 to D8, R68 to R47, U14 to U12
Connections:
- net +3V3 renamed +3.3V

Commit message: working
Parts:
- renumbered C33 to C36, R47 to R49, U12 to U14
Other:
- company: Sierra Lobo INC -> (none)
- title: (none) -> Foras Promineo Payload Interface Board
- moved on the sheet: C36, R49
