File: hardware/revB/pico.kicad_sch (KiCad schematic)
At the start: 8 parts, among them Q20 MMBT4401-7-F, Q21 IRF7404TRPBF, U25 Pico

Commit message: working revB
Parts:
- removed R90: 100k, Resistor_SMD:R_0603_1608Metric, symbol Device:R_US
- added R106: 100, Resistor_SMD:R_0603_1608Metric, symbol Device:R_US
- added R23: 1k, Resistor_SMD:R_0603_1608Metric, symbol Device:R_US
- R91: value 10k -> 1Meg
- R92: value 3.3k -> 10Meg
Connections:
- net at Q20.3 (C), R92.2: now also R106.1; no longer Q21.4 (G)
- net Pico_Tx: now reaches U25.6 (GPIO4)
- net at U25.7 (GPIO5): now also R23.2
- net I2C1_SCL: no longer names the net of U25.5 (GPIO3)
- net I2C1_SDA: no longer names the net of U25.4 (GPIO2)
- net RB_PWR_SW_B: no longer names the net of Q20.1 (B), R91.2
- new net: Q21.4 (G), R106.2
- new net Pico_Rx: R23.1
Other:
- note removed: "Pico used as an I2C slave only to give device heritage"
- moved on the sheet: Q20, R92

Commit message: working revB
Parts:
- Q19: renamed from Q20; value MMBT4401-7-F -> MMBT4401WT1G; footprint Package_TO_SOT_SMD:SOT-23 -> Package_TO_SOT_SMD:SOT-323_SC-70
- renumbered C72 to C48, Q21 to Q20, R91 to R92, R92 to R93, U25 to U22
Changed lines of the file:
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@@
   (symbol (lib_id "power:GND") (at 228.6 100.33 0) (unit 1)
     (in_bom yes) (on_board yes) (dnp no) (fields_autoplaced)
-    (property "Reference" "#PWR0120" (at 228.6 106.68 0)
+    (property "Reference" "#PWR0108" (at 228.6 106.68 0)
       (effects (font (size 1.27 1.27)) hide)
     )
@@
       (project "FP Interface Card"
         (path "/dc2801a1-d539-4721-b31f-fe196b9f13df/dd622a02-7df1-4bf4-8b18-36d28830c650"
-          (reference "#PWR0120") (unit 1)
+          (reference "#PWR0108") (unit 1)
         )
       )
@@
   (symbol (lib_id "power:GND") (at 228.6 87.63 0) (unit 1)
     (in_bom yes) (on_board yes) (dnp no) (fields_autoplaced)
-    (property "Reference" "#PWR0109" (at 228.6 93.98 0)
+    (property "Reference" "#PWR0107" (at 228.6 93.98 0)
       (effects (font (size 1.27 1.27)) hide)
     )
@@
       (project "FP Interface Card"
         (path "/dc2801a1-d539-4721-b31f-fe196b9f13df/dd622a02-7df1-4bf4-8b18-36d28830c650"
-          (reference "#PWR0109") (unit 1)
+          (reference "#PWR0107") (unit 1)
         )
       )
@@
         )
         (path "/dc2801a1-d539-4721-b31f-fe196b9f13df/dd622a02-7df1-4bf4-8b18-36d28830c650"
-          (reference "R90") (unit 1)
+          (reference "R91") (unit 1)
         )
       )
@@
   (symbol (lib_id "power:GND") (at 228.6 125.73 0) (unit 1)
     (in_bom yes) (on_board yes) (dnp no) (fields_autoplaced)
-    (property "Reference" "#PWR0118" (at 228.6 132.08 0)
+    (property "Reference" "#PWR0110" (at 228.6 132.08 0)
       (effects (font (size 1.27 1.27)) hide)
     )
@@
       (project "FP Interface Card"
         (path "/dc2801a1-d539-4721-b31f-fe196b9f13df/dd622a02-7df1-4bf4-8b18-36d28830c650"
-          (reference "#PWR0118") (unit 1)
+          (reference "#PWR0110") (unit 1)
         )
       )
@@
   (symbol (lib_id "power:GND") (at 60.96 113.03 0) (mirror y) (unit 1)
     (in_bom yes) (on_board yes) (dnp no) (fields_autoplaced)
-    (property "Reference" "#PWR0126" (at 60.96 119.38 0)
+    (property "Reference" "#PWR0102" (at 60.96 119.38 0)
       (effects (font (size 1.27 1.27)) hide)
     )
@@
       (project "FP Interface Card"
         (path "/dc2801a1-d539-4721-b31f-fe196b9f13df/dd622a02-7df1-4bf4-8b18-36d28830c650"
-          (reference "#PWR0126") (unit 1)
+          (reference "#PWR0102") (unit 1)
         )
       )
@@
   (symbol (lib_id "Device:R_US") (at 163.83 39.37 0) (unit 1)
     (in_bom yes) (on_board yes) (dnp no)
-    (property "Reference" "R92" (at 154.94 38.1 0)
+    (property "Reference" "R93" (at 154.94 38.1 0)
       (effects (font (size 1.27 1.27)) (justify left))
     )
@@
       (project "FP Interface Card"
         (path "/dc2801a1-d539-4721-b31f-fe196b9f13df/dd622a02-7df1-4bf4-8b18-36d28830c650"
-          (reference "R92") (unit 1)
+          (reference "R93") (unit 1)
         )
       )
@@
   (symbol (lib_id "power:GND") (at 228.6 113.03 0) (unit 1)
     (in_bom yes) (on_board yes) (dnp no) (fields_autoplaced)
-    (property "Reference" "#PWR0115" (at 228.6 119.38 0)
+    (property "Reference" "#PWR0109" (at 228.6 119.38 0)
       (effects (font (size 1.27 1.27)) hide)
     )
@@
       (project "FP Interface Card"
         (path "/dc2801a1-d539-4721-b31f-fe196b9f13df/dd622a02-7df1-4bf4-8b18-36d28830c650"
-          (reference "#PWR0115") (unit 1)
+          (reference "#PWR0109") (unit 1)
         )
       )
@@
   (symbol (lib_id "power:GND") (at 163.83 60.96 0) (mirror y) (unit 1)
     (in_bom yes) (on_board yes) (dnp no)
-    (property "Reference" "#PWR0114" (at 163.83 67.31 0)
+    (property "Reference" "#PWR0106" (at 163.83 67.31 0)
       (effects (font (size 1.27 1.27)) hide)
     )
@@
       (project "FP Interface Card"
         (path "/dc2801a1-d539-4721-b31f-fe196b9f13df/dd622a02-7df1-4bf4-8b18-36d28830c650"
-          (reference "#PWR0114") (unit 1)
+          (reference "#PWR0106") (unit 1)
         )
       )
@@
   (symbol (lib_id "power:GND") (at 60.96 100.33 0) (mirror y) (unit 1)
     (in_bom yes) (on_board yes) (dnp no) (fields_autoplaced)
-    (property "Reference" "#PWR0125" (at 60.96 106.68 0)
+    (property "Reference" "#PWR0101" (at 60.96 106.68 0)
       (effects (font (size 1.27 1.27)) hide)
     )
@@
       (project "FP Interface Card"
         (path "/dc2801a1-d539-4721-b31f-fe196b9f13df/dd622a02-7df1-4bf4-8b18-36d28830c650"
-          (reference "#PWR0125") (unit 1)
+          (reference "#PWR0101") (unit 1)
         )
       )
@@
   (symbol (lib_id "power:GND") (at 60.96 87.63 0) (mirror y) (unit 1)
     (in_bom yes) (on_board yes) (dnp no) (fields_autoplaced)
-    (property "Reference" "#PWR0129" (at 60.96 93.98 0)
+    (property "Reference" "#PWR0100" (at 60.96 93.98 0)
       (effects (font (size 1.27 1.27)) hide)
     )
@@
       (project "FP Interface Card"
         (path "/dc2801a1-d539-4721-b31f-fe196b9f13df/dd622a02-7df1-4bf4-8b18-36d28830c650"
-          (reference "#PWR0129") (unit 1)
+          (reference "#PWR0100") (unit 1)
         )
       )
@@
   (symbol (lib_id "Device:Q_NPN_BEC") (at 161.29 53.34 0) (unit 1)
     (in_bom yes) (on_board yes) (dnp no) (fields_autoplaced)
-    (property "Reference" "Q20" (at 166.37 52.0699 0)
-      (effects (font (size 1.27 1.27)) (justify left))
-    )
-    (property "Value" "MMBT4401-7-F" (at 166.37 54.6099 0)
-      (effects (font (size 1.27 1.27)) (justify left))
-    )
-    (property "Footprint" "Package_TO_SOT_SMD:SOT-23" (at 166.37 50.8 0)
+    (property "Reference" "Q19" (at 166.37 52.0699 0)
+      (effects (font (size 1.27 1.27)) (justify left))
+    )
+    (property "Value" "MMBT4401WT1G" (at 166.37 54.6099 0)
+      (effects (font (size 1.27 1.27)) (justify left))
+    )
+    (property "Footprint" "Package_TO_SOT_SMD:SOT-323_SC-70" (at 166.37 50.8 0)
       (effects (font (size 1.27 1.27)) hide)
     )
@@
       (project "FP Interface Card"
         (path "/dc2801a1-d539-4721-b31f-fe196b9f13df/dd622a02-7df1-4bf4-8b18-36d28830c650"
-          (reference "Q20") (unit 1)
+          (reference "Q19") (unit 1)
         )
       )
@@
   (symbol (lib_id "Device:C") (at 208.28 78.74 0) (unit 1)
     (in_bom yes) (on_board yes) (dnp no) (fields_autoplaced)
-    (property "Reference" "C72" (at 212.09 77.4699 0)
+    (property "Reference" "C48" (at 212.09 77.4699 0)
       (effects (font (size 1.27 1.27)) (justify left))
     )
@@
       (project "FP Interface Card"
         (path "/dc2801a1-d539-4721-b31f-fe196b9f13df/dd622a02-7df1-4bf4-8b18-36d28830c650"
-          (reference "C72") (unit 1)
+          (reference "C48") (unit 1)
         )
       )
@@
   (symbol (lib_id "power:+5V") (at 156.21 35.56 0) (unit 1)
     (in_bom yes) (on_board yes) (dnp no) (fields_autoplaced)
-    (property "Reference" "#PWR0108" (at 156.21 39.37 0)
+    (property "Reference" "#PWR0105" (at 156.21 39.37 0)
       (effects (font (size 1.27 1.27)) hide)
     )
@@
       (project "FP Interface Card"
         (path "/dc2801a1-d539-4721-b31f-fe196b9f13df/dd622a02-7df1-4bf4-8b18-36d28830c650"
-          (reference "#PWR0108") (unit 1)
+          (reference "#PWR0105") (unit 1)
         )
       )
@@
   (symbol (lib_id "power:GND") (at 144.78 135.89 0) (unit 1)
     (in_bom yes) (on_board yes) (dnp no) (fields_autoplaced)
-    (property "Reference" "#PWR0123" (at 144.78 142.24 0)
+    (property "Reference" "#PWR0104" (at 144.78 142.24 0)
       (effects (font (size 1.27 1.27)) hide)
     )
@@
       (project "FP Interface Card"
         (path "/dc2801a1-d539-4721-b31f-fe196b9f13df/dd622a02-7df1-4bf4-8b18-36d28830c650"
-          (reference "#PWR0123") (unit 1)
+          (reference "#PWR0104") (unit 1)
         )
       )
@@
         )
         (path "/dc2801a1-d539-4721-b31f-fe196b9f13df/dd622a02-7df1-4bf4-8b18-36d28830c650"
-          (reference "R71") (unit 1)
+          (reference "R94") (unit 1)
         )
       )
@@
   (symbol (lib_id "RPi_Pico:Pico") (at 144.78 104.14 0) (unit 1)
     (in_bom yes) (on_board yes) (dnp no) (fields_autoplaced)
-    (property "Reference" "U25" (at 144.78 72.39 0)
+    (property "Reference" "U22" (at 144.78 72.39 0)
       (effects (font (size 1.27 1.27)))
     )
@@
       (project "FP Interface Card"
         (path "/dc2801a1-d539-4721-b31f-fe196b9f13df/dd622a02-7df1-4bf4-8b18-36d28830c650"
-          (reference "U25") (unit 1)
+          (reference "U22") (unit 1)
         )
       )
@@
   (symbol (lib_id "SLI-Backplane-Blank-Card-KiCad:IRF7404TRPBF") (at 179.07 43.18 0) (mirror x) (unit 1)
     (in_bom yes) (on_board yes) (dnp no) (fields_autoplaced)
-    (property "Reference" "Q21" (at 185.42 41.9099 0)
+    (property "Reference" "Q20" (at 185.42 41.9099 0)
       (effects (font (size 1.27 1.27)) (justify left))
     )
@@
       (project "FP Interface Card"
         (path "/dc2801a1-d539-4721-b31f-fe196b9f13df/dd622a02-7df1-4bf4-8b18-36d28830c650"
-          (reference "Q21") (unit 1)
+          (reference "Q20") (unit 1)
         )
       )
@@
   (symbol (lib_id "power:GND") (at 60.96 125.73 0) (mirror y) (unit 1)
     (in_bom yes) (on_board yes) (dnp no) (fields_autoplaced)
-    (property "Reference" "#PWR0127" (at 60.96 132.08 0)
+    (property "Reference" "#PWR0103" (at 60.96 132.08 0)
       (effects (font (size 1.27 1.27)) hide)
     )
@@
       (project "FP Interface Card"
         (path "/dc2801a1-d539-4721-b31f-fe196b9f13df/dd622a02-7df1-4bf4-8b18-36d28830c650"
-          (reference "#PWR0127") (unit 1)
+          (reference "#PWR0103") (unit 1)
         )
       )
@@
   (symbol (lib_id "Device:R_US") (at 152.4 53.34 90) (unit 1)
     (in_bom yes) (on_board yes) (dnp no) (fields_autoplaced)
-    (property "Reference" "R91" (at 152.4 46.99 90)
+    (property "Reference" "R92" (at 152.4 46.99 90)
       (effects (font (size 1.27 1.27)))
     )
@@
       (project "FP Interface Card"
         (path "/dc2801a1-d539-4721-b31f-fe196b9f13df/dd622a02-7df1-4bf4-8b18-36d28830c650"
-          (reference "R91") (unit 1)
-        )
-      )
+          (reference "R92") (unit 1)
+        )
+      )

Commit message: updated files
Parts:
- renumbered D8 to D10, Q20 to Q19, Q19 to Q20, R93 to R77, R92 to R79

Commit message: working
Parts:
- R106: value 100 -> 1K
- renumbered C48 to C51, Q19 to Q18, Q20 to Q19, R77 to R75, R79 to R77, U22 to U20
Other:
- company: Sierra Lobo INC -> (none)
- title: (none) -> Foras Promineo Payload Interface Board
Changed lines of the file:
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@@
   (paper "A4")
   (title_block
+    (title "Foras Promineo Payload Interface Board")
     (rev "B")
-    (company "Sierra Lobo INC")
   )
   (junction (at 163.83 43.18) (diameter 0) (color 0 0 0 0)
@@
         )
         (path "/dc2801a1-d539-4721-b31f-fe196b9f13df/dd622a02-7df1-4bf4-8b18-36d28830c650"
-          (reference "R80") (unit 1)
+          (reference "R78") (unit 1)
         )
       )
@@
   (symbol (lib_id "Device:R_US") (at 163.83 39.37 0) (unit 1)
     (in_bom yes) (on_board yes) (dnp no)
-    (property "Reference" "R77" (at 154.94 38.1 0)
+    (property "Reference" "R75" (at 154.94 38.1 0)
       (effects (font (size 1.27 1.27)) (justify left))
     )
@@
       (project "payload-interface-board"
         (path "/dc2801a1-d539-4721-b31f-fe196b9f13df/dd622a02-7df1-4bf4-8b18-36d28830c650"
-          (reference "R77") (unit 1)
+          (reference "R75") (unit 1)
         )
       )
@@
   (symbol (lib_id "Device:Q_NPN_BEC") (at 161.29 53.34 0) (unit 1)
     (in_bom yes) (on_board yes) (dnp no) (fields_autoplaced)
-    (property "Reference" "Q20" (at 166.37 52.0699 0)
+    (property "Reference" "Q19" (at 166.37 52.0699 0)
       (effects (font (size 1.27 1.27)) (justify left))
     )
@@
       (project "payload-interface-board"
         (path "/dc2801a1-d539-4721-b31f-fe196b9f13df/dd622a02-7df1-4bf4-8b18-36d28830c650"
-          (reference "Q20") (unit 1)
+          (reference "Q19") (unit 1)
         )
       )
@@
   (symbol (lib_id "Device:C") (at 208.28 78.74 0) (unit 1)
     (in_bom yes) (on_board yes) (dnp no) (fields_autoplaced)
-    (property "Reference" "C48" (at 212.09 77.4699 0)
+    (property "Reference" "C51" (at 212.09 77.4699 0)
       (effects (font (size 1.27 1.27)) (justify left))
     )
@@
       (project "payload-interface-board"
         (path "/dc2801a1-d539-4721-b31f-fe196b9f13df/dd622a02-7df1-4bf4-8b18-36d28830c650"
-          (reference "C48") (unit 1)
+          (reference "C51") (unit 1)
         )
       )
@@
       (effects (font (size 1.27 1.27)))
     )
-    (property "Value" "100" (at 170.18 48.26 90)
+    (property "Value" "1K" (at 170.18 48.26 90)
       (effects (font (size 1.27 1.27)))
     )
@@
         )
         (path "/dc2801a1-d539-4721-b31f-fe196b9f13df/dd622a02-7df1-4bf4-8b18-36d28830c650"
-          (reference "R78") (unit 1)
+          (reference "R76") (unit 1)
         )
       )
@@
   (symbol (lib_id "RPi_Pico:Pico") (at 144.78 104.14 0) (unit 1)
     (in_bom yes) (on_board yes) (dnp no) (fields_autoplaced)
-    (property "Reference" "U22" (at 144.78 72.39 0)
+    (property "Reference" "U20" (at 144.78 72.39 0)
       (effects (font (size 1.27 1.27)))
     )
@@
       (project "payload-interface-board"
         (path "/dc2801a1-d539-4721-b31f-fe196b9f13df/dd622a02-7df1-4bf4-8b18-36d28830c650"
-          (reference "U22") (unit 1)
+          (reference "U20") (unit 1)
         )
       )
@@
   (symbol (lib_id "SLI-Backplane-Blank-Card-KiCad:IRF7404TRPBF") (at 179.07 43.18 0) (mirror x) (unit 1)
     (in_bom yes) (on_board yes) (dnp no) (fields_autoplaced)
-    (property "Reference" "Q19" (at 185.42 41.9099 0)
+    (property "Reference" "Q18" (at 185.42 41.9099 0)
       (effects (font (size 1.27 1.27)) (justify left))
     )
@@
       (project "payload-interface-board"
         (path "/dc2801a1-d539-4721-b31f-fe196b9f13df/dd622a02-7df1-4bf4-8b18-36d28830c650"
-          (reference "Q19") (unit 1)
+          (reference "Q18") (unit 1)
         )
       )
@@
   (symbol (lib_id "Device:R_US") (at 152.4 53.34 90) (unit 1)
     (in_bom yes) (on_board yes) (dnp no) (fields_autoplaced)
-    (property "Reference" "R79" (at 152.4 46.99 90)
+    (property "Reference" "R77" (at 152.4 46.99 90)
       (effects (font (size 1.27 1.27)))
     )
@@
       (project "payload-interface-board"
         (path "/dc2801a1-d539-4721-b31f-fe196b9f13df/dd622a02-7df1-4bf4-8b18-36d28830c650"
-          (reference "R79") (unit 1)
-        )
-      )
+          (reference "R77") (unit 1)
+        )
+      )
