File: hardware/revB/I2C-Protection.kicad_sch (KiCad schematic)
At the start: 22 parts, among them Q13 BSS138DWQ-7, Q14 MMDT5551-7-F, Q15 BSS138DWQ-7, Q16 MMDT5551-7-F

Commit message: working revB
Parts:
- removed TP30, TP31, TP32, TP33: TestPoint, TestPoint:TestPoint_Pad_D1.0mm, symbol Connector:TestPoint
Changed lines of the file:
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@@
-    (stroke (width 0) (type default))
-  )
-  (wire (pts (xy 210.82 64.77) (xy 214.63 64.77))
     (stroke (width 0) (type default))
   )
@@
     (stroke (width 0) (type default))
   )
-  (wire (pts (xy 210.82 83.82) (xy 214.63 83.82))
-    (stroke (width 0) (type default))
-  )
   (wire (pts (xy 120.65 83.82) (xy 120.65 101.6))
     (stroke (width 0) (type default))
@@
     (stroke (width 0) (type default))
   )
-  (wire (pts (xy 210.82 77.47) (xy 214.63 77.47))
-    (stroke (width 0) (type default))
-  )
   (wire (pts (xy 149.86 114.3) (xy 149.86 121.92))
-    (stroke (width 0) (type default))
-  )
-  (wire (pts (xy 210.82 71.12) (xy 214.63 71.12))
     (stroke (width 0) (type default))
   )
@@
     (effects (font (size 1.27 1.27)) (justify left))
   )
-  (hierarchical_label "SDA_IN" (shape input) (at 210.82 71.12 180) (fields_autoplaced)
-    (effects (font (size 1.27 1.27)) (justify right))
-  )
-  (hierarchical_label "SCL_PROT" (shape input) (at 210.82 77.47 180) (fields_autoplaced)
-    (effects (font (size 1.27 1.27)) (justify right))
-  )
   (hierarchical_label "SCL_PROT" (shape input) (at 133.35 92.71 0) (fields_autoplaced)
     (effects (font (size 1.27 1.27)) (justify left))
@@
   )
   (hierarchical_label "SDA_IN" (shape input) (at 158.75 83.82 180) (fields_autoplaced)
-    (effects (font (size 1.27 1.27)) (justify right))
-  )
-  (hierarchical_label "SCL_IN" (shape input) (at 210.82 64.77 180) (fields_autoplaced)
-    (effects (font (size 1.27 1.27)) (justify right))
-  )
-  (hierarchical_label "SDA_PROT" (shape input) (at 210.82 83.82 180) (fields_autoplaced)
     (effects (font (size 1.27 1.27)) (justify right))
   )
@@
     )
   )
-  (symbol (lib_id "Connector:TestPoint") (at 214.63 71.12 0) (unit 1)
-    (in_bom yes) (on_board yes) (dnp no) (fields_autoplaced)
-    (property "Reference" "TP31" (at 217.17 66.5479 0)
-      (effects (font (size 1.27 1.27)) (justify left))
-    )
-    (property "Value" "TestPoint" (at 217.17 69.0879 0)
-      (effects (font (size 1.27 1.27)) (justify left) hide)
-    )
-    (property "Footprint" "TestPoint:TestPoint_Pad_D1.0mm" (at 219.71 71.12 0)
-      (effects (font (size 1.27 1.27)) hide)
-    )
-    (property "Datasheet" "~" (at 219.71 71.12 0)
-      (effects (font (size 1.27 1.27)) hide)
-    )
-    (pin "1")
-    (instances
-      (project "FP Interface Card"
-        (path "/dc2801a1-d539-4721-b31f-fe196b9f13df/60a3e3f0-4d0a-42d5-9dae-542c30f8587f"
-          (reference "TP31") (unit 1)
-        )
-        (path "/dc2801a1-d539-4721-b31f-fe196b9f13df/51f2d4b3-6068-40f6-b19f-12cc4569573f"
-          (reference "TP16") (unit 1)
-        )
-      )
-    )
-  )
   (symbol (lib_id "mainboard-rescue:MBT2222ADW1T1-Transistor_BJT-mainboard-rescue") (at 125.73 99.06 270) (unit 1)
     (in_bom yes) (on_board yes) (dnp no)
@@
     )
   )
-  (symbol (lib_id "Connector:TestPoint") (at 214.63 83.82 0) (unit 1)
-    (in_bom yes) (on_board yes) (dnp no) (fields_autoplaced)
-    (property "Reference" "TP33" (at 217.17 79.2479 0)
-      (effects (font (size 1.27 1.27)) (justify left))
-    )
-    (property "Value" "TestPoint" (at 217.17 81.7879 0)
-      (effects (font (size 1.27 1.27)) (justify left) hide)
-    )
-    (property "Footprint" "TestPoint:TestPoint_Pad_D1.0mm" (at 219.71 83.82 0)
-      (effects (font (size 1.27 1.27)) hide)
-    )
-    (property "Datasheet" "~" (at 219.71 83.82 0)
-      (effects (font (size 1.27 1.27)) hide)
-    )
-    (pin "1")
-    (instances
-      (project "FP Interface Card"
-        (path "/dc2801a1-d539-4721-b31f-fe196b9f13df/60a3e3f0-4d0a-42d5-9dae-542c30f8587f"
-          (reference "TP33") (unit 1)
-        )
-        (path "/dc2801a1-d539-4721-b31f-fe196b9f13df/51f2d4b3-6068-40f6-b19f-12cc4569573f"
-          (reference "TP18") (unit 1)
-        )
-      )
-    )
-  )
   (symbol (lib_id "Device:R_US") (at 130.81 107.95 0) (unit 1)
     (in_bom yes) (on_board yes) (dnp no)
@@
     )
   )
-  (symbol (lib_id "Connector:TestPoint") (at 214.63 77.47 0) (unit 1)
-    (in_bom yes) (on_board yes) (dnp no) (fields_autoplaced)
-    (property "Reference" "TP32" (at 217.17 72.8979 0)
-      (effects (font (size 1.27 1.27)) (justify left))
-    )
-    (property "Value" "TestPoint" (at 217.17 75.4379 0)
-      (effects (font (size 1.27 1.27)) (justify left) hide)
-    )
-    (property "Footprint" "TestPoint:TestPoint_Pad_D1.0mm" (at 219.71 77.47 0)
-      (effects (font (size 1.27 1.27)) hide)
-    )
-    (property "Datasheet" "~" (at 219.71 77.47 0)
-      (effects (font (size 1.27 1.27)) hide)
-    )
-    (pin "1")
-    (instances
-      (project "FP Interface Card"
-        (path "/dc2801a1-d539-4721-b31f-fe196b9f13df/60a3e3f0-4d0a-42d5-9dae-542c30f8587f"
-          (reference "TP32") (unit 1)
-        )
-        (path "/dc2801a1-d539-4721-b31f-fe196b9f13df/51f2d4b3-6068-40f6-b19f-12cc4569573f"
-          (reference "TP17") (unit 1)
-        )
-      )
-    )
-  )
   (symbol (lib_id "mainboard:3.3V") (at 130.81 68.58 0) (unit 1)
     (in_bom yes) (on_board yes) (dnp no)
@@
         )
       )
-    )
-  )
-  (symbol (lib_id "Connector:TestPoint") (at 214.63 64.77 0) (unit 1)
-    (in_bom yes) (on_board yes) (dnp no) (fields_autoplaced)
-    (property "Reference" "TP30" (at 217.17 60.1979 0)
-      (effects (font (size 1.27 1.27)) (justify left))
-    )
-    (property "Value" "TestPoint" (at 217.17 62.7379 0)
-      (effects (font (size 1.27 1.27)) (justify left) hide)
-    )
-    (property "Footprint" "TestPoint:TestPoint_Pad_D1.0mm" (at 219.71 64.77 0)
-      (effects (font (size 1.27 1.27)) hide)
-    )
-    (property "Datasheet" "~" (at 219.71 64.77 0)
-      (effects (font (size 1.27 1.27)) hide)
-    )
-    (pin "1")
-    (instances
-      (project "FP Interface Card"
-        (path "/dc2801a1-d539-4721-b31f-fe196b9f13df/60a3e3f0-4d0a-42d5-9dae-542c30f8587f"
-          (reference "TP30") (unit 1)
-        )
-        (path "/dc2801a1-d539-4721-b31f-fe196b9f13df/51f2d4b3-6068-40f6-b19f-12cc4569573f"
-          (reference "TP15") (unit 1)
-        )
-      )

Commit message: working revB
Parts:
- renumbered C70 to C46, C71 to C47, Q13 to Q15, Q14 to Q16, Q15 to Q17, Q16 to Q18, R77 to R79, R78 to R80, R79 to R81, R80 to R82, R81 to R83, R82 to R84, R83 to R85, R84 to R86, R85 to R87, R86 to R88, R87 to R89, R88 to R90

Commit message: updated files
Parts:
- renumbered Q16 to Q15, Q18 to Q16, Q15 to Q17, Q17 to Q18, R81 to R65, R86 to R66, R82 to R67, R87 to R68, R80 to R69, R85 to R70, R79 to R71, R84 to R72, R83 to R73, R88 to R74, R89 to R75, R90 to R76
Connections:
- net 3.3V renamed +3.3V

Commit message: working
Parts:
- C58: renamed from C46; value 10nF -> 0.01uF; footprint Capacitor_SMD:C_0603_1608Metric -> Capacitor_SMD:C_0402_1005Metric
- C59: renamed from C47; value 10nF -> 0.01uF; footprint Capacitor_SMD:C_0603_1608Metric -> Capacitor_SMD:C_0402_1005Metric
- R128: renamed from R65; footprint Resistor_SMD:R_0603_1608Metric -> Resistor_SMD:R_0402_1005Metric
- R129: renamed from R66; footprint Resistor_SMD:R_0603_1608Metric -> Resistor_SMD:R_0402_1005Metric
- R130: renamed from R67; footprint Resistor_SMD:R_0603_1608Metric -> Resistor_SMD:R_0402_1005Metric
- R131: renamed from R68; footprint Resistor_SMD:R_0603_1608Metric -> Resistor_SMD:R_0402_1005Metric
- R134: renamed from R71; footprint Resistor_SMD:R_0603_1608Metric -> Resistor_SMD:R_0402_1005Metric
- R135: renamed from R72; footprint Resistor_SMD:R_0603_1608Metric -> Resistor_SMD:R_0402_1005Metric
- R136: renamed from R73; footprint Resistor_SMD:R_0603_1608Metric -> Resistor_SMD:R_0402_1005Metric
- R137: renamed from R74; footprint Resistor_SMD:R_0603_1608Metric -> Resistor_SMD:R_0402_1005Metric
- R138: renamed from R75; now not fitted
- R139: renamed from R76; now not fitted
- renumbered Q15 to Q19, Q16 to Q20, Q17 to Q21, Q18 to Q22, R69 to R132, R70 to R133
Connections:
- net SCL_IN renamed SCL_I
- net SCL_PROT renamed SCL_O
- net SDA_IN renamed SDA_I
- net SDA_PROT renamed SDA_O
Other:
- note added: "Bypass Jumpers"
- note added: "I2C Bus Protection"
- note removed: "DNP"
- note removed: "I2C Bus Protection PIB"
- note removed: "sub'd q7,8 was MBR2222ADW1T1"
- company: Sierra Lobo INC -> (none)
- title: (none) -> Foras Promineo Payload Interface Board
- moved on the sheet: C58, C59, Q19A, Q19B, Q20A, Q20B, Q21A, Q21B, Q22A, Q22B, R128, R129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

Commit message: revB initial commit
Parts:
- removed Q20: MMDT5551-7-F, Package_TO_SOT_SMD:SOT-363_SC-70-6, symbol mainboard-rescue:MBT2222ADW1T1-Transistor_BJT-mainboard-rescue
- added Q11: MMDT2222A, Package_TO_SOT_SMD:SOT-363_SC-70-6, symbol SierraLobo:MMDT2222
- C15: renamed from C58; footprint Capacitor_SMD:C_0402_1005Metric -> Capacitor_SMD:C_0603_1608Metric
- C16: renamed from C59; footprint Capacitor_SMD:C_0402_1005Metric -> Capacitor_SMD:C_0603_1608Metric
- Q10: renamed from Q19; value MMDT5551-7-F -> MMDT2222A; symbol mainboard-rescue:MBT2222ADW1T1-Transistor_BJT-mainboard-rescue -> SierraLobo:MMDT2222
- R41: renamed from R128; footprint Resistor_SMD:R_0402_1005Metric -> Resistor_SMD:R_0603_1608Metric
- R42: renamed from R129; footprint Resistor_SMD:R_0402_1005Metric -> Resistor_SMD:R_0603_1608Metric
- R43: renamed from R130; footprint Resistor_SMD:R_0402_1005Metric -> Resistor_SMD:R_0603_1608Metric
- R44: renamed from R131; footprint Resistor_SMD:R_0402_1005Metric -> Resistor_SMD:R_0603_1608Metric
- R47: renamed from R134; footprint Resistor_SMD:R_0402_1005Metric -> Resistor_SMD:R_0603_1608Metric
- R48: renamed from R135; footprint Resistor_SMD:R_0402_1005Metric -> Resistor_SMD:R_0603_1608Metric
- R49: renamed from R136; footprint Resistor_SMD:R_0402_1005Metric -> Resistor_SMD:R_0603_1608Metric
- R50: renamed from R137; footprint Resistor_SMD:R_0402_1005Metric -> Resistor_SMD:R_0603_1608Metric
- renumbered Q21 to Q14, Q22 to Q15, R132 to R45, R133 to R46, R138 to R51, R139 to R52
Connections:
- net SCL_I: now also Q10.4 (E1), Q10.6 (C2); no longer Q10.1 (E1), Q10.3 (C2)
- net SCL_O: now also Q10.1 (E2), Q10.3 (C1); no longer Q10.4 (E2), Q10.6 (C1)
- net SDA_I: now also Q11.4 (E1), Q11.6 (C2)
- net SDA_O: now also Q11.1 (E2), Q11.3 (C1)
- net at R45.1: now also Q10.5 (B1); no longer Q10.2 (B1)
- net at Q14.6 (D1), R41.2, R45.2: now also Q10.2 (B2); no longer Q10.5 (B2)
- net at Q15.6 (D1), R42.2, R46.2: now also Q11.2 (B2)
- net at R46.1: now also Q11.5 (B1)
Other:
- title: Foras Promineo Payload Interface Board -> Foras Promineo Payload Interface
