File: hardware/revB/load_sw.kicad_sch (KiCad schematic)
At the start: 8 parts, among them Q13 BSZ180, Q2 MMBT4401WT1G

Commit message: revB initial commit
Parts:
- C5: footprint Capacitor_SMD:C_0402_1005Metric -> Capacitor_SMD:C_0603_1608Metric
- R3, R4, R5: footprint Resistor_SMD:R_0402_1005Metric -> Resistor_SMD:R_0603_1608Metric
Other:
- title: Foras Promineo Payload Interface Board -> Foras Promineo Payload Interface
Changed lines of the file:
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@@
   (paper "A4")
   (title_block
-    (title "Foras Promineo Payload Interface Board")
+    (title "Foras Promineo Payload Interface")
     (rev "B")
+    (comment 1 "CH")
+    (comment 2 "CH")
   )
   (junction (at 142.24 73.66) (diameter 0) (color 0 0 0 0)
@@
   )
   (hierarchical_label "VIN" (shape input) (at 74.93 73.66 180) (fields_autoplaced)
-    (effects (font (size 1.27 1.27)) (justify right))
+    (effects (font (size 1.524 1.524)) (justify right))
   )
   (hierarchical_label "EN" (shape input) (at 74.93 100.33 180) (fields_autoplaced)
-    (effects (font (size 1.27 1.27)) (justify right))
+    (effects (font (size 1.524 1.524)) (justify right))
   )
   (hierarchical_label "VOUT" (shape output) (at 223.52 73.66 0) (fields_autoplaced)
-    (effects (font (size 1.27 1.27)) (justify left))
+    (effects (font (size 1.524 1.524)) (justify left))
   )
   (symbol (lib_id "Device:R_US") (at 125.73 100.33 90) (unit 1)
@@
       (effects (font (size 1.27 1.27)))
     )
-    (property "Footprint" "Resistor_SMD:R_0402_1005Metric" (at 125.984 99.314 90)
+    (property "Footprint" "Resistor_SMD:R_0603_1608Metric" (at 125.984 99.314 90)
       (effects (font (size 1.27 1.27)) hide)
     )
@@
       (effects (font (size 1.27 1.27)) hide)
     )
+    (property "Mfr. Part No" "" (at 125.73 100.33 0)
+      (effects (font (size 1.27 1.27)) hide)
+    )
     (pin "1")
     (pin "2")
@@
         )
         (path "/dc2801a1-d539-4721-b31f-fe196b9f13df/7434567b-e3d3-4b0f-9e9c-75cfe7b5f5ad"
-          (reference "R69") (unit 1)
-        )
-        (path "/dc2801a1-d539-4721-b31f-fe196b9f13df/8888f9b5-1ed7-43cb-9174-e948cce171c0"
-          (reference "R73") (unit 1)
-        )
-        (path "/dc2801a1-d539-4721-b31f-fe196b9f13df/24d21d3f-37df-43db-a302-5a6c43abae48/9613f8ce-52d8-40c4-ba4b-e6be8fea7c63"
-          (reference "R77") (unit 1)
+          (reference "R36") (unit 1)
+        )
+        (path "/dc2801a1-d539-4721-b31f-fe196b9f13df/8888f9b5-1ed7-43cb-9174-e948cce171c0"
+          (reference "R40") (unit 1)
         )
       )
@@
       (effects (font (size 1.27 1.27)) (justify left))
     )
-    (property "Footprint" "Capacitor_SMD:C_0402_1005Metric" (at 143.2052 85.09 0)
+    (property "Footprint" "Capacitor_SMD:C_0603_1608Metric" (at 143.2052 85.09 0)
       (effects (font (size 1.27 1.27)) hide)
     )
@@
         )
         (path "/dc2801a1-d539-4721-b31f-fe196b9f13df/7434567b-e3d3-4b0f-9e9c-75cfe7b5f5ad"
-          (reference "C30") (unit 1)
-        )
-        (path "/dc2801a1-d539-4721-b31f-fe196b9f13df/8888f9b5-1ed7-43cb-9174-e948cce171c0"
-          (reference "C31") (unit 1)
-        )
-        (path "/dc2801a1-d539-4721-b31f-fe196b9f13df/24d21d3f-37df-43db-a302-5a6c43abae48/9613f8ce-52d8-40c4-ba4b-e6be8fea7c63"
-          (reference "C32") (unit 1)
+          (reference "C13") (unit 1)
+        )
+        (path "/dc2801a1-d539-4721-b31f-fe196b9f13df/8888f9b5-1ed7-43cb-9174-e948cce171c0"
+          (reference "C14") (unit 1)
         )
       )
@@
       (effects (font (size 1.27 1.27)))
     )
-    (property "Footprint" "Resistor_SMD:R_0402_1005Metric" (at 157.226 86.614 90)
+    (property "Footprint" "Resistor_SMD:R_0603_1608Metric" (at 157.226 86.614 90)
       (effects (font (size 1.27 1.27)) hide)
     )
@@
         )
         (path "/dc2801a1-d539-4721-b31f-fe196b9f13df/7434567b-e3d3-4b0f-9e9c-75cfe7b5f5ad"
-          (reference "R67") (unit 1)
-        )
-        (path "/dc2801a1-d539-4721-b31f-fe196b9f13df/8888f9b5-1ed7-43cb-9174-e948cce171c0"
-          (reference "R71") (unit 1)
-        )
-        (path "/dc2801a1-d539-4721-b31f-fe196b9f13df/24d21d3f-37df-43db-a302-5a6c43abae48/9613f8ce-52d8-40c4-ba4b-e6be8fea7c63"
-          (reference "R75") (unit 1)
+          (reference "R34") (unit 1)
+        )
+        (path "/dc2801a1-d539-4721-b31f-fe196b9f13df/8888f9b5-1ed7-43cb-9174-e948cce171c0"
+          (reference "R38") (unit 1)
         )
       )
@@
         )
         (path "/dc2801a1-d539-4721-b31f-fe196b9f13df/7434567b-e3d3-4b0f-9e9c-75cfe7b5f5ad"
-          (reference "#PWR072") (unit 1)
-        )
-        (path "/dc2801a1-d539-4721-b31f-fe196b9f13df/8888f9b5-1ed7-43cb-9174-e948cce171c0"
-          (reference "#PWR073") (unit 1)
-        )
-        (path "/dc2801a1-d539-4721-b31f-fe196b9f13df/24d21d3f-37df-43db-a302-5a6c43abae48/9613f8ce-52d8-40c4-ba4b-e6be8fea7c63"
-          (reference "#PWR074") (unit 1)
+          (reference "#PWR053") (unit 1)
+        )
+        (path "/dc2801a1-d539-4721-b31f-fe196b9f13df/8888f9b5-1ed7-43cb-9174-e948cce171c0"
+          (reference "#PWR054") (unit 1)
         )
       )
@@
         )
         (path "/dc2801a1-d539-4721-b31f-fe196b9f13df/7434567b-e3d3-4b0f-9e9c-75cfe7b5f5ad"
-          (reference "Q10") (unit 1)
-        )
-        (path "/dc2801a1-d539-4721-b31f-fe196b9f13df/8888f9b5-1ed7-43cb-9174-e948cce171c0"
-          (reference "Q13") (unit 1)
-        )
-        (path "/dc2801a1-d539-4721-b31f-fe196b9f13df/24d21d3f-37df-43db-a302-5a6c43abae48/9613f8ce-52d8-40c4-ba4b-e6be8fea7c63"
-          (reference "Q16") (unit 1)
+          (reference "Q4") (unit 1)
+        )
+        (path "/dc2801a1-d539-4721-b31f-fe196b9f13df/8888f9b5-1ed7-43cb-9174-e948cce171c0"
+          (reference "Q7") (unit 1)
         )
       )
@@
         )
         (path "/dc2801a1-d539-4721-b31f-fe196b9f13df/7434567b-e3d3-4b0f-9e9c-75cfe7b5f5ad"
-          (reference "Q12") (unit 1)
-        )
-        (path "/dc2801a1-d539-4721-b31f-fe196b9f13df/8888f9b5-1ed7-43cb-9174-e948cce171c0"
-          (reference "Q15") (unit 1)
-        )
-        (path "/dc2801a1-d539-4721-b31f-fe196b9f13df/24d21d3f-37df-43db-a302-5a6c43abae48/9613f8ce-52d8-40c4-ba4b-e6be8fea7c63"
-          (reference "Q18") (unit 1)
+          (reference "Q6") (unit 1)
+        )
+        (path "/dc2801a1-d539-4721-b31f-fe196b9f13df/8888f9b5-1ed7-43cb-9174-e948cce171c0"
+          (reference "Q9") (unit 1)
         )
       )
@@
       (effects (font (size 1.27 1.27)))
     )
-    (property "Footprint" "Resistor_SMD:R_0402_1005Metric" (at 167.386 86.614 90)
+    (property "Footprint" "Resistor_SMD:R_0603_1608Metric" (at 167.386 86.614 90)
       (effects (font (size 1.27 1.27)) hide)
     )
@@
         )
         (path "/dc2801a1-d539-4721-b31f-fe196b9f13df/7434567b-e3d3-4b0f-9e9c-75cfe7b5f5ad"
-          (reference "R68") (unit 1)
-        )
-        (path "/dc2801a1-d539-4721-b31f-fe196b9f13df/8888f9b5-1ed7-43cb-9174-e948cce171c0"
-          (reference "R72") (unit 1)
-        )
-        (path "/dc2801a1-d539-4721-b31f-fe196b9f13df/24d21d3f-37df-43db-a302-5a6c43abae48/9613f8ce-52d8-40c4-ba4b-e6be8fea7c63"
-          (reference "R76") (unit 1)
+          (reference "R35") (unit 1)
+        )
+        (path "/dc2801a1-d539-4721-b31f-fe196b9f13df/8888f9b5-1ed7-43cb-9174-e948cce171c0"
+          (reference "R39") (unit 1)
         )
       )
@@
         )
         (path "/dc2801a1-d539-4721-b31f-fe196b9f13df/7434567b-e3d3-4b0f-9e9c-75cfe7b5f5ad"
-          (reference "Q11") (unit 1)
-        )
-        (path "/dc2801a1-d539-4721-b31f-fe196b9f13df/8888f9b5-1ed7-43cb-9174-e948cce171c0"
-          (reference "Q14") (unit 1)
-        )
-        (path "/dc2801a1-d539-4721-b31f-fe196b9f13df/24d21d3f-37df-43db-a302-5a6c43abae48/9613f8ce-52d8-40c4-ba4b-e6be8fea7c63"
-          (reference "Q17") (unit 1)
+          (reference "Q5") (unit 1)
+        )
+        (path "/dc2801a1-d539-4721-b31f-fe196b9f13df/8888f9b5-1ed7-43cb-9174-e948cce171c0"
+          (reference "Q8") (unit 1)
         )
       )
@@
       (effects (font (size 1.27 1.27)) (justify right))
     )
-    (property "Footprint" "Resistor_SMD:R_0402_1005Metric" (at 138.176 81.534 90)
+    (property "Footprint" "Resistor_SMD:R_0603_1608Metric" (at 138.176 81.534 90)
       (effects (font (size 1.27 1.27)) hide)
     )
@@
         )
         (path "/dc2801a1-d539-4721-b31f-fe196b9f13df/7434567b-e3d3-4b0f-9e9c-75cfe7b5f5ad"
-          (reference "R66") (unit 1)
-        )
-        (path "/dc2801a1-d539-4721-b31f-fe196b9f13df/8888f9b5-1ed7-43cb-9174-e948cce171c0"
-          (reference "R70") (unit 1)
-        )
-        (path "/dc2801a1-d539-4721-b31f-fe196b9f13df/24d21d3f-37df-43db-a302-5a6c43abae48/9613f8ce-52d8-40c4-ba4b-e6be8fea7c63"
-          (reference "R74") (unit 1)
-        )
-      )
+          (reference "R33") (unit 1)
+        )
+        (path "/dc2801a1-d539-4721-b31f-fe196b9f13df/8888f9b5-1ed7-43cb-9174-e948cce171c0"
+          (reference "R37") (unit 1)
+        )
+      )
