File: hardware/revB/payload-interface-board.kicad_pcb (KiCad board)
At the start: 6 copper layers, 90.2 x 101.1 mm, 201 parts, among them J1 T1M-10-F-SV-L, J2 T1M-6-F-SV-L, J3 T1M-10-F-SV-L, P1 Card Edge for HSEC8-160-01-S-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, Q1 MMBT4401WT1G, Q10 BSS138DWQ-7, Q11 BSS138DWQ-7, Q12 MMBT4403WT1G, Q13 IRF7404TRPBF, Q14 MMBT4401WT1G, Q15 MMDT5551-7-F, Q16 MMDT5551-7-F, Q17 BSS138DWQ-7, Q18 BSS138DWQ-7, Q19 IRF7404TRPBF, Q2 IRF7404TRPBF, Q20 MMBT4401WT1G, Q3 MMBT4401WT1G, Q4 BC847BM3T5G, Q5 BC847BM3T5G, Q6 BC847BM3T5G, Q7 BC847BM3T5G, Q8 MMDT5551-7-F, Q9 MMDT5551-7-F, U1 LTC4307, U10 MAX7311AAG+, U11 OPA340MDBVTEP, U12 DRV8838DSGT, U13 INA240A3EDRQ1, U14 INA240A3EDRQ1, U15 DRV8838DSGT, U16 INA240A3EDRQ1, U17 OPA340MDBVTEP, U18 OPA340MDBVTEP, U19 imu-stamp-revA, U2 SN74LVCH245APWR, U20 OPA340MDBVTEP, U21 ADM1176-1ARMZ-R7, U22 Pico, U3 SN74LVCH245APWR, U4 RockBlock_9603, U5 DRV8838DSGT, U6 MCP47FVB24-E/MQ, U7 ALM2402QPWPRQ1, U8 ALM2402QPWPRQ1, U9 AD7091R-5BCPZ-RL7

Commit message: working
Parts:
- removed the C11 at (59.5, 87.0)
- removed the C12 at (59.3, 89.0)
- removed the C13 at (69.2, 92.5)
- removed the C14 at (69.2, 95.8)
- removed the C15 at (69.3, 97.8)
- removed the C18 at (82.3, 98.3)
- removed the C19 at (47.8, 104.0)
- removed the C20 at (48.1, 106.0)
- removed the C21 at (44.3, 109.1)
- removed the C22 at (46.3, 109.3)
- removed the C23 at (42.9, 85.1)
- removed the C24 at (54.4, 107.0)
- removed the C25 at (50.6, 114.4)
- removed the C26 at (54.4, 110.6)
- removed the C27 at (50.6, 105.0)
- removed the C5 at (121.9, 68.8)
- removed the C6 at (116.5, 68.8)
- removed D3: SK6805-EC3210R, payload-interface-board:SK6812-EC3210F-RA
- removed D4: RED, SLI-Backplane-Blank-Card-KiCad:APA2107x
- removed D5: YELLOW, SLI-Backplane-Blank-Card-KiCad:APA2107x
- removed D6: GREEN, SLI-Backplane-Blank-Card-KiCad:APA2107x
- removed the D7 at (55.9, 65.0)
- removed the D8 at (69.0, 104.5)
- removed the D9 at (81.8, 104.5)
- removed G***: LOGO, payload-interface-board:Sierra_Lobo_Logo
- removed H1, H2, H3, H4: SLI-Backplane-Blank-Card-KiCad:125mil_hole, SLI-Backplane-Blank-Card-KiCad:125mil_hole
- removed the R18 at (52.4, 68.1)
- removed the R19 at (47.6, 67.1)
- removed the R26 at (50.6, 115.9)
- removed the R28 at (56.0, 110.6)
- removed the R30 at (45.0, 81.5)
- removed the R31 at (74.5, 108.2)
- removed the R32 at (82.7, 108.2)
- removed the R33 at (58.8, 110.7)
- removed the R34 at (56.5, 114.3)
- removed the R35 at (115.1, 85.1)
- removed the R36 at (115.1, 80.5)
- removed the R37 at (113.5, 85.1)
- removed the R38 at (113.5, 80.5)
- removed the R39 at (118.1, 85.1)
- removed the R53 at (65.8, 84.8)
- removed the R54 at (110.2, 113.0)
- removed the R55 at (125.7, 107.7)
- removed the R56 at (121.9, 107.7)
- removed the R57 at (110.2, 107.4)
- removed the R58 at (118.1, 107.7)
- removed the R59 at (80.5, 83.8)
- removed the R61 at (104.2, 143.5)
- removed the R62 at (100.8, 143.0)
- removed the R63 at (104.6, 137.8)
- removed the R64 at (98.2, 157.5)
- removed the R65 at (115.1, 93.9)
- removed the R66 at (115.1, 89.7)
- removed the R67 at (113.5, 93.9)
- removed RN10, RN11, RN9: MAX5490GC01000+T, Package_TO_SOT_SMD:SOT-23
- removed the RN6 at (50.0, 99.8)
- removed RN7, RN8: 1k, payload-interface-board:RAVF164D
- removed the U10 at (47.1, 92.5)
- removed the U11 at (59.9, 114.3)
- removed the U12 at (65.9, 101.7)
- removed the U13 at (66.0, 112.6)
- removed the U14 at (74.5, 112.6)
- removed the U17 at (73.2, 82.1)
- removed the U18 at (65.6, 82.1)
- removed the U20 at (84.0, 82.1)
- removed the U5 at (73.2, 101.8)
- removed the U6 at (61.3, 93.3)
- removed the U7 at (69.2, 90.0)
- removed the U8 at (81.9, 90.0)
- removed the U9 at (50.4, 110.3)
- added C11: 1uF, Capacitor_SMD:C_0603_1608Metric, F.Cu at (243.4, 64.0)
- added C11: 10uF, Capacitor_SMD:C_0805_2012Metric, F.Cu at (159.8, 117.1)
- added C12: 1uF, Capacitor_SMD:C_0603_1608Metric, F.Cu at (243.4, 66.5)
- added C12: 0.1uF, Capacitor_SMD:C_0402_1005Metric, F.Cu at (160.5, 119.1)
- added C13: 0.1uF, Capacitor_SMD:C_0402_1005Metric, F.Cu at (162.8, 117.8)
- added C13: 10uF, Capacitor_SMD:C_0805_2012Metric, F.Cu at (199.3, 70.2)
- added C14: 0.1uF, Capacitor_SMD:C_0402_1005Metric, F.Cu at (191.4, 64.7)
- added C14: 0.1uF, Capacitor_SMD:C_0402_1005Metric, F.Cu at (168.4, 117.1)
- added C15: 0.1uF, Capacitor_SMD:C_0402_1005Metric, F.Cu at (191.4, 66.7)
- added C15: 10nF, Capacitor_SMD:C_0402_1005Metric, F.Cu at (168.4, 118.3)
- added C18: 10uF, Capacitor_SMD:C_0805_2012Metric, F.Cu at (159.8, 140.2)
- added C18: 0.01uF, Capacitor_SMD:C_0402_1005Metric, F.Cu at (154.4, 105.2)
- added C19: 0.1uF, Capacitor_SMD:C_0402_1005Metric, F.Cu at (160.5, 142.2)
- added C19: 0.01uF, Capacitor_SMD:C_0402_1005Metric, F.Cu at (159.3, 105.2)
- added C2: 0.1uF, Capacitor_SMD:C_0402_1005Metric, F.Cu at (203.1, 102.2)
- added C20: 0.1uF, Capacitor_SMD:C_0402_1005Metric, F.Cu at (162.8, 141.0)
- added C20: 10uF, Capacitor_SMD:C_0805_2012Metric, F.Cu at (215.8, 70.2)
- added C21: 0.1uF, Capacitor_SMD:C_0402_1005Metric, F.Cu at (168.4, 140.2)
- added C21: 0.1uF, Capacitor_SMD:C_0402_1005Metric, F.Cu at (207.9, 64.7)
- added C22: 10nF, Capacitor_SMD:C_0402_1005Metric, F.Cu at (168.4, 141.5)
- added C22: 0.1uF, Capacitor_SMD:C_0402_1005Metric, F.Cu at (207.9, 66.7)
- added C23: 10uF, Capacitor_SMD:C_0805_2012Metric, F.Cu at (159.8, 128.3)
- added C23: 0.01uF, Capacitor_SMD:C_0402_1005Metric, F.Cu at (207.9, 68.6)
- added C24: 0.1uF, Capacitor_SMD:C_0402_1005Metric, F.Cu at (160.5, 130.3)
- added C24: 0.1uF, Capacitor_SMD:C_0402_1005Metric, F.Cu at (207.9, 70.6)
- added C25: 10uF, Capacitor_SMD:C_0805_2012Metric, F.Cu at (237.2, 73.8)
- added C25: 0.1uF, Capacitor_SMD:C_0402_1005Metric, F.Cu at (162.8, 129.0)
- added C26: 0.1uF, Capacitor_SMD:C_0402_1005Metric, F.Cu at (229.3, 68.3)
- added C26: 0.1uF, Capacitor_SMD:C_0402_1005Metric, F.Cu at (168.4, 128.3)
- added C27: 0.1uF, Capacitor_SMD:C_0402_1005Metric, F.Cu at (229.3, 70.2)
- added C27: 10nF, Capacitor_SMD:C_0402_1005Metric, F.Cu at (168.4, 129.5)
- added C3: 10uF, Capacitor_SMD:C_0805_2012Metric, F.Cu at (209.6, 106.9)
- added C49: 6pF, Capacitor_SMD:C_0402_1005Metric, F.Cu at (199.2, 48.3)
- added C50: 0.1uF, Capacitor_SMD:C_0402_1005Metric, F.Cu at (202.1, 36.5)
- added C54: 1uF, Capacitor_SMD:C_0603_1608Metric, F.Cu at (147.5, 144.1)
- added C54: 0.1uF, Capacitor_SMD:C_0402_1005Metric, F.Cu at (202.1, 38.4)
- added C55: 0.1uF, Capacitor_SMD:C_0402_1005Metric, F.Cu at (202.1, 40.4)
- added C55: 0.1uF, Capacitor_SMD:C_0402_1005Metric, F.Cu at (146.0, 144.6)
- added C56: 0.1uF, Capacitor_SMD:C_0402_1005Metric, F.Cu at (202.1, 42.4)
- added C56: 1uF, Capacitor_SMD:C_0603_1608Metric, F.Cu at (146.8, 120.9)
- added C57: 0.1uF, Capacitor_SMD:C_0402_1005Metric, F.Cu at (145.3, 121.4)
- added C57: 0.1uF, Capacitor_SMD:C_0402_1005Metric, F.Cu at (202.1, 44.4)
- added C58: 0.01uF, Capacitor_SMD:C_0402_1005Metric, F.Cu at (141.2, 105.7)
- added C59: 0.01uF, Capacitor_SMD:C_0402_1005Metric, F.Cu at (146.1, 105.7)
- added C60: 1uF, Capacitor_SMD:C_0603_1608Metric, F.Cu at (146.8, 132.1)
- added C60: 1uF, Capacitor_SMD:C_0603_1608Metric, F.Cu at (227.0, 19.2)
- added C61: 0.1uF, Capacitor_SMD:C_0402_1005Metric, F.Cu at (245.7, 24.9)
- added C61: 0.1uF, Capacitor_SMD:C_0402_1005Metric, F.Cu at (145.3, 132.6)
- added C62: 1uF, Capacitor_SMD:C_0603_1608Metric, F.Cu at (227.0, 21.7)
- added C63: 1uF, Capacitor_SMD:C_0603_1608Metric, F.Cu at (227.0, 24.2)
- added C64: 1uF, Capacitor_SMD:C_0603_1608Metric, F.Cu at (227.0, 26.7)
- added C65: 0.1uF, Capacitor_SMD:C_0402_1005Metric, F.Cu at (245.7, 26.8)
- added C66: 1uF, Capacitor_SMD:C_0603_1608Metric, F.Cu at (246.5, 50.1)
- added C67: 10uF, Capacitor_SMD:C_0805_2012Metric, F.Cu at (246.7, 47.4)
- added C68: 1uF, Capacitor_SMD:C_0603_1608Metric, F.Cu at (227.0, 29.2)
- added C69: 0.1uF, Capacitor_SMD:C_0402_1005Metric, F.Cu at (245.7, 28.8)
- added C70: 47uF, Capacitor_Tantalum_SMD:CP_EIA-7343-43_Kemet-X, F.Cu at (237.9, 34.2)
- added C71: 47uF, Capacitor_Tantalum_SMD:CP_EIA-7343-43_Kemet-X, F.Cu at (237.9, 40.0)
- added C72: 10uF, Capacitor_SMD:C_0805_2012Metric, F.Cu at (227.2, 38.9)
- added C73: 47uF, Capacitor_Tantalum_SMD:CP_EIA-7343-43_Kemet-X, F.Cu at (87.1, 33.8)
- added C74: 10uF, Capacitor_SMD:C_0805_2012Metric, F.Cu at (104.1, 36.8)
- added C75: 10uF, Capacitor_SMD:C_0805_2012Metric, F.Cu at (101.9, 36.8)
- added C76: 0.1uF, Capacitor_SMD:C_0402_1005Metric, F.Cu at (105.9, 37.1)
- added C77: 0.1uF, Capacitor_SMD:C_0402_1005Metric, F.Cu at (108.2, 34.5)
- added C78: 10uF, Capacitor_SMD:C_0805_2012Metric, F.Cu at (110.7, 28.2)
- added C79: 10uF, Capacitor_SMD:C_0805_2012Metric, F.Cu at (113.0, 28.2)
- added C80: DNP, Capacitor_SMD:C_0603_1608Metric, F.Cu at (105.4, 40.9)
- added C81: 1uF, Capacitor_SMD:C_0603_1608Metric, F.Cu at (233.0, 112.1)
- added C82: 0.1uF, Capacitor_SMD:C_0402_1005Metric, F.Cu at (240.7, 111.8)
- added C83: 1uF, Capacitor_SMD:C_0603_1608Metric, F.Cu at (233.0, 114.6)
- added C84: 0.1uF, Capacitor_SMD:C_0402_1005Metric, F.Cu at (240.7, 113.8)
- added C85: 1uF, Capacitor_SMD:C_0603_1608Metric, F.Cu at (233.0, 117.1)
- added C86: 0.1uF, Capacitor_SMD:C_0402_1005Metric, F.Cu at (240.7, 115.8)
- added D11: SK6805-EC3210R, payload-interface-board:SK6812-EC3210F-RA, F.Cu at (214.6, 49.9)
- added D12: SK6805-EC3210R, payload-interface-board:SK6812-EC3210F-RA, F.Cu at (214.6, 53.0)
- added D13: SK6805-EC3210R, payload-interface-board:SK6812-EC3210F-RA, F.Cu at (214.6, 56.1)
- added D14: B260S1F-7, Diode_SMD:D_SOD-123F, F.Cu at (112.0, 34.0)
- added D7: SP1326-01LTG, Diode_SMD:D_SOD-523, F.Cu at (164.6, 124.7)
- added D7: SP1326-01LTG, Diode_SMD:D_SOD-523, F.Cu at (199.1, 60.4)
- added D8: SP1326-01LTG, Diode_SMD:D_SOD-523, F.Cu at (164.6, 147.8)
- added D8: SP1326-01LTG, Diode_SMD:D_SOD-523, F.Cu at (215.6, 60.4)
- added D9: SP1326-01LTG, Diode_SMD:D_SOD-523, F.Cu at (164.6, 135.9)
- added D9: SP1326-01LTG, Diode_SMD:D_SOD-523, F.Cu at (237.0, 64.0)
- added J4: Conn_01x02, Connector_PinHeader_2.54mm:PinHeader_1x02_P2.54mm_Vertical_SMD_Pin1Left, F.Cu at (249.4, 66.3)
- added J5: JST 03B-SR, Connector_JST:JST_SH_SM03B-SRSS-TB_1x03-1MP_P1.00mm_Horizontal, F.Cu at (191.0, 39.3)
- added J6: JST 03B-SR, Connector_JST:JST_SH_SM03B-SRSS-TB_1x03-1MP_P1.00mm_Horizontal, F.Cu at (191.0, 46.9)
- added JP1: Wire Cut Jumper, Resistor_SMD:R_0603_1608Metric, F.Cu at (243.4, 69.0)
- added JP2: Wire Cut Jumper, Resistor_SMD:R_0603_1608Metric, F.Cu at (189.1, 24.2)
- added JP3: Wire Cut Jumper, Resistor_SMD:R_0603_1608Metric, F.Cu at (189.1, 26.7)
- added L1: 22uH, Inductor_SMD:L_Vishay_IHLP-2525, F.Cu at (118.1, 31.0)
- added Q21: BSS138DWQ-7, Package_TO_SOT_SMD:SOT-363_SC-70-6, F.Cu at (140.0, 103.4)
- added Q22: BSS138DWQ-7, Package_TO_SOT_SMD:SOT-363_SC-70-6, F.Cu at (144.8, 103.4)
- added R10: 988k, Resistor_SMD:R_0603_1608Metric, F.Cu at (202.7, 122.4)
- added R100: 0, Resistor_SMD:R_0603_1608Metric, F.Cu at (197.1, 26.7)
- added R101: 330, Resistor_SMD:R_0603_1608Metric, F.Cu at (149.3, 144.1)
- added R101: 0, Resistor_SMD:R_0603_1608Metric, F.Cu at (197.1, 29.2)
- added R102: 0, Resistor_SMD:R_0603_1608Metric, F.Cu at (197.1, 31.7)
- added R103: 10k, Resistor_SMD:R_0402_1005Metric, F.Cu at (207.9, 38.5)
- added R104: 0, Resistor_SMD:R_0603_1608Metric, F.Cu at (197.1, 34.2)
- added R105: 10k, Resistor_SMD:R_0402_1005Metric, F.Cu at (207.9, 40.5)
- added R106: 0, Resistor_SMD:R_0603_1608Metric, F.Cu at (201.1, 19.2)
- added R107: 0, Resistor_SMD:R_0603_1608Metric, F.Cu at (201.1, 21.7)
- added R108: 330, Resistor_SMD:R_0603_1608Metric, F.Cu at (201.1, 24.2)
- added R108: 1k, Resistor_SMD:R_0402_1005Metric, F.Cu at (138.8, 143.9)
- added R109: 100, Resistor_SMD:R_0603_1608Metric, F.Cu at (201.1, 26.7)
- added R11: 4.7k, Resistor_SMD:R_0603_1608Metric, F.Cu at (202.7, 117.3)
- added R110: 1k, Resistor_SMD:R_0402_1005Metric, F.Cu at (138.8, 145.1)
- added R110: 100, Resistor_SMD:R_0603_1608Metric, F.Cu at (201.1, 29.2)
- added R111: 1k, Resistor_SMD:R_0402_1005Metric, F.Cu at (138.8, 146.4)
- added R111: 0, Resistor_SMD:R_0603_1608Metric, F.Cu at (201.1, 31.7)
- added R112: 0, Resistor_SMD:R_0603_1608Metric, F.Cu at (201.1, 34.2)
- added R112: 330, Resistor_SMD:R_0603_1608Metric, F.Cu at (148.6, 120.9)
- added R113: 10k, Resistor_SMD:R_0402_1005Metric, F.Cu at (207.9, 42.5)
- added R113: 1k, Resistor_SMD:R_0402_1005Metric, F.Cu at (138.2, 120.7)
- added R114: 1k, Resistor_SMD:R_0402_1005Metric, F.Cu at (138.2, 122.0)
- added R114: 0, Resistor_SMD:R_0603_1608Metric, F.Cu at (205.1, 19.2)
- added R115: 1k, Resistor_SMD:R_0402_1005Metric, F.Cu at (138.2, 123.2)
- added R115: 0, Resistor_SMD:R_0603_1608Metric, F.Cu at (205.1, 21.7)
- added R116: 100, Resistor_SMD:R_0603_1608Metric, F.Cu at (205.1, 24.2)
- added R117: 100, Resistor_SMD:R_0603_1608Metric, F.Cu at (205.1, 26.7)
- added R118: 10k, Resistor_SMD:R_0402_1005Metric, F.Cu at (207.9, 44.4)
- added R119: ?, Resistor_SMD:R_0603_1608Metric, F.Cu at (205.1, 29.2)
- added R120: 330, Resistor_SMD:R_0603_1608Metric, F.Cu at (148.6, 132.1)
- added R120: ?, Resistor_SMD:R_0603_1608Metric, F.Cu at (205.1, 31.7)
- added R121: 1k, Resistor_SMD:R_0402_1005Metric, F.Cu at (138.2, 131.8)
- added R121: ?, Resistor_SMD:R_0603_1608Metric, F.Cu at (205.1, 34.2)
- added R122: 10k, Resistor_SMD:R_0402_1005Metric, F.Cu at (207.9, 46.4)
- added R123: 1k, Resistor_SMD:R_0402_1005Metric, F.Cu at (210.8, 36.5)
- added R123: 1k, Resistor_SMD:R_0402_1005Metric, F.Cu at (138.2, 133.1)
- added R124: 1k, Resistor_SMD:R_0402_1005Metric, F.Cu at (210.8, 38.5)
- added R124: 1k, Resistor_SMD:R_0402_1005Metric, F.Cu at (138.2, 134.4)
- added R125: 1k, Resistor_SMD:R_0402_1005Metric, F.Cu at (210.8, 40.5)
- added R126: 1k, Resistor_SMD:R_0402_1005Metric, F.Cu at (210.8, 42.5)
- added R127: 1k, Resistor_SMD:R_0402_1005Metric, F.Cu at (210.8, 44.4)
- added R128: 10k, Resistor_SMD:R_0402_1005Metric, F.Cu at (141.0, 100.6)
- added R129: 10k, Resistor_SMD:R_0402_1005Metric, F.Cu at (146.1, 100.6)
- added R130: 10k, Resistor_SMD:R_0402_1005Metric, F.Cu at (139.2, 100.1)
- added R131: 10k, Resistor_SMD:R_0402_1005Metric, F.Cu at (144.3, 100.1)
- added R132: 680, Resistor_SMD:R_0603_1608Metric, F.Cu at (140.0, 95.5)
- added R133: 680, Resistor_SMD:R_0603_1608Metric, F.Cu at (144.8, 95.5)
- added R134: 100k, Resistor_SMD:R_0402_1005Metric, F.Cu at (138.9, 105.7)
- added R135: 100k, Resistor_SMD:R_0402_1005Metric, F.Cu at (143.8, 105.7)
- added R136: 200K, Resistor_SMD:R_0402_1005Metric, F.Cu at (139.2, 101.1)
- added R137: 200K, Resistor_SMD:R_0402_1005Metric, F.Cu at (144.3, 101.1)
- added R138: 0, Resistor_SMD:R_0603_1608Metric, F.Cu at (140.0, 93.7)
- added R139: 0, Resistor_SMD:R_0603_1608Metric, F.Cu at (144.8, 93.7)
- added R140: 330, Resistor_SMD:R_0603_1608Metric, F.Cu at (227.0, 31.7)
- added R141: 300mR, Resistor_SMD:R_0805_2012Metric, F.Cu at (245.1, 32.7)
- added R142: 1k, Resistor_SMD:R_0402_1005Metric, F.Cu at (239.6, 18.9)
- added R143: 1k, Resistor_SMD:R_0402_1005Metric, F.Cu at (239.6, 20.9)
- added R144: 1k, Resistor_SMD:R_0402_1005Metric, F.Cu at (239.6, 22.9)
- added R145: 330, Resistor_SMD:R_0603_1608Metric, F.Cu at (231.0, 19.2)
- added R146: 300mR, Resistor_SMD:R_0805_2012Metric, F.Cu at (245.1, 35.7)
- added R147: 1k, Resistor_SMD:R_0402_1005Metric, F.Cu at (242.5, 18.9)
- added R148: 1k, Resistor_SMD:R_0402_1005Metric, F.Cu at (242.5, 20.9)
- added R149: 1k, Resistor_SMD:R_0402_1005Metric, F.Cu at (242.5, 22.9)
- added R150: 10k, Resistor_SMD:R_0603_1608Metric, F.Cu at (231.0, 21.7)
- added R151: 12.4k, Resistor_SMD:R_0603_1608Metric, F.Cu at (231.0, 24.2)
- added R152: 330, Resistor_SMD:R_0603_1608Metric, F.Cu at (231.0, 26.7)
- added R153: 4.1k, Resistor_SMD:R_0603_1608Metric, F.Cu at (231.0, 29.2)
- added R154: ?, Resistor_SMD:R_0805_2012Metric, F.Cu at (245.1, 38.6)
- added R155: 1k, Resistor_SMD:R_0402_1005Metric, F.Cu at (245.4, 18.9)
- added R156: 1k, Resistor_SMD:R_0402_1005Metric, F.Cu at (245.4, 20.9)
- added R157: 1k, Resistor_SMD:R_0402_1005Metric, F.Cu at (245.4, 22.9)
- added R158: 1k, Resistor_SMD:R_0402_1005Metric, F.Cu at (101.9, 40.4)
- added R159: 49.9k, Resistor_SMD:R_0603_1608Metric, F.Cu at (103.6, 40.9)
- added R160: 100k, Resistor_SMD:R_0603_1608Metric, F.Cu at (118.4, 39.6)
- added R161: 29.4k, Resistor_SMD:R_0603_1608Metric, F.Cu at (116.6, 39.6)
- added R162: 100k, Resistor_SMD:R_0402_1005Metric, F.Cu at (120.1, 39.1)
- added R163: 220, Resistor_SMD:R_0603_1608Metric, F.Cu at (233.0, 119.6)
- added R164: 220, Resistor_SMD:R_0603_1608Metric, F.Cu at (233.0, 122.1)
- added R165: 220, Resistor_SMD:R_0603_1608Metric, F.Cu at (233.0, 124.7)
- added R30: 110k, Resistor_SMD:R_0603_1608Metric, F.Cu at (194.8, 65.0)
- added R30: 300mR, Resistor_SMD:R_0805_2012Metric, F.Cu at (168.6, 148.2)
- added R31: 300mR, Resistor_SMD:R_0805_2012Metric, F.Cu at (168.4, 124.7)
- added R31: 1k, Resistor_SMD:R_0402_1005Metric, F.Cu at (188.5, 60.1)
- added R32: ?, Resistor_SMD:R_0805_2012Metric, F.Cu at (168.4, 136.0)
- added R32: 100k, Resistor_SMD:R_0402_1005Metric, F.Cu at (188.5, 62.1)
- added R33: 110k, Resistor_SMD:R_0603_1608Metric, F.Cu at (194.8, 67.5)
- added R33: 110k, Resistor_SMD:R_0603_1608Metric, F.Cu at (152.8, 123.0)
- added R34: 1k, Resistor_SMD:R_0402_1005Metric, F.Cu at (157.0, 118.9)
- added R34: 1k, Resistor_SMD:R_0402_1005Metric, F.Cu at (188.5, 64.1)
- added R35: 110k, Resistor_SMD:R_0603_1608Metric, F.Cu at (152.8, 121.2)
- added R35: 1k, Resistor_SMD:R_0402_1005Metric, F.Cu at (188.5, 66.1)
- added R36: 1k, Resistor_SMD:R_0402_1005Metric, F.Cu at (164.1, 117.8)
- added R36: 100k, Resistor_SMD:R_0402_1005Metric, F.Cu at (188.5, 68.1)
- added R37: 1k, Resistor_SMD:R_0402_1005Metric, F.Cu at (188.5, 70.1)
- added R37: 1k, Resistor_SMD:R_0402_1005Metric, F.Cu at (165.4, 117.8)
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- renumbered RN2 to RN3, RN3 to RN4, RN4 to RN6, U2 to U3, U3 to U5
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Connections:
- net /H1-17 renamed /RX_4
- net /H1-18 renamed /TX_4
- net /H1-19 renamed /RX_2
- net /H1-20 renamed /TX_2
- net /H1-39 renamed /RX_3
- net /H1-40 renamed /TX_3
- net /H1-6 renamed /PYLD_RESET
- C1 pad 1: +3.3V -> LED_VCC
- C10 pad 2: /CHS -> Net-(C10-Pad2)
- C16 pad 1: +5V -> /MTQ Control/3V3A
- C17 pad 1: +5V -> /MTQ Control/3V3A
- C28 pad 1: /MT Drivers/2.5V_ADCout -> /MTQ Control/3V3A
- C29 pad 1: +3.3V -> /MTQ Control/3V3A
- C30 pad 1: GND -> +5V
- C30 pad 2: Net-(U11-+) -> Net-(Q12-C)
- C31 pad 1: Net-(Q10B-G1) -> 5V_PL
- C31 pad 2: GND -> Net-(Q15-C)
- C32 pad 1: Net-(Q11B-G1) -> /MTQ Control/5VIN
- C32 pad 2: GND -> Net-(Q18-C)
- C33 pad 1: +3.3V -> /MTQ Control/3V3D
- C34 pad 1: +3.3V -> +1V1
- C35 pad 1: +3.3V -> +1V1
- C36 pad 1: +3.3V -> /MTQ Control/3V3D
- C37 pad 1: +3.3V -> /MTQ Control/3V3D
- C38 pad 1: +3.3V -> /MTQ Control/3V3D
- C39 pad 1: +3.3V -> /MTQ Control/3V3D
- C40 pad 1: +3.3V -> /MTQ Control/3V3D
- C41 pad 1: +5V -> /MTQ Control/3V3D
- C42 pad 1: +5V -> /MTQ Control/3V3D
- C43 pad 1: +3.3V -> /MTQ Control/3V3D
- C44 pad 1: +5V -> /MTQ Control/3V3D
- C45 pad 1: Net-(U21-TIMER) -> /MTQ Control/3V3D
- C46 pad 1: Net-(Q17B-G1) -> +1V1
- C47 pad 1: Net-(Q18B-G1) -> /MTQ Control/MCU/3V3A
- C48 pad 1: Net-(D10-A) -> /MTQ Control/MCU/XIN
- C7 pad 2: /CHS -> Net-(C7-Pad2)
- C8 pad 2: /CHS -> Net-(C8-Pad2)
- C9 pad 2: /CHS -> Net-(C9-Pad2)
- D1 pad 1: /MT Drivers/Full Bridge 2/OUT2 -> GND
- D1 pad 2: /MT Drivers/Y+ -> Net-(D1-DOUT)
- D10 pad 1: Net-(D10-K) -> GND
- D10 pad 2: Net-(D10-A) -> Net-(D10-DOUT)
- D2 pad 2: Net-(D2-DOUT) -> /DOUT
- D2 pad 3: Net-(D2-DIN) -> Net-(D1-DOUT)
- D2 pad 4: +3.3V -> LED_VCC
- J1 pad 2: /RB_CTS -> unconnected-(J1-Pin_2-Pad2)
- J1 pad 3: /RB_RTS -> unconnected-(J1-Pin_3-Pad3)
- J1 pad 4: /RB_NetAv -> unconnected-(J1-Pin_4-Pad4)
- J1 pad 5: /RB_RI -> unconnected-(J1-Pin_5-Pad5)
- J1 pad 7: /RB_OnOff -> /OnOff
- J1 pad 8: /RB_5V_IN -> /RB_Vcc
- J1 pad 9: /RB_Li-iON -> unconnected-(J1-Pin_9-Pad9)
- J2 pad 1: /MT Drivers/X- -> /X-
- J2 pad 2: /MT Drivers/X+ -> /X+
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Routing:
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- added copper zone on B.Cu, net unconnected-(P1-Pin_74-Pad74)
- removed copper zone on B.Cu, net +3.3V
- removed copper zone on B.Cu, net +5V
- removed copper zone on B.Cu, net /MT Drivers/Full Bridge 1/OUT2
- removed copper zone on B.Cu, net /MT Drivers/Full Bridge 2/OUT2
- removed copper zone on B.Cu, net /MT Drivers/Full Bridge 3/OUT2
- removed copper zone on B.Cu, net /MT Drivers/X+
- removed copper zone on B.Cu, net /MT Drivers/X_Drive
- removed copper zone on B.Cu, net /MT Drivers/Y+
- removed copper zone on B.Cu, net /MT Drivers/Y_Drive
- removed copper zone on B.Cu, net /MT Drivers/Z+
- removed copper zone on B.Cu, net /MT Drivers/Z_drive
- removed copper zone on B.Cu, net /Payload Interface/5V_PYLD
- removed copper zone on F.Cu, net /Payload Interface/5V_PYLD
- removed copper zone on B.Cu, net /Payload Interface/5V_sns
- removed copper zone on F.Cu, net /RB_5V_IN
- removed copper zone on B.Cu, net 5V_RF
- removed copper zone on F.Cu, net 5V_RF
- removed copper zone on B.Cu, net Net-(D10-A)
Other:
- board text removed: "Foras Promineo Payload Interface Board C.Hillis 2/21"

Commit message: revB initial commit
Parts:
- removed the C1 at (203.1, 100.2)
- removed the C11 at (243.4, 64.0)
- removed the C11 at (159.8, 117.1)
- removed the C12 at (243.4, 66.5)
- removed the C12 at (160.5, 119.1)
- removed the C13 at (162.8, 117.8)
- removed the C13 at (199.3, 70.2)
- removed the C14 at (191.4, 64.7)
- removed the C14 at (168.4, 117.1)
- removed the C15 at (191.4, 66.7)
- removed the C15 at (168.4, 118.3)
- removed the C16 at (191.4, 68.6)
- removed C17, C19, C20, C21 (x2), C22, C24 (x2), C25, C26 (x2), C27, C29, C32, C33, C34, C35, C36, C37, C38, C39, C40, C41, C42, C43, C47, C50, C54, C55 (x2), C56, C57 (x2), C61 (x2), C65, C69, C76, C77, C82, C84, C86: 0.1uF, Capacitor_SMD:C_0402_1005Metric
- removed C18, C20, C23, C25, C44, C67, C72, C74, C75, C78, C79: 10uF, Capacitor_SMD:C_0805_2012Metric
- removed C18, C19, C23, C28: 0.01uF, Capacitor_SMD:C_0402_1005Metric
- removed the C2 at (203.1, 102.2)
- removed C22, C27: 10nF, Capacitor_SMD:C_0402_1005Metric
- removed C45, C46, C54, C56, C60 (x2), C62, C63, C64, C66, C68, C81, C83, C85: 1uF, Capacitor_SMD:C_0603_1608Metric
- removed C48, C49: 6pF, Capacitor_SMD:C_0402_1005Metric
- removed C70, C71, C73: 47uF, Capacitor_Tantalum_SMD:CP_EIA-7343-43_Kemet-X
- removed C80: DNP, Capacitor_SMD:C_0603_1608Metric
- removed D10, D11, D12, D13: SK6805-EC3210R, payload-interface-board:SK6812-EC3210F-RA
- removed D14: B260S1F-7, Diode_SMD:D_SOD-123F
- removed D7 (x2), D8 (x2), D9 (x2): SP1326-01LTG, Diode_SMD:D_SOD-523
- removed the J2 at (50.5, 98.8)
- removed J4: Conn_01x02, Connector_PinHeader_2.54mm:PinHeader_1x02_P2.54mm_Vertical_SMD_Pin1Left
- removed J5, J6: JST 03B-SR, Connector_JST:JST_SH_SM03B-SRSS-TB_1x03-1MP_P1.00mm_Horizontal
- removed JP1, JP2, JP3: Wire Cut Jumper, Resistor_SMD:R_0603_1608Metric
- removed L1: 22uH, Inductor_SMD:L_Vishay_IHLP-2525
- removed the Q1 at (205.9, 100.6)
- removed Q16, Q17: BSZ180, SierraLobo:PG-TSDSON-8_3.3x3.3mm
- removed Q18: MMBT4401WT1G, Package_TO_SOT_SMD:SOT-323_SC-70
- removed Q19, Q20: MMDT5551-7-F, Package_TO_SOT_SMD:SOT-363_SC-70-6
- removed Q21, Q22: BSS138DWQ-7, Package_TO_SOT_SMD:SOT-363_SC-70-6
- removed the Q4 at (205.9, 109.2)
- removed the Q6 at (153.2, 97.3)
- removed the Q7 at (158.0, 97.3)
- removed the Q8 at (153.2, 102.9)
- removed the Q9 at (158.0, 102.9)
- removed the R1 at (214.2, 117.1)
- removed R100, R101, R102, R104, R106, R107, R111, R112, R114, R115, R83, R85, R89, R90, R91, R92, R93, R94, R95, R96, R97, R98, R99: 0, Resistor_SMD:R_0603_1608Metric
- removed R101, R108, R112, R120, R140, R145, R152: 330, Resistor_SMD:R_0603_1608Metric
- removed R103, R105, R113, R118, R122, R78, R86, R87, R88: 10k, Resistor_SMD:R_0402_1005Metric
- removed R108, R110, R111, R113, R114, R115, R121, R123 (x2), R124 (x2), R125, R126, R127, R142, R143, R144, R147, R148, R149, R155, R156, R157, R158, R54 (x2), R55, R56, R57 (x2), R59 (x2), R62 (x2), R63, R64, R65 (x2), R67, R75, R76, R79, R81, R84: 1k, Resistor_SMD:R_0402_1005Metric
- removed R109, R110, R116, R117: 100, Resistor_SMD:R_0603_1608Metric
- removed R119, R120, R121: ?, Resistor_SMD:R_0603_1608Metric
- removed R141, R146: 300mR, Resistor_SMD:R_0805_2012Metric
- removed R150: 10k, Resistor_SMD:R_0603_1608Metric
- removed R151: 12.4k, Resistor_SMD:R_0603_1608Metric
- removed R153: 4.1k, Resistor_SMD:R_0603_1608Metric
- removed R154: ?, Resistor_SMD:R_0805_2012Metric
- removed R159: 49.9k, Resistor_SMD:R_0603_1608Metric
- removed R160: 100k, Resistor_SMD:R_0603_1608Metric
- removed R161: 29.4k, Resistor_SMD:R_0603_1608Metric
- removed R162, R56, R58, R60, R64, R66, R74, R77: 100k, Resistor_SMD:R_0402_1005Metric
- removed R163, R164, R165: 220, Resistor_SMD:R_0603_1608Metric
- removed the R3 at (214.2, 121.1)
- removed the R30 at (194.8, 65.0)
- removed the R30 at (168.6, 148.2)
- removed the R31 at (168.4, 124.7)
- removed the R31 at (188.5, 60.1)
- removed the R32 at (168.4, 136.0)
- removed the R32 at (188.5, 62.1)
- removed the R33 at (194.8, 67.5)
- removed the R33 at (152.8, 123.0)
- removed the R34 at (157.0, 118.9)
- removed the R34 at (188.5, 64.1)
- removed the R35 at (152.8, 121.2)
- removed the R35 at (188.5, 66.1)
- removed the R36 at (164.1, 117.8)
- removed the R36 at (188.5, 68.1)
- removed the R37 at (188.5, 70.1)
- removed the R37 at (165.4, 117.8)
- removed the R38 at (163.6, 116.1)
- removed the R38 at (154.2, 100.1)
- removed the R39 at (159.3, 100.1)
- removed the R39 at (166.6, 117.8)
- removed the R4 at (214.2, 123.1)
- removed the R40 at (152.4, 99.6)
- removed the R41 at (157.5, 99.6)
- removed the R42 at (153.2, 95.0)
- removed the R43 at (158.0, 95.0)
- removed the R44 at (152.1, 105.2)
- removed the R45 at (157.0, 105.2)
- removed the R46 at (152.4, 100.6)
- removed the R47 at (157.5, 100.6)
- removed the R48 at (153.2, 93.2)
- removed the R49 at (158.0, 93.2)
- removed the R5 at (217.1, 117.1)
- removed the R50 at (211.3, 65.0)
- removed the R51 at (205.0, 60.1)
- removed the R52 at (205.0, 62.1)
- removed R53 (x2), R55, R58, R61 (x2), R63: 110k, Resistor_SMD:R_0603_1608Metric
- removed the R7 at (217.1, 121.1)
- removed the R8 at (217.1, 123.1)
- removed R80, R82: 27, Capacitor_SMD:C_0402_1005Metric
- removed the R9 at (220.0, 117.1)
- removed SW1, SW2: KMR231NG LFS, SierraLobo:KMR2_4.6X2.8
- removed U10, U11, U13, U14, U8: DRV8838DSGT, Package_SON:WSON-8-1EP_2x2mm_P0.5mm_EP0.9x1.6mm
- removed U10, U12, U13, U9: TLV4110xDGN, Package_SO:MSOP-8-1EP_3x3mm_P0.65mm_EP1.68x1.88mm
- removed U11, U12, U14, U15, U8, U9: INA199A2xDCK, Package_TO_SOT_SMD:SOT-363_SC-70-6
- removed U16: MR25H10MDF, Package_DFN_QFN:DFN-8-1EP_6x5mm_P1.27mm_EP2x2mm
- removed U17: RP2040, Package_DFN_QFN:QFN-56-1EP_7x7mm_P0.4mm_EP3.2x3.2mm_ThermalVias
- removed U17, U18, U20 (x2), U22, U24: DAC121S101Q, Package_TO_SOT_SMD:TSOT-23-6
- removed U18: ATSAMD51J19A-AU, Package_QFP:TQFP-64_10x10mm_P0.5mm
- removed U19: MAX708RESA-T, Package_SO:SO-8_3.9x4.9mm_P1.27mm
- removed U21: MCP1700T-33, Package_TO_SOT_SMD:SOT-89-3
- removed U23: ATL431BQ, Package_TO_SOT_SMD:SOT-23
- removed U25: LMR16020, Package_SO:Texas_HSOP-8-1EP_3.9x4.9mm_P1.27mm_ThermalVias
- removed U26, U27, U28: MCP9700AT-E/LT, Package_TO_SOT_SMD:SOT-353_SC-70-5
- removed the U4 at (65.3, 138.8)
- removed the U6 at (248.0, 72.1)
- removed the U6 at (158.5, 122.2)
- removed the U7 at (193.6, 61.4)
- removed the U7 at (164.6, 121.6)
- added C4: 1uF, Capacitor_SMD:C_0603_1608Metric, F.Cu at (111.0, 123.7)
- added C5: 0.1uF, Capacitor_SMD:C_0603_1608Metric, F.Cu at (113.5, 120.9)
- added C7: 1uF, Capacitor_SMD:C_0603_1608Metric, F.Cu at (46.7, 111.0)
- added C8: 0.1uF, Capacitor_SMD:C_0603_1608Metric, F.Cu at (49.3, 108.2)
- added D3: ORANGE, SierraLobo:APA2107x, F.Cu at (49.7, 65.4)
- added D4: GREEN, SierraLobo:APA2107x, B.Cu at (55.0, 65.4)
- added G***: LOGO, SierraLobo:SLI_logo_15x9, F.Cu at (57.4, 85.9)
- added H1: SLI-Backplane-Blank-Card-KiCad:125mil_hole, SierraLobo:125mil_hole, F.Cu at (122.7, 74.5)
- added H2: SLI-Backplane-Blank-Card-KiCad:125mil_hole, SierraLobo:125mil_hole, F.Cu at (125.2, 160.3)
- added H3: SLI-Backplane-Blank-Card-KiCad:125mil_hole, SierraLobo:125mil_hole, F.Cu at (49.0, 74.5)
- added H4: SLI-Backplane-Blank-Card-KiCad:125mil_hole, SierraLobo:125mil_hole, F.Cu at (45.2, 160.3)
- added Q10: MMDT2222A, Package_TO_SOT_SMD:SOT-363_SC-70-6, F.Cu at (109.2, 85.0)
- added Q11: MMDT2222A, Package_TO_SOT_SMD:SOT-363_SC-70-6, F.Cu at (109.2, 80.2)
- added Q14: BSS138DWQ-7, Package_TO_SOT_SMD:SOT-363_SC-70-6, F.Cu at (118.9, 85.0)
- added Q15: BSS138DWQ-7, Package_TO_SOT_SMD:SOT-363_SC-70-6, F.Cu at (118.9, 80.2)
- added R11: 10k, Resistor_SMD:R_0603_1608Metric, F.Cu at (84.3, 79.2)
- added R15: 10k, Resistor_SMD:R_0603_1608Metric, F.Cu at (93.2, 92.5)
- added R19: 220, Resistor_SMD:R_0603_1608Metric, F.Cu at (109.5, 123.7)
- added R21: 220, Resistor_SMD:R_0603_1608Metric, F.Cu at (45.2, 111.0)
- added R26: 1.5k, Resistor_SMD:R_0402_1005Metric, B.Cu at (47.5, 67.1)
- added R27: 1.5k, Resistor_SMD:R_0402_1005Metric, F.Cu at (49.7, 67.1)
- added R28: 1.5k, Resistor_SMD:R_0402_1005Metric, B.Cu at (54.6, 67.1)
- added R30: 10k, Resistor_SMD:R_0402_1005Metric, B.Cu at (55.2, 70.0)
- added R31: 10k, Resistor_SMD:R_0402_1005Metric, F.Cu at (54.9, 70.0)
- added R32: 10k, Resistor_SMD:R_0402_1005Metric, F.Cu at (48.6, 69.6)
- added TP10: ${NET_NAME(1)}, TestPoint:TestPoint_Keystone_5000-5004_Miniature, F.Cu at (124.7, 140.5)
- added TP11: ${NET_NAME(1)}, TestPoint:TestPoint_Keystone_5000-5004_Miniature, F.Cu at (102.4, 160.8)
- added TP12: ${NET_NAME(1)}, TestPoint:TestPoint_Keystone_5000-5004_Miniature, F.Cu at (106.7, 160.8)
- added TP13: ${NET_NAME(1)}, TestPoint:TestPoint_Keystone_5000-5004_Miniature, F.Cu at (111.0, 160.8)
- added TP14: ${NET_NAME(1)}, TestPoint:TestPoint_Keystone_5000-5004_Miniature, F.Cu at (115.3, 160.8)
- added TP15: ${NET_NAME(1)}, SierraLobo:Keystone_5027, F.Cu at (124.7, 149.1)
- added TP16: ${NET_NAME(1)}, TestPoint:TestPoint_Keystone_5000-5004_Miniature, F.Cu at (124.7, 129.3)
- added TP17: ${NET_NAME(1)}, TestPoint:TestPoint_Keystone_5000-5004_Miniature, F.Cu at (46.0, 100.8)
- added TP18: ${NET_NAME(1)}, TestPoint:TestPoint_Keystone_5000-5004_Miniature, F.Cu at (124.7, 116.1)
- added TP19: ${NET_NAME(1)}, TestPoint:TestPoint_Keystone_5000-5004_Miniature, F.Cu at (124.7, 111.8)
- added TP2: ${NET_NAME(1)}, TestPoint:TestPoint_Keystone_5000-5004_Miniature, F.Cu at (46.0, 87.9)
- added TP20: ${NET_NAME(1)}, TestPoint:TestPoint_Keystone_5000-5004_Miniature, F.Cu at (124.7, 107.4)
- added TP21: ${NET_NAME(1)}, SierraLobo:Keystone_5027, F.Cu at (124.7, 124.7)
- added TP22: ${NET_NAME(1)}, TestPoint:TestPoint_Keystone_5000-5004_Miniature, F.Cu at (124.7, 120.4)
- added TP3: ${NET_NAME(1)}, TestPoint:TestPoint_Keystone_5000-5004_Miniature, F.Cu at (46.0, 92.2)
- added TP4: ${NET_NAME(1)}, TestPoint:TestPoint_Keystone_5000-5004_Miniature, F.Cu at (46.0, 83.6)
- added TP5: ${NET_NAME(1)}, TestPoint:TestPoint_Keystone_5000-5004_Miniature, F.Cu at (88.2, 102.6)
- added TP6: ${NET_NAME(1)}, TestPoint:TestPoint_Keystone_5000-5004_Miniature, F.Cu at (83.1, 102.6)
- added TP7: ${NET_NAME(1)}, SierraLobo:Keystone_5027, F.Cu at (46.0, 96.5)
- added TP9: ${NET_NAME(1)}, TestPoint:TestPoint_Keystone_5000-5004_Miniature, F.Cu at (124.7, 144.8)
- added U2: RockBlock_9603, SierraLobo:RockBlock_9603, F.Cu at (72.1, 137.5)
- added U5: MCP9700AT-E/LT, Package_TO_SOT_SMD:SOT-353_SC-70-5, F.Cu at (113.5, 123.7)
- added U7: MCP9700AT-E/LT, Package_TO_SOT_SMD:SOT-353_SC-70-5, F.Cu at (49.3, 111.0)
- C1: renamed from C4; footprint Capacitor_SMD:C_0402_1005Metric -> Capacitor_SMD:C_0603_1608Metric
- C10: renamed from C8; footprint Capacitor_SMD:C_0402_1005Metric -> Capacitor_SMD:C_0603_1608Metric
- C11: renamed from C9; footprint Capacitor_SMD:C_0402_1005Metric -> Capacitor_SMD:C_0603_1608Metric
- C12: renamed from C10; footprint Capacitor_SMD:C_0402_1005Metric -> Capacitor_SMD:C_0603_1608Metric
- C13: renamed from C30; footprint Capacitor_SMD:C_0402_1005Metric -> Capacitor_SMD:C_0603_1608Metric
- C14: renamed from C31; footprint Capacitor_SMD:C_0402_1005Metric -> Capacitor_SMD:C_0603_1608Metric
- C15: renamed from C58; footprint Capacitor_SMD:C_0402_1005Metric -> Capacitor_SMD:C_0603_1608Metric
- C16: renamed from C59; footprint Capacitor_SMD:C_0402_1005Metric -> Capacitor_SMD:C_0603_1608Metric
- C2: renamed from C5; footprint Capacitor_SMD:C_0402_1005Metric -> Capacitor_SMD:C_0603_1608Metric
- C3: renamed from C6; footprint Capacitor_SMD:C_0402_1005Metric -> Capacitor_SMD:C_0603_1608Metric
- C9: renamed from C7; footprint Capacitor_SMD:C_0402_1005Metric -> Capacitor_SMD:C_0603_1608Metric
- D1: value SK6805-EC3210R -> RED; footprint payload-interface-board:SK6812-EC3210F-RA -> SierraLobo:APA2107x; moved to B.Cu
- D2: value SK6805-EC3210R -> YELLOW; footprint payload-interface-board:SK6812-EC3210F-RA -> SierraLobo:APA2107x; moved to B.Cu
- Q2: value BC847BM3T5G -> MMDT2222A; footprint Package_TO_SOT_SMD:SOT-723 -> Package_TO_SOT_SMD:SOT-363_SC-70-6; moved to B.Cu
- Q3: value BC847BM3T5G -> MMDT2222A; footprint Package_TO_SOT_SMD:SOT-723 -> Package_TO_SOT_SMD:SOT-363_SC-70-6
- R1: renamed from R17; footprint Resistor_SMD:R_0402_1005Metric -> Resistor_SMD:R_0603_1608Metric
- R12: renamed from R16; footprint Resistor_SMD:R_0402_1005Metric -> Resistor_SMD:R_0603_1608Metric
- R13: renamed from R18; footprint Resistor_SMD:R_0402_1005Metric -> Resistor_SMD:R_0603_1608Metric
- R14: renamed from R19; footprint Resistor_SMD:R_0402_1005Metric -> Resistor_SMD:R_0603_1608Metric
- R16: renamed from R24; value 1k -> 10k; footprint Resistor_SMD:R_0402_1005Metric -> Resistor_SMD:R_0603_1608Metric
- R17: renamed from R26; footprint Resistor_SMD:R_0402_1005Metric -> Resistor_SMD:R_0603_1608Metric
- R18: renamed from R28; footprint Resistor_SMD:R_0402_1005Metric -> Resistor_SMD:R_0603_1608Metric
- R2: renamed from R20; footprint Resistor_SMD:R_0402_1005Metric -> Resistor_SMD:R_0603_1608Metric
- R22: renamed from R13; footprint Resistor_SMD:R_0402_1005Metric -> Resistor_SMD:R_0603_1608Metric
- R25: renamed from R2; moved to B.Cu
- R29: renamed from R6; value 1.5k -> 10k; moved to B.Cu
- R33: renamed from R66; footprint Resistor_SMD:R_0402_1005Metric -> Resistor_SMD:R_0603_1608Metric
- R34: renamed from R67; footprint Resistor_SMD:R_0402_1005Metric -> Resistor_SMD:R_0603_1608Metric
- R35: renamed from R68; footprint Resistor_SMD:R_0402_1005Metric -> Resistor_SMD:R_0603_1608Metric
- R36: renamed from R69; footprint Resistor_SMD:R_0402_1005Metric -> Resistor_SMD:R_0603_1608Metric
- R37: renamed from R70; footprint Resistor_SMD:R_0402_1005Metric -> Resistor_SMD:R_0603_1608Metric
- R38: renamed from R71; footprint Resistor_SMD:R_0402_1005Metric -> Resistor_SMD:R_0603_1608Metric
- R39: renamed from R72; footprint Resistor_SMD:R_0402_1005Metric -> Resistor_SMD:R_0603_1608Metric
- R40: renamed from R73; footprint Resistor_SMD:R_0402_1005Metric -> Resistor_SMD:R_0603_1608Metric
- R41: renamed from R128; footprint Resistor_SMD:R_0402_1005Metric -> Resistor_SMD:R_0603_1608Metric
- R42: renamed from R129; footprint Resistor_SMD:R_0402_1005Metric -> Resistor_SMD:R_0603_1608Metric
- R43: renamed from R130; footprint Resistor_SMD:R_0402_1005Metric -> Resistor_SMD:R_0603_1608Metric
- R44: renamed from R131; footprint Resistor_SMD:R_0402_1005Metric -> Resistor_SMD:R_0603_1608Metric
- R47: renamed from R134; footprint Resistor_SMD:R_0402_1005Metric -> Resistor_SMD:R_0603_1608Metric
- R48: renamed from R135; footprint Resistor_SMD:R_0402_1005Metric -> Resistor_SMD:R_0603_1608Metric
- R49: renamed from R136; footprint Resistor_SMD:R_0402_1005Metric -> Resistor_SMD:R_0603_1608Metric
- R5: renamed from R21; footprint Resistor_SMD:R_0402_1005Metric -> Resistor_SMD:R_0603_1608Metric
- R50: renamed from R137; footprint Resistor_SMD:R_0402_1005Metric -> Resistor_SMD:R_0603_1608Metric
- R6: renamed from R22; footprint Resistor_SMD:R_0402_1005Metric -> Resistor_SMD:R_0603_1608Metric
- RN1, RN3, RN4, RN6: footprint payload-interface-board:RAVF164D -> Resistor_SMD:R_Array_Convex_4x0402
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- renumbered C3 to C6, J3 to J2, Q5 to Q1, Q10 to Q4, Q11 to Q5, Q12 to Q6, Q13 to Q7, Q14 to Q8, Q15 to Q9, R29 to R10, R10 to R20, R14 to R23, R15 to R24, R11 to R3, R12 to R4, R132 to R45, R133 to R46, R138 to R51, R139 to R52, R23 to R7, R25 to R8, R27 to R9, U2 to U1, U5 to U4, U1 to U6
Connections:
- net /Load Switch 2/VOUT renamed /5V_PYLD_IN
- net /RB_Vcc renamed /RB_VCC
- net 5V_PL renamed /5V_PYLD
- D1 pad 1: GND -> Net-(D1-K)
- D1 pad 2: Net-(D1-DOUT) -> Net-(D1-A)
- D2 pad 1: GND -> Net-(D2-K)
- D2 pad 2: /DOUT -> Net-(D2-A)
- P1 pad 14: /LED_PWR -> unconnected-(P1-Pin_14-Pad14)
- P1 pad 15: /DIN_LED -> /LED_PWR
- P1 pad 16: /DOUT_LED -> unconnected-(P1-Pin_16-Pad16)
- P1 pad 19: GND -> unconnected-(P1-Pin_19-Pad19)
- P1 pad 20: GND -> unconnected-(P1-Pin_20-Pad20)
- P1 pad 22: /RB_OnOff_IN -> /RB_EN
- P1 pad 30: unconnected-(P1-Pin_30-Pad30) -> /IMU_EN
- P1 pad 33: /TEMP_C -> unconnected-(P1-Pin_33-Pad33)
- P1 pad 35: unconnected-(P1-Pin_35-Pad35) -> GND
- P1 pad 36: unconnected-(P1-Pin_36-Pad36) -> GND
- P1 pad 41: /RX_4 -> unconnected-(P1-Pin_41-Pad41)
- P1 pad 42: /TX_4 -> unconnected-(P1-Pin_42-Pad42)
- Q2 pad 1: Net-(Q2-B) -> GND
- Q2 pad 2: GND -> Net-(Q2B-B2)
- Q2 pad 3: Net-(D4-K) -> Net-(D1-K)
- Q3 pad 1: Net-(Q3-B) -> GND
- Q3 pad 2: GND -> Net-(Q3B-B2)
- R25 pad 1: LED_VCC -> /IMU_EN
- R25 pad 2: Net-(D3-A) -> Net-(D1-A)
- R29 pad 1: Net-(Q1-B) -> Net-(Q2A-B1)
- R29 pad 2: /RED_LED -> /LED_PWR
- RN1 pad 3: /PICO_TxD -> GND
- RN2 pad 5: Net-(U3-B4) -> Net-(U3-B3)
- RN2 pad 6: Net-(U3-B5) -> Net-(U3-B4)
- RN2 pad 7: Net-(U3-B6) -> Net-(U3-B5)
- RN2 pad 8: Net-(U3-B7) -> Net-(U3-B6)
- RN4 pad 6: /TX_4 -> GND
- RN5 pad 1: Net-(U5-A7) -> Net-(U4-A6)
- RN5 pad 2: Net-(U5-A6) -> Net-(U4-A5)
- RN5 pad 3: Net-(U5-A5) -> Net-(U4-A4)
- RN5 pad 4: Net-(U5-A4) -> Net-(U4-A3)
- U3 pad 16: /RX_4 -> Net-(U3-B3)
- U4 pad 4: /PICO_RxD -> Net-(U4-A3)
- U4 pad 5: Net-(U5-A4) -> Net-(U4-A4)
- U4 pad 6: Net-(U5-A5) -> Net-(U4-A5)
- U4 pad 7: Net-(U5-A6) -> Net-(U4-A6)
- U4 pad 8: Net-(U5-A7) -> Net-(U4-A7)
- U6 pad 3: /SCL_IMU -> /SCL
- U6 pad 4: /SDA_IMU -> /SDA
Routing:
- net /5V_PYLD_IN: track 0.00 -> 143.2 mm, vias 0 -> 5
- net /SERVO_PWR_CTRL: track 0.00 -> 134.6 mm, vias 0 -> 3
- net /PYLD_RESET: track 0.00 -> 133.2 mm, vias 0 -> 2
- net /IMU_EN: track 0.00 -> 127.1 mm, vias 0 -> 7
- net /PYLD_PWR_EN: track 0.00 -> 120.9 mm, vias 0 -> 3
- net /TEMP_A: track 0.00 -> 109.0 mm, vias 0 -> 1
- net /PYLD_TXD: track 0.00 -> 91.7 mm, vias 0 -> 2
- net /PYLD_RXD: track 0.00 -> 91.1 mm, vias 0 -> 2
- net /RB_PWR_EN: track 0.00 -> 69.5 mm
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- added copper zone on In2.Cu, net +3.3V
- added copper zone on F.Cu, net +5V
- added copper zone on In2.Cu, net +5V
- added copper zone on F.Cu, net /5V_PYLD
- added copper zone on In2.Cu, net /5V_PYLD
- added copper zone on F.Cu, net /5V_PYLD_IN
- added copper zone on F.Cu, net /RB_VCC
- removed copper zone on In3.Cu, net +3.3V
- removed copper zone on In1.Cu, net +5V
- removed copper zone on B.Cu, net GND
- removed copper zone on In2.Cu, net GND
- removed copper zone on In4.Cu, net GND
- removed copper zone on B.Cu, net unconnected-(P1-Pin_74-Pad74)
Other:
- outline, holes or cut-outs redrawn
- copper layers 6 -> 4
- board text added: "1. Class 3 for PCBway, class 2 for US vendor. 2. Nelco N7000-2HT preferred for flight, but PCBway SH260 is acceptable."
- board text added: "1. Class 3 preferred"
- board text added: "1. IPC-6012E Class 2 2. Matte Green soldermask, White silkscreen. 3. Fabricate on SH260 4. 1oz outer, 1oz inner copper. 5. Bevel edge connector 30 degrees minimum. 6. Board target thickness shall be 0.062{dblquote} 7. Immersion gold plating on finger thickness shall be 2U{dblquote}"
- board text added: "1. J-STD-001G Class 2 2. BOM provided with submitted files shall be the controlling document for component information. 3. Do not apply solder to pads of DNP components 4. Assemble with leaded solder."
- board text added: "1. Stake components specified in BOM with 3M 2216 2. Conformal Coat with Arathane 5750: Ensure coating does not prevent electrical contact with connectors and mounting holes."
- board text added: "3550.00 mils x 3982.07 mils"
- board text added: "4"
- board text added: "62 mils"
- board text added: "7.87 mils"
- board text added: "8.00 mils / 8.00 mils"
- board text added: "ASSEMBLY COMMENTS:"
- board text added: "ASSEMBLY NOTES:"
- board text added: "CH 6/23"
- board text added: "FAB COMMENTS:"
- board text added: "FAB NOTES:"
- board text added: "FORAS PROMINEO PAYLOAD INTERFACE BOARD revB"
- board text added: "VENDOR ASSEMBLY NOTES:"
- board text added: "Yes, bevelled 30deg minimum."
- board text removed: "0.2000 mm"
- board text removed: "0.2032 mm / 0.1524 mm"
- board text removed: "1.6000 mm"
- board text removed: "6"
- board text removed: "90.1700 mm x 101.1445 mm"
- board text removed: "Add 45deg chamfer to the gold fingers Fabricate with leaded solder"
- board text removed: "HILLIS"
- board text removed: "NOTES"
- board text removed: "Yes"
