File: hardware/revB/payload-interface-board.kicad_sch (KiCad schematic)
At the start: 27 parts, among them J1 T1M-10-F-SV-L, P1 Card Edge for HSEC8-160-01-S-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, Q1 MMBT4401WT1G, Q2 IRF7404TRPBF, Q3 MMBT4401WT1G, U1 LTC4307, U2 SN74LVCH245APWR, U3 SN74LVCH245APWR, U4 RockBlock_9603

Commit message: working
Parts:
- removed C1: 0.01uF, Capacitor_SMD:C_0603_1608Metric, symbol Device:C
- removed Q2: IRF7404TRPBF, Package_SO:SO-8_3.9x4.9mm_P1.27mm, symbol SLI-Backplane-Blank-Card-KiCad:IRF7404TRPBF
- removed U1: LTC4307, Package_SO:MSOP-8_3x3mm_P0.65mm, symbol mainboard_SLI:LTC4307
- removed U4: RockBlock_9603, payload-interface-board:RockBlock_9603, symbol FP-Interface-Card:RockBlock_9603
- added C1 (x2): 1uF, Capacitor_SMD:C_0603_1608Metric, symbol Device:C
- added C1, C10, C2, C7, C8, C9: 0.1uF, Capacitor_SMD:C_0402_1005Metric, symbol Device:C
- added C3: 10uF, Capacitor_SMD:C_0805_2012Metric, symbol Device:C
- added C4: 0.01uF, Capacitor_SMD:C_0402_1005Metric, symbol Device:C
- added D208 (x2): SK6805-EC3210R, payload-interface-board:SK6812-EC3210F-RA, symbol FP-Interface-Card:SK6812-EC321F_4
- added D3: RED, SLI-Backplane-Blank-Card-KiCad:APA2107x, symbol Device:D
- added D4: YELLOW, SLI-Backplane-Blank-Card-KiCad:APA2107x, symbol Device:D
- added D5: GREEN, SLI-Backplane-Blank-Card-KiCad:APA2107x, symbol Device:D
- added D6: ORANGE, SLI-Backplane-Blank-Card-KiCad:APA2107x, symbol Device:D
- added H1, H2, H3, H4: SLI-Backplane-Blank-Card-KiCad:125mil_hole, SLI-Backplane-Blank-Card-KiCad:125mil_hole, symbol Mechanical:MountingHole_Pad
- added J2: T1M-6-F-SV-L, payload-interface-board:SAMTEC_T1M-06-F-SV-L, symbol Connector_Generic:Conn_01x06
- added J3: T1M-10-F-SV-L, payload-interface-board:SAMTEC_T1M-10-F-SV-L, symbol Connector_Generic:Conn_02x05_Odd_Even
- added J4: Conn_01x02, Connector_PinHeader_2.54mm:PinHeader_1x02_P2.54mm_Vertical_SMD_Pin1Left, symbol Connector_Generic:Conn_01x02
- added J4 (x3): T1M-02-F-SV-L, SierraLobo:SAMTEC_T1M-02-F-SV-L-P, symbol Connector_Generic:Conn_01x02
- added JP1: Wire Cut Jumper, Resistor_SMD:R_0603_1608Metric, symbol Jumper:Jumper_2_Bridged
- added Q2, Q4: BC847BM3T5G, Package_TO_SOT_SMD:SOT-723, symbol Device:Q_NPN_BEC
- added Q39: MMDT3946, Package_TO_SOT_SMD:SOT-363_SC-70-6, symbol Transistor_BJT:MMDT3946
- added R10: 988k, Resistor_SMD:R_0603_1608Metric, symbol Device:R_US
- added R11, R12: 4.7k, Resistor_SMD:R_0603_1608Metric, symbol Device:R_US
- added R13, R16: 10k, Resistor_SMD:R_0402_1005Metric, symbol Device:R_US
- added R14: 105k, Resistor_SMD:R_0603_1608Metric, symbol Device:R_US
- added R15: 576k, Resistor_SMD:R_0603_1608Metric, symbol Device:R_US
- added R17, R20, R21, R22: 100k, Resistor_SMD:R_0402_1005Metric, symbol Device:R_US
- added R23, R25, R27, R29: 0, Resistor_SMD:R_0603_1608Metric, symbol Device:R_US
- added R24: 1k, Resistor_SMD:R_0402_1005Metric, symbol Device:R_US
- added R7, R8: 1.5k, Resistor_SMD:R_0402_1005Metric, symbol Device:R_US
- added RN2 (x2): 10k, Resistor_SMD:R_Array_Convex_4x0402, symbol SierraLobo:R_Network04_US
- added U1: imu-stamp-revA, payload-interface-board:imu-stamp-revA-SMD, symbol FP-Interface-Card:imu-stamp-revA
- added U15: NCP164ASN330T1G, Package_TO_SOT_SMD:TSOT-23-5, symbol SierraLobo:NCP164ASN330T1G
- added U2: LTC4307, Package_SO:MSOP-8_3x3mm_P0.65mm, symbol mainboard_SLI:LTC4307
- added U4: RockBlock_9603, SierraLobo:RockBlock_9603, symbol SierraLobo:RockBlock_9603
- C5, C6: renamed from C32; footprint Capacitor_SMD:C_0603_1608Metric -> Capacitor_SMD:C_0402_1005Metric; Manufacturer (none) -> TDK; Mfr. Part No (none) -> CGA2B3X7R1H104K050BE
- Q1, Q3: value MMBT4401WT1G -> BC847BM3T5G; footprint Package_TO_SOT_SMD:SOT-323_SC-70 -> Package_TO_SOT_SMD:SOT-723
- R1: value 4.7k -> 1k; footprint Resistor_SMD:R_0603_1608Metric -> Resistor_SMD:R_0402_1005Metric
- R18: renamed from R7; footprint Resistor_SMD:R_0603_1608Metric -> Resistor_SMD:R_0402_1005Metric
- R19: renamed from R8; footprint Resistor_SMD:R_0603_1608Metric -> Resistor_SMD:R_0402_1005Metric
- R2: value 4.7k -> 1.5k; footprint Resistor_SMD:R_0603_1608Metric -> Resistor_SMD:R_0402_1005Metric
- R26: renamed from R10; footprint Resistor_SMD:R_0603_1608Metric -> Resistor_SMD:R_0402_1005Metric
- R28: renamed from R11; footprint Resistor_SMD:R_0603_1608Metric -> Resistor_SMD:R_0402_1005Metric
- R3, R5: value 10Meg -> 1.5k; footprint Resistor_SMD:R_0603_1608Metric -> Resistor_SMD:R_0402_1005Metric
- R4, R9: value 1Meg -> 1.5k; footprint Resistor_SMD:R_0603_1608Metric -> Resistor_SMD:R_0402_1005Metric
- R6: value 100 -> 1.5k; footprint Resistor_SMD:R_0603_1608Metric -> Resistor_SMD:R_0402_1005Metric
- renumbered RN2 to RN3, RN3 to RN4, RN4 to RN6, U2 to U3, U3 to U5
Connections:
- net BP_LED_PWR is gone; now on net DIN_LED: P1.15 (Pin_15)
- net H1-36 is gone; now on net 5V_PL: P1.78 (Pin_78)
- net H1-37 is gone; now on net GND: P1.81 (Pin_81)
- net H1-38 is gone; now on net GND: P1.82 (Pin_82)
- net +3.3V: now also C3.1, C4.1, R11.1, R12.1, U1.1 (VCC), U2.1 (EN), U2.8 (VCC); no longer P1.58 (Pin_58), R1.1, R2.1
- net DIN_LED: no longer P1.14 (Pin_14)
- net GND: now also C1.2, C1.2, C1.2, C10.1, C2.2, C3.2, C4.2, C7.1, C8.1, C9.1, D208.1 (VSS), D208.1 (VSS), J3.10 (Pin_10), J3.8 (Pin_8), J3.9 (Pin_9), Q2.2 (E), Q39.1 (E1), Q4.2 (E), R15.2, R16.1, R21.1, R24.2, RN2.1, RN2.2, RN2.3, RN2.4, RN2.5, RN2.6, RN2.7, RN2.8, U1.10 (GND), U1.2 (GND), U1.9 (GND), U15.2 (GND), U2.4 (GND)
- net PYLD_RXD: now also J3.6 (Pin_6)
- net PYLD_TXD: now also J3.5 (Pin_5)
- net RB_RxD: now also R23.2, R29.2; no longer U5.3 (A2)
- net RB_TxD: now also R25.2, R27.2; no longer RN1.2
- net SCL_IMU: now also U1.3 (SCL)
- net SDA_IMU: now also U1.4 (SDA)
- net RED_LED: now reaches R6.2
- net at Q3.1 (B): now also R8.1; no longer R9.2
- net at U5.5 (A4): now also RN2.4
- net at U5.6 (A5): now also RN2.3
- net at U5.7 (A6): now also RN2.2
- net at U5.8 (A7): now also RN2.1
- net at U5.9 (A8): now also R24.1
- net at Q1.1 (B): now also R6.1; no longer R4.2
- net at U3.11 (B8): now also R16.2
- net at U3.12 (B7): now also RN2.8
- net at U3.13 (B6): now also RN2.7
- net at U3.14 (B5): now also RN2.6
- net at U3.15 (B4): now also RN2.5
- net +X_SOLAR_PWR: no longer names the net of P1.8 (Pin_8)
- net +X_SOLAR_RTN: no longer names the net of P1.6 (Pin_6)
- net +X_SOLAR_TLE: no longer names the net of P1.4 (Pin_4)
- net +Y_SOLAR_PWR: no longer names the net of P1.117 (Pin_117)
- net +Y_SOLAR_RTN: no longer names the net of P1.115 (Pin_115)
- net +Y_SOLAR_TLE: no longer names the net of P1.113 (Pin_113)
- net -X_SOLAR_PWR: no longer names the net of P1.118 (Pin_118)
- net -X_SOLAR_RTN: no longer names the net of P1.116 (Pin_116)
- net -X_SOLAR_TLE: no longer names the net of P1.114 (Pin_114)
- net -Z_SOLAR_PWR: no longer names the net of P1.7 (Pin_7)
- net -Z_SOLAR_RTN: no longer names the net of P1.5 (Pin_5)
- net -Z_SOLAR_TLE: no longer names the net of P1.3 (Pin_3)
- net 5V_RF renamed LED_VCC
- net LED_VCC: now also R2.1, R4.1, C1.1, C2.1, D208.4 (VDD), D208.4 (VDD); no longer P1.73 (Pin_73), P1.74 (Pin_74)
- net 5V_USB: no longer names the net of P1.70 (Pin_70)
- net BATT_NTC: no longer names the net of P1.11 (Pin_11)
- net H1-10: no longer names the net of P1.26 (Pin_26)
- net H1-11 renamed PYLD_PWR_EN
- net H1-12: no longer names the net of P1.30 (Pin_30)
- net H1-13 renamed TEMP_C
- net H1-14: no longer names the net of P1.34 (Pin_34)
- net H1-17 renamed RX_4
- net H1-18 renamed TX_4
- net H1-19 renamed RX_2
- net H1-20 renamed TX_2
- net H1-21: no longer names the net of P1.49 (Pin_49)
- net H1-22: no longer names the net of P1.50 (Pin_50)
- net H1-23: no longer names the net of P1.53 (Pin_53)
- net H1-24: no longer names the net of P1.54 (Pin_54)
- net H1-25: no longer names the net of P1.57 (Pin_57)
- net H1-27: no longer names the net of P1.61 (Pin_61)
- net H1-28: no longer names the net of P1.62 (Pin_62)
- net H1-30: no longer names the net of P1.66 (Pin_66)
- net H1-31: no longer names the net of P1.69 (Pin_69)
- net H1-35 renamed 5V_PL
- net H1-39 renamed RX_3
- net H1-40 renamed TX_3
- net H1-42: no longer names the net of P1.90 (Pin_90)
- net H1-44: no longer names the net of P1.94 (Pin_94)
- net H1-48: no longer names the net of P1.102 (Pin_102)
- net H1-5 renamed SERVO_PWR_CTRL
- net SERVO_PWR_CTRL: now also J3.7 (Pin_7)
- net H1-51: no longer names the net of P1.109 (Pin_109)
- net H1-52: no longer names the net of P1.110 (Pin_110)
- net H1-6 renamed PYLD_RESET
- net PYLD_RESET: now also J3.4 (Pin_4)
- net H1-7: no longer names the net of R9.1
- net H1-7: now also Q4.1 (B); no longer P1.21 (Pin_21)
- net H1-8 renamed RB_OnOff_IN
- net RB_OnOff_IN: no longer R4.1
- net H1-9: no longer names the net of P1.25 (Pin_25)
- net H2-10 renamed TEMP_B
- net H2-11: no longer names the net of P1.31 (Pin_31)
- net H2-12: no longer names the net of P1.32 (Pin_32)
- net H2-13: no longer names the net of P1.35 (Pin_35)
- net H2-14: no longer names the net of P1.36 (Pin_36)
- net H2-15: no longer names the net of P1.39 (Pin_39)
- net H2-16: no longer names the net of P1.40 (Pin_40)
- net H2-17: no longer names the net of P1.43 (Pin_43)
- net H2-18: no longer names the net of P1.44 (Pin_44)
- net H2-19: no longer names the net of P1.47 (Pin_47)
- net H2-2: no longer names the net of P1.12 (Pin_12)
- net H2-20: no longer names the net of P1.48 (Pin_48)
- net H2-21: no longer names the net of P1.51 (Pin_51)
- net H2-22: no longer names the net of P1.52 (Pin_52)
- net H2-23: no longer names the net of P1.55 (Pin_55)
- net H2-24: no longer names the net of P1.56 (Pin_56)
- net H2-33: no longer names the net of P1.75 (Pin_75)
- net H2-34: no longer names the net of P1.76 (Pin_76)
- net H2-35: no longer names the net of P1.79 (Pin_79)
- net H2-36: no longer names the net of P1.80 (Pin_80)
- net H2-37: no longer names the net of P1.83 (Pin_83)
- net H2-38: no longer names the net of P1.84 (Pin_84)
- net H2-39: no longer names the net of P1.87 (Pin_87)
- net H2-40: no longer names the net of P1.88 (Pin_88)
- net H2-41: no longer names the net of P1.91 (Pin_91)
- net H2-42: no longer names the net of P1.92 (Pin_92)
- net H2-43: no longer names the net of P1.95 (Pin_95)
- net H2-44: no longer names the net of P1.96 (Pin_96)
- net H2-7: no longer names the net of P1.23 (Pin_23)
- net H2-8: no longer names the net of P1.24 (Pin_24)
- net H2-9 renamed TEMP_A
- net RBF: no longer names the net of P1.37 (Pin_37)
- net RBF_RET: no longer names the net of P1.38 (Pin_38)
- net RB_5V_IN renamed RB_Vcc
- net RB_CTS: no longer names the net of J1.2 (Pin_2)
- net RB_Li-iON: no longer names the net of J1.9 (Pin_9)
- net RB_NetAv: no longer names the net of J1.4 (Pin_4)
- removed net RB_OnOff: J1.7 (Pin_7), Q1.3 (C), R3.2
- net RB_RI: no longer names the net of J1.5 (Pin_5)
- net RB_RTS: no longer names the net of J1.3 (Pin_3)
- net SCL_PIB renamed DIN
- net SDA_PIB: no longer names the net of R2.2
- net SDA_PIB: now also D3.2 (A)
- net SELF_TEST: no longer names the net of P1.101 (Pin_101)
- net SEP1: no longer names the net of P1.1 (Pin_1)
- net SEP1_RET: no longer names the net of P1.9 (Pin_9)
- net SEP2: no longer names the net of P1.2 (Pin_2)
- net SEP2_RET: no longer names the net of P1.10 (Pin_10)
- net SEP3: no longer names the net of P1.119 (Pin_119)
- net SEP3_RET: no longer names the net of P1.111 (Pin_111)
- net SEP4: no longer names the net of P1.120 (Pin_120)
- net SEP4_RET: no longer names the net of P1.112 (Pin_112)
- removed net VBATT+: P1.100 (Pin_100), P1.97 (Pin_97), P1.98 (Pin_98), P1.99 (Pin_99)
- removed net VBATT-: P1.105 (Pin_105), P1.106 (Pin_106), P1.107 (Pin_107), P1.108 (Pin_108)
- net ~{BP_LED_EN}: no longer names the net of P1.13 (Pin_13)
- net ~{RESET}: no longer names the net of P1.65 (Pin_65)
- new net: D5.1 (K), Q3.3 (C)
- new net: Q39.3 (C2), R22.1
- new net: Q39.2 (B1), R22.2
- new net: C10.2, H4.1
- new net: C7.2, H1.1
- new net: C1.1, J4.1 (Pin_1), U15.5 (VOUT)
- new net: J4.2 (Pin_2), JP1.1 (A)
- new net: Q39.5 (B2), R20.2
- new net: D208.2 (DOUT), D208.3 (DIN)
- new net: D208.3 (DIN), R1.1
- new net: D4.1 (K), Q2.3 (C)
- new net: D4.2 (A), R3.2
- new net: Q2.1 (B), R7.1
- new net: R13.2, U1.5 (EN)
- new net: R10.1, U1.6 (XOR_REF)
- new net: R10.2, R14.1, U1.7 (XORL2)
- new net: R14.2, R15.1, U1.8 (XORL1)
- new net: D5.2 (A), R4.2
- new net: D3.1 (K), Q1.3 (C)
- new net: C8.2, H2.1
- new net: D6.2 (A), R5.2
- new net: C9.2, H3.1
- new net: D6.1 (K), Q4.3 (C)
- new net 3V3D: JP1.2 (B)
- new net DOUT: D208.2 (DOUT)
- new net GRN_LED: R8.2
- new net I2C-Protection-1/SCL_O: U2.3 (SCLIN)
- new net I2C-Protection-1/SDA_O: U2.6 (SDAIN)
- new net IMU_EN: R13.1
- new net LED_PWR: P1.14 (Pin_14)
- new net Load Switch 2/VOUT: J3.1 (Pin_1), J3.2 (Pin_2), J3.3 (Pin_3)
- new net ORG_LED: R9.2
- new net OnOff: J1.7 (Pin_7), Q39.6 (C1), R17.2
- new net RB_EN: R20.1, R21.2
- new net RB_PWR_EN: P1.21 (Pin_21)
- new net RB_RxD_in: R23.1, R25.1, RN1.2
- new net RB_TxD_in: R27.1, R29.1, U5.3 (A2)
- new net SCL: R11.2, U2.2 (SCLOUT)
- new net SDA: R12.2, U2.7 (SDAOUT)
- new net VBUS: C1.1, U15.1 (VIN), U15.3 (EN)
- new net VIO: Q39.4 (E2), R17.1
- new net X+: J2.2 (Pin_2)
- new net X-: J2.1 (Pin_1)
- new net Y+: J2.4 (Pin_4)
- new net Y-: J2.3 (Pin_3)
- new net YEL_LED: R7.2
- new net Z+: J2.6 (Pin_6)
- new net Z-: J2.5 (Pin_5)
- no-connect marks 16 -> 92
Other:
- removed sheet Backplane Card Interface
- removed sheet IMU
- removed sheet MT Drivers
- removed sheet Payload Interface
- removed sheet Pico
- added sheet Load Switch 1 (load_sw.kicad_sch)
- added sheet Load Switch 2 (load_sw.kicad_sch)
- added sheet MTQ Control (mtq_control.kicad_sch)
- added sheet Temp Sensors (temp_sensors.kicad_sch)
- sheet I2C-Protection-1 ports: added SCL_I, SCL_O, SDA_I, SDA_O; removed SCL_IN, SCL_PROT, SDA_IN, SDA_PROT
- sheet I2C-Protection-2 ports: added SCL_I, SCL_O, SDA_I, SDA_O; removed SCL_IN, SCL_PROT, SDA_IN, SDA_PROT
- note added: "1. Monitor payload current 2. Monitor Rockblock current"
- note added: "Chassis"
- note added: "DIO"
- note added: "I2C BUFFER"
- note added: "Input Load Switch"
- note added: "Input Power Decoupling"
- note added: "LEDs"
- note added: "LOAD SWITCH"
- note added: "Mounting Holes"
- note added: "OnOff high = Rockblock ON"
- note added: "PAYLOAD INTERFACE"
- note added: "REDUNDANT IMU"
- note added: "ROCKBLOCK INTERFACE"
- note added: "Serial In"
- note added: "Serial Out"
- note added: "To MTs"
- note added: "Tx = IN"
- note added: "USB POWER"
- note added: "VERIFY CONNNECTOR"
- note added: "double check"
- note added: "gyro addr: 0x6A, 0x6D accel addr: 0x4E, 0x49 mag addr: 0x32, 0x35"
- note added: "xor ch1 = 0x5 xor ch2 = 0x6"
- note removed: "Card Edge to PIB Signals"
- note removed: "DNP!!"
- note removed: "I2C Buffer"
- note removed: "IN"
- note removed: "OUT"
- note removed: "RB has a low power sleep, but this is to disconnect in case of failure."
- note removed: "RX_MCU_2"
- note removed: "RX_MCU_3"
- note removed: "RX_MCU_4"
- note removed: "Serial IO Buffers"
- note removed: "TO FORAS PROMINEO PAYLOAD"
- note removed: "TO ROCKBLOCK 9603"
- note removed: "TX_MCU_2"
- note removed: "TX_MCU_3"
- note removed: "TX_MCU_4"
- company: Sierra Lobo INC. -> (none)
- moved on the sheet: C5, C6, P1, R18, R19, R26, R28, RN1, RN3, RN4, RN6, U3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

Commit message: revB initial commit
Parts:
- removed C1 (x2): 1uF, Capacitor_SMD:C_0603_1608Metric, symbol Device:C
- removed C1, C2: 0.1uF, Capacitor_SMD:C_0402_1005Metric, symbol Device:C
- removed D208 (x2): SK6805-EC3210R, payload-interface-board:SK6812-EC3210F-RA, symbol FP-Interface-Card:SK6812-EC321F_4
- removed J2: T1M-6-F-SV-L, payload-interface-board:SAMTEC_T1M-06-F-SV-L, symbol Connector_Generic:Conn_01x06
- removed J4: Conn_01x02, Connector_PinHeader_2.54mm:PinHeader_1x02_P2.54mm_Vertical_SMD_Pin1Left, symbol Connector_Generic:Conn_01x02
- removed J4 (x3): T1M-02-F-SV-L, SierraLobo:SAMTEC_T1M-02-F-SV-L-P, symbol Connector_Generic:Conn_01x02
- removed JP1: Wire Cut Jumper, Resistor_SMD:R_0603_1608Metric, symbol Jumper:Jumper_2_Bridged
- removed Q1, Q2, Q3, Q4: BC847BM3T5G, Package_TO_SOT_SMD:SOT-723, symbol Device:Q_NPN_BEC
- removed R1: 1k, Resistor_SMD:R_0402_1005Metric, symbol Device:R_US
- removed R3, R4, R5, R7, R8, R9: 1.5k, Resistor_SMD:R_0402_1005Metric, symbol Device:R_US
- removed U15: NCP164ASN330T1G, Package_TO_SOT_SMD:TSOT-23-5, symbol SierraLobo:NCP164ASN330T1G
- added C100 (x2): 0.1uF, Capacitor_SMD:C_0603_1608Metric, symbol Device:C
- added C99 (x2): 1uF, Capacitor_SMD:C_0603_1608Metric, symbol Device:C
- added Q2, Q3: MMDT2222A, Package_TO_SOT_SMD:SOT-363_SC-70-6, symbol SierraLobo:MMDT2222
- added R11, R15: 10k, Resistor_SMD:R_0603_1608Metric, symbol Device:R_US
- added R26, R27, R28: 1.5k, Resistor_SMD:R_0402_1005Metric, symbol Device:R_US
- added R30, R31, R32: 10k, Resistor_SMD:R_0402_1005Metric, symbol Device:R_US
- added R36 (x2): 220, Resistor_SMD:R_0603_1608Metric, symbol Device:R_US
- added TP10, TP11, TP12, TP13, TP14, TP16, TP17, TP18, TP19, TP2, TP20, TP22, TP3, TP4, TP5, TP6, TP9: ${NET_NAME(1)}, TestPoint:TestPoint_Keystone_5000-5004_Miniature, symbol Connector:TestPoint_Small
- added TP15, TP21, TP7: ${NET_NAME(1)}, SierraLobo:Keystone_5027, symbol Connector:TestPoint_Small
- added U24 (x2): MCP9700AT-E/LT, Package_TO_SOT_SMD:SOT-353_SC-70-5, symbol Sensor_Temperature:MCP9700Ax-ELT
- C1: renamed from C4; footprint Capacitor_SMD:C_0402_1005Metric -> Capacitor_SMD:C_0603_1608Metric
- C10: renamed from C8; footprint Capacitor_SMD:C_0402_1005Metric -> Capacitor_SMD:C_0603_1608Metric
- C11: renamed from C9; footprint Capacitor_SMD:C_0402_1005Metric -> Capacitor_SMD:C_0603_1608Metric
- C12: renamed from C10; footprint Capacitor_SMD:C_0402_1005Metric -> Capacitor_SMD:C_0603_1608Metric
- C2: renamed from C5; footprint Capacitor_SMD:C_0402_1005Metric -> Capacitor_SMD:C_0603_1608Metric
- C3: renamed from C6; footprint Capacitor_SMD:C_0402_1005Metric -> Capacitor_SMD:C_0603_1608Metric
- C9: renamed from C7; footprint Capacitor_SMD:C_0402_1005Metric -> Capacitor_SMD:C_0603_1608Metric
- D1: renamed from D3; footprint SLI-Backplane-Blank-Card-KiCad:APA2107x -> SierraLobo:APA2107x
- D2: renamed from D4; footprint SLI-Backplane-Blank-Card-KiCad:APA2107x -> SierraLobo:APA2107x
- D3: renamed from D6; footprint SLI-Backplane-Blank-Card-KiCad:APA2107x -> SierraLobo:APA2107x
- D4: renamed from D5; footprint SLI-Backplane-Blank-Card-KiCad:APA2107x -> SierraLobo:APA2107x
- H1, H2, H3, H4: footprint SLI-Backplane-Blank-Card-KiCad:125mil_hole -> SierraLobo:125mil_hole
- R1: renamed from R17; footprint Resistor_SMD:R_0402_1005Metric -> Resistor_SMD:R_0603_1608Metric
- R12: renamed from R16; footprint Resistor_SMD:R_0402_1005Metric -> Resistor_SMD:R_0603_1608Metric
- R13: renamed from R18; footprint Resistor_SMD:R_0402_1005Metric -> Resistor_SMD:R_0603_1608Metric
- R14: renamed from R19; footprint Resistor_SMD:R_0402_1005Metric -> Resistor_SMD:R_0603_1608Metric
- R16: renamed from R24; value 1k -> 10k; footprint Resistor_SMD:R_0402_1005Metric -> Resistor_SMD:R_0603_1608Metric
- R17: renamed from R26; footprint Resistor_SMD:R_0402_1005Metric -> Resistor_SMD:R_0603_1608Metric
- R18: renamed from R28; footprint Resistor_SMD:R_0402_1005Metric -> Resistor_SMD:R_0603_1608Metric
- R2: renamed from R20; footprint Resistor_SMD:R_0402_1005Metric -> Resistor_SMD:R_0603_1608Metric
- R22: renamed from R13; footprint Resistor_SMD:R_0402_1005Metric -> Resistor_SMD:R_0603_1608Metric
- R29: renamed from R6; value 1.5k -> 10k
- R5: renamed from R21; footprint Resistor_SMD:R_0402_1005Metric -> Resistor_SMD:R_0603_1608Metric
- R6: renamed from R22; footprint Resistor_SMD:R_0402_1005Metric -> Resistor_SMD:R_0603_1608Metric
- RN1: footprint payload-interface-board:RAVF164D -> Resistor_SMD:R_Array_Convex_4x0402
- RN2: Manufacturer Stackpole Electronics -> (none); Mfr. Part No RAVF164DJT10K0 -> (none)
- RN3, RN4, RN6: footprint payload-interface-board:RAVF164D -> Resistor_SMD:R_Array_Convex_4x0402; Manufacturer (none) -> Panasonic; Mfr. Part No (none) -> EXB-28V102JX
- renumbered C3 to C6, J3 to J2, R29 to R10, R10 to R20, R14 to R23, R15 to R24, R2 to R25, R11 to R3, R12 to R4, R23 to R7, R25 to R8, R27 to R9, U2 to U1, U4 to U2, U5 to U4, U1 to U6
Connections:
- net DIN_LED is gone; now on net LED_PWR: P1.15 (Pin_15)
- net LED_VCC is gone; now on net IMU_EN: R25.1
- net PICO_RxD is gone; now on an unnamed net: U4.4 (A3)
- net PICO_TxD is gone; now on net GND: RN1.3
- net RB_OnOff_IN is gone; now on net RB_EN: P1.22 (Pin_22)
- net RED_LED is gone; now on net LED_PWR: R29.2
- net SCL_IMU is gone; now on net SCL: U6.3 (SCL)
- net SDA_IMU is gone; now on net SDA: U6.4 (SDA)
- net +3.3V: now also R26.1, R36.1, R36.1, TP22.1
- net GND: now also P1.35 (Pin_35), P1.36 (Pin_36), RN4.6, C100.2, C100.2, C99.2, C99.2, Q2.1 (E2), Q2.4 (E1), Q3.1 (E2), Q3.4 (E1), R11.1, R15.2, TP15.1, TP21.1, TP7.1, U24.2 (GND), U24.2 (GND); no longer P1.19 (Pin_19), P1.20 (Pin_20)
- net IMU_EN: now also P1.30 (Pin_30), TP20.1
- net LED_PWR: now also R30.2, R31.2, R32.2; no longer P1.14 (Pin_14)
- net PYLD_PWR_EN: now also TP10.1
- net PYLD_RESET: now also TP11.1
- net PYLD_RXD: now also TP13.1
- net PYLD_TXD: now also TP12.1
- net RB_EN: now also TP4.1
- net RB_PWR_EN: now also TP3.1
- net RB_RxD: now also TP5.1
- net RB_TxD: now also TP6.1
- net SCL: now also TP18.1
- net SDA: now also TP19.1
- net SERVO_PWR_CTRL: now also TP14.1
- net TEMP_A: now also C100.1, TP16.1, U24.3 (V_{OUT})
- net TEMP_B: now also C100.1, TP17.1, U24.3 (V_{OUT})
- net at R29.1: now also Q2.5 (B1)
- net at D4.1 (K): now also Q3.6 (C2)
- net at D2.1 (K): now also Q2.6 (C2)
- net at D2.2 (A): now also R26.2
- net at D4.2 (A): now also R28.2
- net at D1.1 (K): now also Q2.3 (C1)
- net at RN2.4: no longer U4.5 (A4)
- net at RN2.3: now also U4.5 (A4); no longer U4.6 (A5)
- net at RN2.2: now also U4.6 (A5); no longer U4.7 (A6)
- net at RN2.1: now also U4.7 (A6); no longer U4.8 (A7)
- net at D3.2 (A): now also R27.2
- net at RN2.5: now also U3.16 (B3); no longer U3.15 (B4)
- net at RN2.6: now also U3.15 (B4); no longer U3.14 (B5)
- net at RN2.7: now also U3.14 (B5); no longer U3.13 (B6)
- net at U3.12 (B7): now also R11.2; no longer RN2.8
- net at D3.1 (K): now also Q3.3 (C1)
- net 5V_PL renamed 5V_PYLD
- net DOUT_LED: no longer names the net of P1.16 (Pin_16)
- net Load Switch 2/VOUT renamed 5V_PYLD_IN
- net 5V_PYLD_IN: now also R28.1, TP9.1
- net RB_Vcc renamed RB_VCC
- net RB_VCC: now also R27.1, TP2.1
- net RX_4: no longer names the net of P1.41 (Pin_41)
- net RX_4: no longer U3.16 (B3)
- net TEMP_C: no longer names the net of P1.33 (Pin_33)
- net TX_4: no longer names the net of P1.42 (Pin_42)
- net TX_4: no longer RN4.6
- new net: Q3.5 (B1), R31.1
- new net: Q3.2 (B2), R32.1
- new net: Q2.2 (B2), R30.1
- new net: C99.1, R36.2, U24.4 (V_{DD}) (x2)
- new net: R15.1, U4.8 (A7)
- new net: RN2.8, U3.13 (B6)
- no-connect marks 92 -> 94
Other:
- removed sheet I2C-Protection-2
- removed sheet MTQ Control
- removed sheet Temp Sensors
- note added: "1. Monitor payload current? 2. Monitor Rockblock current? 3. OCP ckt? rockblock heritage is that it didnt work... 4. Input Power Decoupling?"
- note added: "EDGE CONNECTOR"
- note added: "NOTES:"
- note added: "TEMP SENSORS"
- note removed: "1. Monitor payload current 2. Monitor Rockblock current"
- note removed: "Edge Connector"
- note removed: "Input Load Switch"
- note removed: "Input Power Decoupling"
- note removed: "To MTs"
- note removed: "USB POWER"
- title: Foras Promineo Payload Interface Board -> Foras Promineo Payload Interface
- moved on the sheet: C1, C10, C11, C12, C2, C3, C6, C9, D1, D2, D3, D4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
