File: hardware/revB/temp_sensors.kicad_sch (KiCad schematic)
At the start: 12 parts, among them U24 MCP9700AT-E/LT

Commit message: revB initial commit
Parts:
- removed C100 (x3): 0.1uF, Capacitor_SMD:C_0402_1005Metric, symbol Device:C
- removed C99 (x3): 1uF, Capacitor_SMD:C_0603_1608Metric, symbol Device:C
- removed R36 (x3): 220, Resistor_SMD:R_0603_1608Metric, symbol Device:R_US
- removed U24 (x3): MCP9700AT-E/LT, Package_TO_SOT_SMD:SOT-353_SC-70-5, symbol Sensor_Temperature:MCP9700Ax-ELT
