File: revB/I2C-Protection.kicad_sch (KiCad schematic)
At the start: 18 parts, among them Q10 MMDT2222A, Q11 MMDT2222A, Q14 BSS138DWQ-7, Q15 BSS138DWQ-7

Commit message: updated BOM
Parts:
- C15, C16: Manufacturer (none) -> TDK Corporation; Mfr. Part No (none) -> CGA3E2X7R1H103K080AE
- Q10, Q11: Manufacturer (none) -> Diodes Incorporated; Mfr. Part No (none) -> MMDT2222A-7-F
- Q14, Q15: value BSS138DWQ-7 -> BSS138; Manufacturer (none) -> Diodes Incorporated; Mfr. Part No (none) -> BSS138DWQ-7
- R41, R42, R43, R44: Manufacturer (none) -> Stackpole Electronics Inc; Mfr. Part No (none) -> RMCF0603FT10K0
- R45, R46: Manufacturer (none) -> Stackpole Electronics Inc; Mfr. Part No (none) -> RMCF0603FT680R
- R47, R48: Manufacturer (none) -> Stackpole Electronics Inc; Mfr. Part No (none) -> RMCF0603FT100K
- R49, R50: value 200K -> 200k; Manufacturer (none) -> Stackpole Electronics Inc; Mfr. Part No (none) -> RMCF0603FT200K
- R51, R52: Manufacturer (none) -> Stackpole Electronics Inc; Mfr. Part No (none) -> RMCF0603ZT0R00
