File: revB/load_sw.kicad_sch (KiCad schematic)
At the start: 8 parts, among them Q13 BSZ180, Q2 MMBT4401WT1G

Commit message: updated BOM
Parts:
- C5: Manufacturer TDK -> TDK Corporation
- Q13: Manufacturer (none) -> Infineon Technologies; Mfr. Part No (none) -> BSZ180P03NS3GATMA1
- Q2: value MMBT4401WT1G -> MMBT4401; Manufacturer (none) -> onsemi; Mfr. Part No (none) -> MMBT4401WT1G
- R3, R5: Manufacturer (none) -> Stackpole Electronics Inc; Mfr. Part No (none) -> RMCF0603FT100K
- R4: Manufacturer (none) -> Stackpole Electronics Inc; Mfr. Part No (none) -> RMCF0603FG1K00
Changed lines of the file:
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@@
       (effects (font (size 1.27 1.27)) hide)
     )
-    (property "Datasheet" "~" (at 125.73 100.33 0)
-      (effects (font (size 1.27 1.27)) hide)
-    )
-    (property "Manufacturer" "" (at 125.73 100.33 0)
+    (property "Datasheet" "https://www.seielect.com/Catalog/SEI-RMCF_RMCP.pdf" (at 125.73 100.33 0)
+      (effects (font (size 1.27 1.27)) hide)
+    )
+    (property "Manufacturer" "Stackpole Electronics Inc" (at 125.73 100.33 0)
       (effects (font (size 1.27 1.27)) hide)
     )
@@
       (effects (font (size 1.27 1.27)) hide)
     )
-    (property "Description" "" (at 125.73 100.33 0)
-      (effects (font (size 1.27 1.27)) hide)
-    )
-    (property "Mfr. Part No" "" (at 125.73 100.33 0)
+    (property "Description" "RES 100K OHM 1% 1/10W 0603" (at 125.73 100.33 0)
+      (effects (font (size 1.27 1.27)) hide)
+    )
+    (property "Mfr. Part No" "RMCF0603FT100K" (at 125.73 100.33 0)
       (effects (font (size 1.27 1.27)) hide)
     )
@@
       (effects (font (size 1.27 1.27)) hide)
     )
-    (property "Datasheet" "~" (at 142.24 81.28 0)
+    (property "Datasheet" "https://product.tdk.com/en/system/files?file=dam/doc/product/capacitor/ceramic/mlcc/catalog/mlcc_automotive_soft_en.pdf" (at 142.24 81.28 0)
       (effects (font (size 1.27 1.27)) hide)
     )
@@
       (effects (font (size 1.27 1.27)) hide)
     )
-    (property "Manufacturer" "TDK" (at 142.24 81.28 0)
+    (property "Manufacturer" "TDK Corporation" (at 142.24 81.28 0)
       (effects (font (size 1.27 1.27)) hide)
     )
@@
       (effects (font (size 1.27 1.27)) hide)
     )
-    (property "Datasheet" "~" (at 156.21 86.36 0)
+    (property "Datasheet" "https://www.seielect.com/Catalog/SEI-RMCF_RMCP.pdf" (at 156.21 86.36 0)
+      (effects (font (size 1.27 1.27)) hide)
+    )
+    (property "Description" "RES 1K OHM 1% 1/10W 0603" (at 156.21 86.36 0)
+      (effects (font (size 1.27 1.27)) hide)
+    )
+    (property "Manufacturer" "Stackpole Electronics Inc" (at 156.21 86.36 0)
+      (effects (font (size 1.27 1.27)) hide)
+    )
+    (property "Mfr. Part No" "RMCF0603FG1K00" (at 156.21 86.36 0)
       (effects (font (size 1.27 1.27)) hide)
     )
@@
       (effects (font (size 1.27 1.27)) hide)
     )
-    (property "Datasheet" "BSZ180P03NS3GATMA1" (at 167.64 49.53 0)
+    (property "Datasheet" "https://www.infineon.com/dgdl/Infineon-BSZ180P03NS3_G-DS-v02_01-en.pdf?fileId=db3a304326dfb13001271f04398f4ec1" (at 167.64 49.53 0)
+      (effects (font (size 1.27 1.27)) hide)
+    )
+    (property "Description" "MOSFET P-CH 30V 9A/39.6A TSDSON" (at 166.37 58.42 0)
+      (effects (font (size 1.27 1.27)) hide)
+    )
+    (property "Manufacturer" "Infineon Technologies" (at 166.37 58.42 0)
+      (effects (font (size 1.27 1.27)) hide)
+    )
+    (property "Mfr. Part No" "BSZ180P03NS3GATMA1" (at 166.37 58.42 0)
       (effects (font (size 1.27 1.27)) hide)
     )
@@
       (effects (font (size 1.27 1.27)) (justify left))
     )
-    (property "Value" "MMBT4401WT1G" (at 139.7 101.5999 0)
+    (property "Value" "MMBT4401" (at 139.7 101.5999 0)
       (effects (font (size 1.27 1.27)) (justify left))
     )
@@
       (effects (font (size 1.27 1.27)) hide)
     )
-    (property "Datasheet" "~" (at 134.62 100.33 0)
+    (property "Datasheet" "https://www.onsemi.com/pdf/datasheet/mmbt4401wt1-d.pdf" (at 134.62 100.33 0)
+      (effects (font (size 1.27 1.27)) hide)
+    )
+    (property "Description" "TRANS NPN 40V 0.6A SC70-3" (at 134.62 100.33 0)
+      (effects (font (size 1.27 1.27)) hide)
+    )
+    (property "Manufacturer" "onsemi" (at 134.62 100.33 0)
+      (effects (font (size 1.27 1.27)) hide)
+    )
+    (property "Mfr. Part No" "MMBT4401WT1G" (at 134.62 100.33 0)
       (effects (font (size 1.27 1.27)) hide)
     )
@@
       (effects (font (size 1.27 1.27)) hide)
     )
-    (property "Datasheet" "~" (at 166.37 86.36 0)
+    (property "Datasheet" "https://www.seielect.com/Catalog/SEI-RMCF_RMCP.pdf" (at 166.37 86.36 0)
+      (effects (font (size 1.27 1.27)) hide)
+    )
+    (property "Description" "RES 1K OHM 1% 1/10W 0603" (at 166.37 86.36 0)
+      (effects (font (size 1.27 1.27)) hide)
+    )
+    (property "Manufacturer" "Stackpole Electronics Inc" (at 166.37 86.36 0)
+      (effects (font (size 1.27 1.27)) hide)
+    )
+    (property "Mfr. Part No" "RMCF0603FG1K00" (at 166.37 86.36 0)
       (effects (font (size 1.27 1.27)) hide)
     )
@@
       (effects (font (size 1.27 1.27)) hide)
     )
-    (property "Datasheet" "BSZ180P03NS3GATMA1" (at 157.48 64.77 0)
+    (property "Datasheet" "https://www.infineon.com/dgdl/Infineon-BSZ180P03NS3_G-DS-v02_01-en.pdf?fileId=db3a304326dfb13001271f04398f4ec1" (at 157.48 64.77 0)
+      (effects (font (size 1.27 1.27)) hide)
+    )
+    (property "Description" "MOSFET P-CH 30V 9A/39.6A TSDSON" (at 156.21 73.66 0)
+      (effects (font (size 1.27 1.27)) hide)
+    )
+    (property "Manufacturer" "Infineon Technologies" (at 156.21 73.66 0)
+      (effects (font (size 1.27 1.27)) hide)
+    )
+    (property "Mfr. Part No" "BSZ180P03NS3GATMA1" (at 156.21 73.66 0)
       (effects (font (size 1.27 1.27)) hide)
     )
@@
       (effects (font (size 1.27 1.27)) hide)
     )
-    (property "Datasheet" "~" (at 137.16 81.28 0)
-      (effects (font (size 1.27 1.27)) hide)
-    )
-    (property "Manufacturer" "" (at 137.16 81.28 0)
+    (property "Datasheet" "https://www.seielect.com/Catalog/SEI-RMCF_RMCP.pdf" (at 137.16 81.28 0)
+      (effects (font (size 1.27 1.27)) hide)
+    )
+    (property "Manufacturer" "Stackpole Electronics Inc" (at 137.16 81.28 0)
       (effects (font (size 1.27 1.27)) hide)
     )
@@
       (effects (font (size 1.27 1.27)) hide)
     )
-    (property "Description" "" (at 137.16 81.28 0)
-      (effects (font (size 1.27 1.27)) hide)
-    )
+    (property "Description" "RES 100K OHM 1% 1/10W 0603" (at 137.16 81.28 0)
+      (effects (font (size 1.27 1.27)) hide)
+    )
+    (property "Mfr. Part No" "RMCF0603FT100K" (at 137.16 81.28 0)
+      (effects (font (size 1.27 1.27)) hide)
+    )
