File: revB/payload-interface-board.kicad_sch (KiCad schematic)
At the start: 91 parts, among them J1 T1M-10-F-SV-L, J2 T1M-10-F-SV-L, P1 Card Edge for HSEC8-160-01-S-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, Q2 MMDT2222A, Q3 MMDT2222A, Q39 MMDT3946, U1 LTC4307, U2 RockBlock_9603, U24 MCP9700AT-E/LT, U3 SN74LVCH245APWR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

Commit message: updated BOM
Parts:
- C1: Manufacturer (none) -> TDK Corporation; Mfr. Part No (none) -> CGA3E2X7R1H103K080AE
- C10, C100, C11, C12, C2, C3, C9: Manufacturer TDK -> TDK Corporation
- C6: Manufacturer (none) -> TDK Corporation; Mfr. Part No (none) -> CGA4J1X7S1E106K125AE
- C99: Manufacturer (none) -> TDK Corporation; Mfr. Part No (none) -> CGA3E1X7R1E105K080AE
- D1: Manufacturer (none) -> Kingbright; Mfr. Part No (none) -> APA2107LSECK/J3-PRV
- D2: Manufacturer (none) -> Kingbright; Mfr. Part No (none) -> APA2107SYCK
- D3: Manufacturer (none) -> Kingbright; Mfr. Part No (none) -> APA2107SECK
- D4: Manufacturer (none) -> Kingbright; Mfr. Part No (none) -> APA2107CGCK
- H1, H2, H3, H4, P1: now left out of the parts list
- J1, J2: Manufacturer (none) -> Samtec; Mfr. Part No (none) -> T1M-10-F-SV-L
- Q2, Q3: Manufacturer (none) -> Diodes Incorporated
- Q39: Manufacturer (none) -> Diodes Incorporated; Mfr. Part No (none) -> MMDT3946-7-F
- R1, R2, R5, R6: Manufacturer (none) -> Stackpole Electronics Inc; Mfr. Part No (none) -> RMCF0603FT100K
- R10, R7, R8, R9: Manufacturer (none) -> Stackpole Electronics Inc; Mfr. Part No (none) -> RMCF0603ZT0R00
- R11, R12, R15, R16, R22: Manufacturer (none) -> Stackpole Electronics Inc; Mfr. Part No (none) -> RMCF0603FT10K0
- R13, R14, R17, R18: Manufacturer (none) -> Stackpole Electronics Inc; Mfr. Part No (none) -> RMCF0603FG1K00
- R20: value 988k -> 976k; Manufacturer (none) -> Stackpole Electronics Inc; Mfr. Part No (none) -> RMCF0603FT976K
- R23: Manufacturer (none) -> Stackpole Electronics Inc; Mfr. Part No (none) -> RMCF0603FT105K
- R24: Manufacturer (none) -> Stackpole Electronics Inc; Mfr. Part No (none) -> RMCF0603FT576K
- R25, R26, R27, R28: Manufacturer (none) -> Stackpole Electronics Inc; Mfr. Part No (none) -> RMCF0402FT1K50
- R29, R30, R31, R32: Manufacturer (none) -> Stackpole Electronics Inc; Mfr. Part No (none) -> RMCF0402FT10K0
- R3, R4: Manufacturer (none) -> Stackpole Electronics Inc; Mfr. Part No (none) -> RMCF0603FT4K70
- R36: Manufacturer (none) -> Stackpole Electronics Inc; Mfr. Part No (none) -> RMCF0603FT220R
- RN1: Manufacturer (none) -> Panasonic; Mfr. Part No (none) -> EXB-28V102JX
- RN2: Manufacturer (none) -> Panasonic; Mfr. Part No (none) -> EXB-28V103JX
- TP10, TP11, TP12, TP13, TP14, TP16, TP17, TP18, TP19, TP2, TP20, TP22, TP3, TP4, TP5, TP6, TP9: Mfr. Part No 500x -> 5002
- U1: Manufacturer (none) -> Analog Devices; Mfr. Part No (none) -> LTC4307IMS8#TRPBF
- U2: Manufacturer (none) -> Ground Control; Mfr. Part No (none) -> FP-RB-9603
- U24: Manufacturer (none) -> Microchip Technology; Mfr. Part No (none) -> MCP9700AT-E/LT
- U3, U4: Manufacturer (none) -> Texas Instruments; Mfr. Part No (none) -> SN74LVCH245APWR
- U6: Manufacturer (none) -> Sierra Lobo; Mfr. Part No (none) -> RD21-6005A
